File: V1/Design/HW.ACIM-MCU-E70/HW.ACIM-MCU-E70.kicad_pcb (KiCad board)
At the start: 4 copper layers, 32 x 20 mm, 31 parts, among them J1 HEADER 2x15POS, J2 HEADER 2x15POS, U1 dsPIC33AKxxxMC106, U2 12MHz

Commit message: HW.ACIM-MCU-E70 schematic update 1
Parts:
- removed C22, C24, C26: 10uF, SAMPI:CAP0402
- added C5: 100nF, SAMPI:CAP0402, F.Cu at (119.5, 95.7)
- added C6: 100nF, SAMPI:CAP0402, F.Cu at (119.5, 98.0)
- added FT1: 1K@100MHz, SAMPI:IND0402, F.Cu at (119.5, 100.3)
- added FT2: 1K@100MHz, SAMPI:IND0402, F.Cu at (119.5, 102.6)
- added R4: 10K, SAMPI:RES0402, F.Cu at (119.5, 104.9)
- added R5: 1K, SAMPI:RES0402, F.Cu at (119.5, 107.2)
- added TP5: ERASE, SAMPI:TP1MM, F.Cu at (122.8, 96.3)
- added TP6: VCORE, SAMPI:TP1MM, F.Cu at (122.8, 99.9)
- C2: value 10uF -> 100nF
- C3: value 10uF -> 2.2uF
- U1: value dsPIC33AKxxxMC106 -> ATSAME70J20B
- moved C20 19.6 mm to (89.9, 100.2), turned to -45 degrees
- moved U2 18.8 mm to (91.6, 98.1), turned to -135 degrees
- moved C19 18.2 mm to (93.7, 96.5), turned to 135 degrees
- moved C23 9.85 mm to (113.0, 116.2)
- moved C10 9.85 mm to (111.3, 117.9)
- moved C2 9.85 mm to (113.9, 115.3)
- moved C12 9.35 mm to (92.9, 116.9)
- moved C13 9.35 mm to (92.1, 116.1)
- moved C28 7.72 mm to (93.8, 90.3)
- moved C4 7.72 mm to (95.5, 88.6)
- moved C27 7.72 mm to (94.6, 89.5)
- moved C3 7.72 mm to (96.3, 87.8)
- moved C21 6.42 mm to (97.7, 116.2)
- moved R2 6.42 mm to (98.5, 117.0)
- moved C1 6.28 mm to (104.7, 87.7)
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Connections:
- C10 pad 2: +3V3 -> Net-(U1-VDDOUT)
- C19 pad 2: Net-(U1-OSCO/CLKO/RP33/IOMF5/RC0) -> Net-(U1-PB8/XOUT)
- C2 pad 2: +3V3 -> Net-(U1-VDDOUT)
- C20 pad 2: Net-(U1-OSCI/CLKI/RP34/IOMF6/RC1) -> Net-(U1-PB9/XIN)
- C3 pad 2: +3V3 -> Net-(U1-VDDOUT)
- C4 pad 2: +3V3 -> Net-(U1-VDDOUT)
- J1 pad 17: /PFC_PWM_ENB -> unconnected-(J1-Pad17)
- J1 pad 18: /PFC_PWM_B -> unconnected-(J1-Pad18)
- J1 pad 19: /PFC_PWM_ENA -> unconnected-(J1-Pad19)
- J1 pad 20: /PFC_PWM_A -> unconnected-(J1-Pad20)
- J1 pad 21: /VAC_DIV -> unconnected-(J1-Pad21)
- J1 pad 22: /~{PFC_FLT} -> unconnected-(J1-Pad22)
- J1 pad 24: /PFC_IB_SEN -> unconnected-(J1-Pad24)
- J1 pad 26: /PFC_IA_SEN -> unconnected-(J1-Pad26)
- J1 pad 27: /ENC_HOME -> unconnected-(J1-Pad27)
- J1 pad 29: /ENC_IDX -> unconnected-(J1-Pad29)
- J2 pad 1: /VBUS -> /USB_VBUS
- J2 pad 2: /PGD -> /SWDIO
- J2 pad 21: /MC_TEMP_SEN -> unconnected-(J2-Pad21)
- J2 pad 23: /MC_VU_DIV -> unconnected-(J2-Pad23)
- J2 pad 25: /MC_VV_DIV -> unconnected-(J2-Pad25)
- J2 pad 4: /PGC -> /SWDCLK
- U1 pad 10: AGND -> +3V3
- U1 pad 11: AVDD -> /IDC_SEN
- U1 pad 12: unconnected-(U1-OA1OUT/AD1AN0/CMP1A/RP3/RA2-Pad12) -> /MC_IV_SEN
- U1 pad 13: unconnected-(U1-OA1IN-/AD1ANN1/AD2AN0/RP4/RA3-Pad13) -> Net-(U1-VDDOUT)
- U1 pad 14: unconnected-(U1-OA1IN+/AD1AN1/CMP1B/RP5/RA4-Pad14) -> GND
- U1 pad 15: unconnected-(U1-OA3OUT/AD1AN3/CMP3A/RP6/RA5-Pad15) -> /USB_VBUS
- U1 pad 16: unconnected-(U1-OA3IN-/AD1AN2/RP7/RA6-Pad16) -> /SLED
- U1 pad 18: GND -> /MC_PWM_WH
- U1 pad 19: +3V3 -> unconnected-(U1-PA14/PWM0.H3/PWM1.H1/QSPI_CLK-Pad19)
- U1 pad 20: unconnected-(U1-OA2OUT/AD2AN1/CMP2A/RP17/INT0/RB0-Pad20) -> /MC_PWM_VL
- U1 pad 21: unconnected-(U1-TMS/OA2IN-/AD1AN4/AD2ANN1/RP18/RB1-Pad21) -> /MC_PWM_WL
- U1 pad 22: unconnected-(U1-OA2IN+/AD2AN4/CMP2B/RP19/RB2-Pad22) -> /MC_PWM_UL
- U1 pad 24: unconnected-(U1-AD2AN10/RP26/RB9-Pad24) -> Net-(U1-VDDOUT)
- U1 pad 25: GND -> /ENC_B
- U1 pad 26: +3V3 -> /ENC_A
- U1 pad 27: /PGD -> /MC_PWM_UH
- U1 pad 28: /PGC -> /DB_TXD
- U1 pad 29: unconnected-(U1-AD1ANN2/AD1AN8/RP23/RB6-Pad29) -> /MC_PWM_VH
- U1 pad 3: unconnected-(U1-PGC2/DACOUT1/AD1AN7/AD2AN3/CMP1D/CMP2D/CMP3D/RP2/SCL2/RA1-Pad3) -> Net-(U1-VDDOUT)
- U1 pad 31: unconnected-(U1-RP27/SCK2/RB10-Pad31) -> GND
- U1 pad 32: unconnected-(U1-RP28/SDI2/RB11-Pad32) -> /DV_RXD
- U1 pad 33: unconnected-(U1-RP41/IOMD11/IOMF11/PCI20/RC8-Pad33) -> /DB_RXD
- U1 pad 34: unconnected-(U1-RP42/IOMD10/SDO2/IOMF10/PCI19/RC9-Pad34) -> /DV_TXD
- U1 pad 35: unconnected-(U1-RP39/RC6-Pad35) -> /SWDIO
- U1 pad 36: unconnected-(U1-RP40/RC7-Pad36) -> /~{MCLR}
- U1 pad 37: Net-(U1-OSCO/CLKO/RP33/IOMF5/RC0) -> unconnected-(U1-TST-Pad37)
- U1 pad 38: Net-(U1-OSCI/CLKI/RP34/IOMF6/RC1) -> Net-(U1-PB12/PWM0.L1/ERASE)
- U1 pad 39: GND -> /SWDCLK
- U1 pad 4: GND -> +3V3
- U1 pad 40: +3V3 -> unconnected-(U1-PA3/SDA0/USLONCOL1-Pad40)
- U1 pad 42: unconnected-(U1-RP38/PWM4L/RC5-Pad42) -> +3V3
- U1 pad 43: /MC_PWM_WH -> unconnected-(U1-PD11/PWM0.H0-Pad43)
- U1 pad 44: /MC_PWM_WL -> unconnected-(U1-PD10/PWM0.L0-Pad44)
- U1 pad 46: unconnected-(U1-RP44/IOMD8/IOMF8/RC11-Pad46) -> /SDA
- U1 pad 47: GND -> /SCL
- U1 pad 48: +3V3 -> unconnected-(U1-PD9/PWM0.F2-Pad48)
- U1 pad 5: +3V3 -> AVDD
- U1 pad 51: /MC_PWM_VH -> unconnected-(U1-PD6/PWM1.L3-Pad51)
- U1 pad 52: /MC_PWM_VL -> Net-(U1-VDDPLL)
- U1 pad 53: /MC_PWM_UH -> unconnected-(U1-PD5/PWM1.H2-Pad53)
- U1 pad 54: /MC_PWM_UL -> unconnected-(U1-PD4/PWM1.L2-Pad54)
- U1 pad 55: /SDA -> unconnected-(U1-PD3/PWM1.H1/USRI0-Pad55)
- U1 pad 58: unconnected-(U1-RP57/ASDA2/IOMD6/IOMF3/RD8-Pad58) -> +3V3
- U1 pad 59: GND -> /USB_N
- U1 pad 6: unconnected-(U1-AD1AN10/RP12/RA11-Pad6) -> GND
- U1 pad 60: +3V3 -> /USB_P
- U1 pad 61: /SCL -> Net-(U1-VDDOUT)
- U1 pad 62: unconnected-(U1-RP60/RD11-Pad62) -> Net-(U1-PB8/XOUT)
- U1 pad 63: unconnected-(U1-RP61/PCI21/RD12-Pad63) -> Net-(U1-PB9/XIN)
- U1 pad 64: /~{MCLR} -> +3V3
- U1 pad 7: unconnected-(U1-AD2AN9/ISRC3/IBIAS3/RP9/RA8-Pad7) -> /MC_VR_DIV
- U1 pad 8: unconnected-(U1-AD1ANN3/AD1AN9/RP10/RA9-Pad8) -> /MC_IU_SEN
- U1 pad 9: unconnected-(U1-AD2ANN3/AD2AN7/RP11/RA10-Pad9) -> /VDC_DIV
- U2 pad 1: Net-(U1-OSCO/CLKO/RP33/IOMF5/RC0) -> Net-(U1-PB8/XOUT)
- U2 pad 3: Net-(U1-OSCI/CLKI/RP34/IOMF6/RC1) -> Net-(U1-PB9/XIN)
Routing:
- net /USB_P: track 0.00 -> 21.0 mm
- net /USB_N: track 0.00 -> 20.5 mm
- net /SLED: track 0.00 -> 14.1 mm
- net /USB_VBUS: track 0.00 -> 14.0 mm, vias 0 -> 1
- net +3V3: track 12.1 -> 0.00 mm
- net AGND: track 5.02 -> 0.00 mm
- net /~{MCLR}: track 4.00 -> 0.00 mm
- net AVDD: track 3.81 -> 0.00 mm
- net Net-(D1-PadA): track 0.00 -> 1.30 mm
- removed copper zone on B.Cu, net GND
- removed copper zone on F.Cu, net GND
- removed copper zone on In1.Cu, net GND
- removed copper zone on In2.Cu, net GND
Other:
- board text added: "HW.ACIM-MCU-E70"
- board text removed: "HW.ACIM-MCU-33AK"

Commit message: HW.ACIM-MCU-E70 schematic update 2
Connections:
- FT2 pad 2: +3V3 -> GND
Changed lines of the file:
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@@
 			(size 0.5 0.6)
 			(layers "F.Cu" "F.Paste" "F.Mask")
-			(net 5 "+3V3")
+			(net 1 "GND")
 			(pinfunction "2")
 			(pintype "bidirectional")
