File: V1/Design/HW.ACIM-MCU-E70/HW.ACIM-MCU-E70.kicad_sch (KiCad schematic)
At the start: 31 parts, among them J1 HEADER 2x15POS, J2 HEADER 2x15POS, U1 ATSAME70J20B, U2 12MHz

Commit message: HW.ACIM-MCU-E70 schematic
Parts:
- removed C22, C24, C26: 10uF, SAMPI:CAP0402, symbol SAMPI:CERCAP
- added C5, C6: 100nF, SAMPI:CAP0402, symbol SAMPI:CERCAP
- added FT1, FT2: 1K@100MHz, symbol SAMPI:FerriteBead
- added R4: 10K, SAMPI:RES0402, symbol SAMPI:RES
- added R5: 1K, SAMPI:RES0402, symbol SAMPI:RES
- added TP6: VCORE, SAMPI:TP1MM, symbol Liem:TESTPOINT
- added U3: ADC-8CH, SAMPI:SOIC16-3.9, symbol SAMPI:ADC-8CH
- C2: value 10uF -> 100nF; MNP GRM155C80J106ME11D -> GRM155R71H104ME14D
- C3: value 10uF -> 2.2uF
Connections:
- net PGC is gone; now on net SWDCLK: J2.4
- net PGD is gone; now on net SWDIO: J2.2
- net +3V3: now also U1.10 (VDDIO), U1.4 (VDDIN), U1.42 (VDDIO), U1.58 (VDDIO), U1.64 (VDDPLLUSB), FT2.2; no longer C10.2, C2.2, C3.2, C4.2
- net AGND: now also FT2.1
- net AVDD: now also U1.5 (VREFP)
- net DB_RXD: now also U1.33 (PA9/PWM0.F0/URXD0)
- net DB_TXD: now also U1.28 (PA10/UTXD0)
- net DV_RXD: now also U1.32 (PA5/PWM1.L3/URXD1)
- net DV_TXD: now also U1.34 (PA4/SCL0/UTXD1)
- net ENC_A: now also U1.26 (PD21/PWM0.H1/QEI3A)
- net ENC_B: now also U1.25 (PD22/PWM0.H2/QEI3B)
- net GND: now also U1.14 (GND), U1.31 (GND), U1.6 (GND), C5.1, C6.1, R4.1
- net IDC_SEN: now also U1.11 (PB3/AD0.2/USRTS0)
- net MC_IU_SEN: now also U1.8 (PB0/AD0.10/PWM0.H0/USRXD0)
- net MC_IV_SEN: now also U1.12 (PA21/AD0.1/PWM1.F0/USRXD1)
- net MC_PWM_UH: now also U1.27 (PA11/PWM0.H0/PWM1.L0)
- net MC_PWM_UL: now also U1.22 (PD24/PWM0.L0)
- net MC_PWM_VH: now also U1.29 (PA12/PWM0.H1/PWM1.H0)
- net MC_PWM_VL: now also U1.20 (PD25/PWM0.L1/URXD2)
- net MC_PWM_WH: now also U1.18 (PA13/PWM0.H2/PWM1.L1)
- net MC_PWM_WL: now also U1.21 (PD26/PWM0.L2/UTXD1/UTXD2)
- net USB_N: now also U1.59 (DM)
- net USB_P: now also U1.60 (DP)
- net VDC_DIV: now also U1.9 (PB2/AD0.5/USCTS0)
- net ~{MCLR}: now also U1.36 (NRST)
- net at TP5.1, U1.38 (PB12/PWM0.L1/ERASE): now also R4.2
- net at U1.13 (VDDCORE): now also C10.2, C2.2, C3.2, C4.2, U1.24 (VDDCORE), U1.3 (VDDOUT), U1.61 (VDDCORE), C6.2, FT1.2, TP6.1
- net SWDIO: now reaches U1.35 (PB6/SWDIO)
- net SWDCLK: now reaches U1.39 (PB7/SWDCLK)
- net at U1.52 (VDDPLL): now also C5.2, FT1.1
- net DV_CTS: no longer names the net of J2.12
- net DV_CTS: now also R5.1
- net DV_RTS: no longer names the net of J2.11
- net DV_RTS: now also R5.2
- net ENC_HOME: no longer names the net of J1.27
- net ENC_IDX: no longer names the net of J1.29
- net PFC_IA_SEN renamed MC_ALT_IU_SEN
- net PFC_IB_SEN renamed MC_ALT_IV_SEN
- net PFC_PWM_A: no longer names the net of J1.20
- net PFC_PWM_B: no longer names the net of J1.18
- net PFC_PWM_ENA: no longer names the net of J1.19
- net PFC_PWM_ENB: no longer names the net of J1.17
- net SCL: no longer names the net of J1.11
- net SDA: no longer names the net of J1.12
- net VAC_DIV renamed MC_VW_DIV
- net VBUS: no longer names the net of J2.1
- net ~{PFC_FLT}: no longer names the net of J1.22
- no-connect marks 0 -> 12
Other:
- moved on the sheet: C1, C10, C12, C13, C19, C20, C21, C23, C25, C27, C28, C3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

Commit message: HW.ACIM-MCU-E70 schematic update 1
Parts:
- removed U3: ADC-8CH, SAMPI:SOIC16-3.9, symbol SAMPI:ADC-8CH
- FT1, FT2: footprint (none) -> SAMPI:IND0402; MFT (none) -> Murata; MNP (none) -> BLM15AG102SH1D
Connections:
- net MC_VR_DIV: now also U1.7 (PB1/AD1.0/PWM0.H1/USTXD0)
- net SLED: now also U1.16 (PA8/PWM1.H3/XOUT32)
- net DV_CTS: now reaches J2.12, R5.1
- net DV_RTS: now reaches J2.11, R5.2
- net USB_VBUS: now reaches J2.1
- net USB_VBUS: now also U1.15 (PA7/PWM0.H3/XIN32)
- net SCL: now reaches J1.11
- net SCL: now also U1.47 (PB5/PWM0.L0/SCL1)
- net SDA: now reaches J1.12
- net SDA: now also U1.46 (PB4/PWM0.H2/SDA1/USTXD1)
- net MC_ALT_IU_SEN: no longer names the net of J1.26
- net MC_ALT_IV_SEN: no longer names the net of J1.24
- net MC_TEMP_SEN: no longer names the net of J2.21
- net MC_VU_DIV: no longer names the net of J2.23
- net MC_VV_DIV: no longer names the net of J2.25
- net MC_VW_DIV: no longer names the net of J1.21
- no-connect marks 12 -> 15
Other:
- moved on the sheet: C5

Commit message: HW.ACIM-MCU-E70 schematic update 2
Connections:
- net +3V3: no longer FT2.2
- net GND: now also FT2.2
Other:
- moved on the sheet: C1, C27, C28, FT2, R3
