File: V1/Design/HW.ACIM-INV/Power.kicad_sch (KiCad schematic)
At the start: 42 parts, among them J1 HIGH VOLT, J4 LOW VOLT, U14 LDO 3.3V/1.5A, U18 LDO 3.3V/250mA, U8 LDO 3.3V±0.1%/20mA

Commit message: V1 schematic update 2
Parts:
- removed C102, C103: 100pF/2kV, SAMPI:CAP1206, symbol SAMPI:CERCAP
- removed C48, C55, C85, C87: 10uF, SAMPI:CAP0603, symbol SAMPI:CERCAP
- removed C49: 22pF, SAMPI:CAP0603, symbol SAMPI:CERCAP
- removed C50, C53, C78, C79, C86, C88: 100nF, SAMPI:CAP0603, symbol SAMPI:CERCAP
- removed C83: 220uF/6.3V, SAMPI:CAP1411, symbol SAMPI:ELECCAP
- removed MD1: DC-DC, Liem:B1524S-1WR3, symbol SAMPI:DC-DC
- removed TP10: 24V, SAMPI:TP1MM, symbol SAMPI:TESTPOINT
- removed TP11: GND1, SAMPI:TP1MM, symbol SAMPI:TESTPOINT
- removed TP12: 15V, SAMPI:TP1MM, symbol SAMPI:TESTPOINT
- removed TP13: 5V, SAMPI:TP1MM, symbol SAMPI:TESTPOINT
- removed TP14: 3V3, SAMPI:TP1MM, symbol SAMPI:TESTPOINT
- removed TP15: VREF, SAMPI:TP1MM, symbol SAMPI:TESTPOINT
- removed TP16: VDC, SAMPI:TP1MM, symbol SAMPI:TESTPOINT
- removed TP17: AVDD, SAMPI:TP1MM, symbol SAMPI:TESTPOINT
- removed TP18: PGND, SAMPI:TP1MM, symbol SAMPI:TESTPOINT
- removed TP19: GND, SAMPI:TP1MM, symbol SAMPI:TESTPOINT
- removed TP20: AGND, SAMPI:TP1MM, symbol SAMPI:TESTPOINT
- removed U14: LDO 3.3V/1.5A, SAMPI:DFN8_3x3_MCHP, symbol SAMPI:MCP1727
- removed U18: LDO 3.3V/250mA, SAMPI:SOT23, symbol SAMPI:LDO
- removed U8: LDO 3.3V±0.1%/20mA, SAMPI:SOT-23-6_MCHP, symbol SAMPI:MCP1501
Connections:
- net ~{INV_FAULT} is gone; now on net GND: J4.2
- net ~{PWR_FAULT} is gone; now on net GND: J4.1
- net +15V: now also J4.5; no longer J4.6
- net +3V3: now also J4.3
- net +3V3_ISO: now also J4.9
- net GND: no longer J4.3, J4.5
- net GND_ISO: now also J4.8; no longer J4.9
- no-connect marks 1 -> 0
Other:
- note added: "SAFE-ZONE"
- note removed: "ISOLATED POWER SAFE-ZONE"
- moved on the sheet: C1, C32, C54, C56, C57, C58, C59, C75, FT1, FT2, FT3, J4

Commit message: V1 schematic update 3
Parts:
- removed J4: LOW VOLT, SAMPI:HDM1x10x2.54_TH_RA, symbol SAMPI:SIL10
- added J2: LOW VOLT, symbol SAMPI:SIL12
Connections:
- net +15V: now also J2.7
- net +24V_ISO: now also J2.12
- net +3V3: now also J2.5
- net +3V3_ISO: now also J2.11
- net +5V: now also J2.6
- net GND: now also J2.1, J2.2
- net GND_ISO: now also J2.10
- new net DEV_RELAY: J2.3
- new net PWR_RELAY: J2.4
Changed lines of the file:
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@@
+		)
+	)
+	(hierarchical_label "DEV_RELAY"
+		(shape input)
+		(at 31.75 82.55 0)
+		(fields_autoplaced yes)
+		(effects
+			(font
+				(size 1.27 1.27)
+			)
+			(justify left)
+		)
+	)
+	(hierarchical_label "PWR_RELAY"
+		(shape input)
+		(at 31.75 80.01 0)
+		(fields_autoplaced yes)
+		(effects
+			(font
+				(size 1.27 1.27)
+			)
+			(justify left)
 		)
 	)
@@
 				(path "/20f80521-75f2-4ccc-bb34-c9566e70ef5c/34b63420-23a7-4d2d-affc-c07be2bf5f59"
 					(reference "#PWR0107")
-					(unit 1)
-				)
-			)
-		)
-	)
-	(symbol
-		(lib_id "SAMPI:SIL10")
-		(at 31.75 86.36 180)
-		(unit 1)
-		(exclude_from_sim no)
-		(in_bom yes)
-		(on_board yes)
-		(dnp no)
-		(property "Reference" "J4"
-			(at 24.13 72.39 0)
-			(effects
-				(font
-					(size 1.5 1.5)
-					(bold yes)
-				)
-				(justify left)
-			)
-		)
-		(property "Value" "LOW VOLT"
-			(at 25.4 68.58 90)
-			(effects
-				(font
-					(size 1.27 1.27)
-				)
-				(justify left)
-			)
-		)
-		(property "Footprint" "SAMPI:HDM1x10x2.54_TH_RA"
-			(at 31.75 86.36 0)
-			(effects
-				(font
-					(size 1.27 1.27)
-				)
-				(hide yes)
-			)
-		)
-		(property "Datasheet" ""
-			(at 31.75 86.36 0)
-			(effects
-				(font
-					(size 1.27 1.27)
-				)
-				(hide yes)
-			)
-		)
-		(property "Description" "CONN HDR 10POS 0.1 TIN PCB R/A"
-			(at 31.75 86.36 0)
-			(effects
-				(font
-					(size 1.27 1.27)
-				)
-				(hide yes)
-			)
-		)
-		(property "MFT" "Sullins"
-			(at 31.75 86.36 0)
-			(effects
-				(font
-					(size 1.27 1.27)
-				)
-				(hide yes)
-			)
-		)
-		(property "MNP" "PPTC101LGBN-RC"
-			(at 31.75 86.36 0)
-			(effects
-				(font
-					(size 1.27 1.27)
-				)
-				(hide yes)
-			)
-		)
-		(property "Checked" "OK"
-			(at 31.75 86.36 0)
-			(effects
-				(font
-					(size 1.27 1.27)
-				)
-				(hide yes)
-			)
-		)
-		(pin "8"
-		)
-		(pin "1"
-		)
-		(pin "2"
-		)
-		(pin "10"
-		)
-		(pin "4"
-		)
-		(pin "3"
-		)
-		(pin "9"
-		)
-		(pin "5"
-		)
-		(instances
-			(project "HW.ACIM-INV"
-				(path "/20f80521-75f2-4ccc-bb34-c9566e70ef5c/34b63420-23a7-4d2d-affc-c07be2bf5f59"
-					(reference "J4")
 					(unit 1)
 				)
@@
 	)
 	(symbol
+		(lib_id "SAMPI:SIL12")
+		(at 29.21 92.71 180)
+		(unit 1)
+		(exclude_from_sim no)
+		(in_bom yes)
+		(on_board yes)
+		(dnp no)
+		(property "Reference" "J2"
+			(at 24.13 76.835 0)
+			(effects
+				(font
+					(size 1.27 1.27)
+					(thickness 0.254)
+					(bold yes)
+				)
+				(justify left)
+			)
+		)
+		(property "Value" "LOW VOLT"
+			(at 26.035 72.3901 90)
+			(effects
+				(font
+					(size 1.27 1.27)
+				)
+				(justify left)
+			)
+		)
+		(property "Footprint" ""
+			(at 29.21 92.71 0)
+			(effects
+				(font
+					(size 1.27 1.27)
+				)
+				(hide yes)
+			)
+		)
+		(property "Datasheet" ""
+			(at 29.21 92.71 0)
+			(effects
+				(font
+					(size 1.27 1.27)
+				)
+				(hide yes)
+			)
+		)
+		(property "Description" ""
+			(at 29.21 92.71 0)
+			(effects
+				(font
+					(size 1.27 1.27)
+				)
+				(hide yes)
+			)
+		)
+		(pin "4"
+		)
+		(pin "3"
+		)
+		(pin "10"
+		)
+		(pin "2"
+		)
+		(pin "6"
+		)
+		(pin "1"
+		)
+		(pin "5"
+		)
+		(pin "7"
+		)
+		(pin "11"
+		)
+		(pin "12"
+		)
+		(instances
+			(project ""
+				(path "/20f80521-75f2-4ccc-bb34-c9566e70ef5c/34b63420-23a7-4d2d-affc-c07be2bf5f59"
+					(reference "J2")
+					(unit 1)
+				)
+			)
+		)
+	)
+	(symbol
 		(lib_id "power:GND")
 		(at 90.17 39.37 0)
@@
 	(symbol
 		(lib_id "power:GND")
-		(at 31.75 82.55 90)
+		(at 31.75 87.63 90)
 		(unit 1)
 		(exclude_from_sim no)
@@
 		(dnp no)
 		(property "Reference" "#PWR068"
-			(at 38.1 82.55 0)
+			(at 38.1 87.63 0)
 			(effects
 				(font
@@
 		)
 		(property "Value" "GND"
-			(at 36.195 82.55 90)
+			(at 36.195 87.63 90)
 			(effects
 				(font
@@
 		)
 		(property "Footprint" ""
-			(at 31.75 82.55 0)
-			(effects
-				(font
-					(size 1.27 1.27)
-				)
-				(hide yes)
-			)
-		)
-		(property "Datasheet" ""
-			(at 31.75 82.55 0)
+			(at 31.75 87.63 0)
+			(effects
+				(font
+					(size 1.27 1.27)
+				)
+				(hide yes)
+			)
+		)
+		(property "Datasheet" ""
+			(at 31.75 87.63 0)
 			(effects
 				(font
@@
 		)
 		(property "Description" ""
-			(at 31.75 82.55 0)
+			(at 31.75 87.63 0)
 			(effects
 				(font
@@
 	(symbol
 		(lib_id "power:GND")
-		(at 31.75 80.01 90)
+		(at 31.75 85.09 90)
 		(unit 1)
 		(exclude_from_sim no)
@@
 		(dnp no)
 		(property "Reference" "#PWR064"
-			(at 38.1 80.01 0)
+			(at 38.1 85.09 0)
 			(effects
 				(font
@@
 		)
 		(property "Value" "GND"
-			(at 36.195 80.01 90)
+			(at 36.195 85.09 90)
 			(effects
 				(font
@@
 		)
 		(property "Footprint" ""
-			(at 31.75 80.01 0)
-			(effects
-				(font
-					(size 1.27 1.27)
-				)
-				(hide yes)
-			)
-		)
-		(property "Datasheet" ""
-			(at 31.75 80.01 0)
+			(at 31.75 85.09 0)
+			(effects
+				(font
+					(size 1.27 1.27)
+				)
+				(hide yes)
+			)
+		)
+		(property "Datasheet" ""
+			(at 31.75 85.09 0)
 			(effects
 				(font
@@
 		)
 		(property "Description" ""
-			(at 31.75 80.01 0)
-			(effects
-				(font
+			(at 31.75 85.09 0)
+			(effects
+				(font

Commit message: V1 schematic update 4
Parts:
- J2: footprint (none) -> SAMPI:HDM1x12x2.54_TH_RA; MFT (none) -> Sullins; MNP (none) -> PBC12SBAN
Connections:
- net +3V3_ISO renamed +5V_ISO
Changed lines of the file:
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@@
-	)
-	(symbol
-		(lib_id "SAMPI:+3V3_ISO")
-		(at 31.75 62.23 270)
-		(mirror x)
-		(unit 1)
-		(exclude_from_sim no)
-		(in_bom yes)
-		(on_board yes)
-		(dnp no)
-		(property "Reference" "#PWR0227"
-			(at 27.94 62.23 0)
-			(effects
-				(font
-					(size 1.27 1.27)
-				)
-				(hide yes)
-			)
-		)
-		(property "Value" "+3V3_ISO"
-			(at 38.735 62.23 90)
-			(effects
-				(font
-					(size 1.27 1.27)
-					(bold yes)
-				)
-			)
-		)
-		(property "Footprint" ""
-			(at 31.75 62.23 0)
-			(effects
-				(font
-					(size 1.27 1.27)
-				)
-				(hide yes)
-			)
-		)
-		(property "Datasheet" ""
-			(at 31.75 62.23 0)
-			(effects
-				(font
-					(size 1.27 1.27)
-				)
-				(hide yes)
-			)
-		)
-		(property "Description" "Power symbol creates a global label with name \"+3V3_ISO\""
-			(at 31.75 62.23 0)
-			(effects
-				(font
-					(size 1.27 1.27)
-				)
-				(hide yes)
-			)
-		)
-		(pin "1"
-		)
-		(instances
-			(project "HW.ACIM-INV"
-				(path "/20f80521-75f2-4ccc-bb34-c9566e70ef5c/34b63420-23a7-4d2d-affc-c07be2bf5f59"
-					(reference "#PWR0227")
-					(unit 1)
-				)
-			)
-		)
 	)
 	(symbol
@@
 			)
 		)
-		(property "Footprint" ""
+		(property "Footprint" "SAMPI:HDM1x12x2.54_TH_RA"
 			(at 29.21 92.71 0)
 			(effects
@@
 			)
 		)
-		(property "Description" ""
+		(property "Description" "CONN HEADER R/A 12POS 2.54MM"
+			(at 29.21 92.71 0)
+			(effects
+				(font
+					(size 1.27 1.27)
+				)
+				(hide yes)
+			)
+		)
+		(property "MNP" "PBC12SBAN"
+			(at 29.21 92.71 0)
+			(effects
+				(font
+					(size 1.27 1.27)
+				)
+				(hide yes)
+			)
+		)
+		(property "MFT" "Sullins"
 			(at 29.21 92.71 0)
 			(effects
@@
 					(unit 1)
 				)
+			)
+		)
+	)
+	(symbol
+		(lib_id "Liem:+5V_ISO")
+		(at 31.75 62.23 270)
+		(unit 1)
+		(exclude_from_sim no)
+		(in_bom yes)
+		(on_board yes)
+		(dnp no)
+		(property "Reference" "#PWR052"
+			(at 27.94 62.23 0)
+			(effects
+				(font
+					(size 1.27 1.27)
+				)
+				(hide yes)
+			)
+		)
+		(property "Value" "+5V_ISO"
+			(at 34.925 62.23 90)
+			(effects
+				(font
+					(size 1.27 1.27)
+					(bold yes)
+				)
+				(justify left)
+			)
+		)
+		(property "Footprint" ""
+			(at 31.75 62.23 0)
+			(effects
+				(font
+					(size 1.27 1.27)
+				)
+				(hide yes)
+			)
+		)
+		(property "Datasheet" ""
+			(at 31.75 62.23 0)
+			(effects
+				(font
+					(size 1.27 1.27)
+				)
+				(hide yes)
+			)
+		)
+		(property "Description" "Power symbol creates a global label with name \"+5V_ISO\""
+			(at 31.75 62.23 0)
+			(effects
+				(font
+					(size 1.27 1.27)
+				)
+				(hide yes)
+			)
+		)
+		(pin "1"
+		)
+		(instances
+			(project ""
+				(path "/20f80521-75f2-4ccc-bb34-c9566e70ef5c/34b63420-23a7-4d2d-affc-c07be2bf5f59"
+					(reference "#PWR052")
+					(unit 1)
+				)

Commit message: V1 schematic update 5
Parts:
- removed C32: 220uF/6.3V, SAMPI:CAP1411, symbol SAMPI:ELECCAP
- removed C54: 10uF, SAMPI:CAP0603, symbol SAMPI:CERCAP
- removed C75: 100uF/450V, SAMPI:CAP_ELEC-18.0x51.5-LS7.5, symbol SAMPI:ELECCAP
- removed FT1: 120R@100MHz, SAMPI:FT0603, symbol SAMPI:FerriteBead
- removed J1: HIGH VOLT, SAMPI:HDM1x10x2.54_TH_RA, symbol SAMPI:SIL10
- removed J2: LOW VOLT, SAMPI:HDM1x12x2.54_TH_RA, symbol SAMPI:SIL12
- added B1: 220V/50W, SAMPI:LAMP_6.35MM, symbol SAMPI:Lamp
- added BR1: 400V/10A, SAMPI:GBJ25xx, symbol SAMPI:BRIDGE
- added C32: 1uF/400V, SAMPI:ECWFE2W105, symbol SAMPI:CERCAP
- added C49, C53, C61, C64, C75: 100pF/2kV, SAMPI:CAP1206, symbol SAMPI:CERCAP
- added C50, C63, C65, C67, C69, C76, C77, C78, C84, C89, C92: 100nF, SAMPI:CAP0603, symbol SAMPI:CERCAP
- added C54, C90: 470uF/35V, SAMPI:CAP_ELEC-10.3x10.3-DIA10, symbol SAMPI:ELECCAP
- added C55, C72, C80, C81, C83, C88: 10uF, SAMPI:CAP0603, symbol SAMPI:CERCAP
- added C62, C70, C82: 10uF/35V, SAMPI:CAP0603, symbol SAMPI:CERCAP
- added C66, C85: 3.3nF, SAMPI:CAP0603, symbol SAMPI:CERCAP
- added C68: 47uF/35V, SAMPI:CAP_ELEC-6.6x6.6-DIA6.3, symbol SAMPI:ELECCAP
- added C71: 220uF/6.3V, SAMPI:CAP1411, symbol SAMPI:ELECCAP
- added C79: 100nF/400V, SAMPI:CAP_FILM_6.0x12.0x12.5-P10, symbol SAMPI:CERCAP
- added C86, C87: 22pF, SAMPI:CAP0603, symbol SAMPI:CERCAP
- added C91: 680uF/450V, SAMPI:ESMQ451VSN681MA50S, symbol SAMPI:ELECCAP
- added D18: 24V, SAMPI:DO-214AA, symbol SAMPI:DIODE-TVS
- added D22: 75V/150mA, SAMPI:SOD-323, symbol SAMPI:DIODE-REC
- added F1: 10A, SAMPI:01000056Z, symbol SAMPI:FUSE
- added FT1: 4.5mH/10A, SAMPI:ToroidCoil-3119-13-D1, symbol SAMPI:CK_Choke_2
- added FT4: 120R@100MHz, SAMPI:FT0603, symbol SAMPI:FerriteBead
- added G2: 300V, SAMPI:GDT1812_3532, symbol SAMPI:GDT
- added J1: AC POWER INPUT, SAMPI:TMB3_9.5, symbol SAMPI:SIL03
- added L1, L2, L4, L6, L7: 4.7uH/100mA, SAMPI:IND0805, symbol SAMPI:IND
- added L3: 22uH/1.5A, SAMPI:IND6045, symbol SAMPI:IND
- added L5: 68uH/1A, SAMPI:IND6045, symbol SAMPI:IND
- added M4, M5, M6, M7: 470V/1.2kA, SAMPI:MOV5MM, symbol SAMPI:MOV
- added MD1: 24V/10W, SAMPI:LD10-23BxxR2-RC, symbol SAMPI:AC-DC
- added MD3, MD4: DC-DC, SAMPI:B1524S-1WR3, symbol SAMPI:DC-DC
- added Q11: 20V/1A, SAMPI:SOT23, symbol SAMPI:FET_N-CH
- added R82, R86, R92: 100K, SAMPI:RES0603, symbol SAMPI:RES
- added R83, R84, R85, R88: 1M, SAMPI:RES1206, symbol SAMPI:RES
- added R87: 180K, 1%, SAMPI:RES0603, symbol SAMPI:RES
- added R89: 53.6K, 1%, SAMPI:RES0603, symbol SAMPI:RES
- added R90, R93: 10K, 1%, SAMPI:RES0603, symbol SAMPI:RES
- added R91: 10K, SAMPI:RES0603, symbol SAMPI:RES
- added RL2: 5V/30A, SAMPI:SLA-12VDC-SL-C, symbol SAMPI:RELAY-SPST-6P
- added U10: 5V/1.5A, SAMPI:TDFN8_2x3_MCHP, symbol SAMPI:MCP16311-TDFN
- added U13: LDO 3.3V/1.5A, SAMPI:DFN8_3x3_MCHP, symbol SAMPI:MCP1727
- added U14: 24V/1A, SAMPI:TDFN8_2x3_MCHP, symbol SAMPI:MCP16311-TDFN
- C1: value 1uF/400V -> 100nF/400V; footprint SAMPI:ECWFE2W105 -> SAMPI:CAP_FILM_6.0x12.0x12.5-P10; MFT Panasonic -> VISHAY; MNP ECW-FE2W105K -> BFC233824104; Unit Price 0.72 -> 1.5
- C56: value 3.3nF -> 100pF/2kV; footprint SAMPI:CAP0603 -> SAMPI:CAP1206; MFT Samsung -> WE; MNP CL10B332KB8NNNC -> 885342208022; Unit Price 0.031 -> 0.19
- C57: value 22pF -> 10uF; MFT Walsin -> Samsung; MNP 0603N220J500CT -> CL10A106MQ8NNNC; Unit Price 0.012 -> 0.079
- C58: value 22pF -> 100nF; MFT Walsin -> Samsung; MNP 0603N220J500CT -> CL10B104KB8NNNC; Unit Price 0.012 -> 0.0146
- C59: value 10uF -> 1uF/400V; footprint SAMPI:CAP0603 -> SAMPI:ECWFE2W105; MFT Samsung -> Panasonic; MNP CL10A106MQ8NNNC -> ECW-FE2W105K; Unit Price 0.079 -> 0.72
Connections:
- net +15V: now also C58.2, C85.2, C89.2, C90.+, L2.1, L5.2, R87.2
- net +24V_ISO: now also C67.2, C68.+, MD3.4 (DC+)
- net +3V3: now also C78.2, C81.2, C86.2, FT4.1, U13.7 (SEN/ADJ), U13.8 (VOUT); no longer C56.2, C57.2, FT3.1
- net +5V: now also C65.2, C66.2, C69.2, C71.+, C72.2, D22.K, L3.2, L4.1, R89.2, RL2.2 (COIL2), U13.1 (VIN1), U13.2 (VIN2), U13.3 (~{SHDN})
- net +5V_ISO: now also C76.2, C80.2, MD4.4 (DC+)
- net AGND: now also FT2.1, C87.1, C88.1; no longer C58.1, C59.1
- net AVDD: now also C87.2, C88.2, FT4.2; no longer C58.2, C59.2, FT3.2
- net CHASSIS: now also C56.2, C49.2, C53.2, C61.2, G2.1, J1.1
- net DEV_RELAY: now also R91.1
- net GND: now also C58.1, FT2.2, FT3.1, C50.1, C54.-, C55.1, C62.1, C64.1, C65.1, C69.1, C70.1, C71.-, C72.1, C75.1, C77.1, C78.1, C81.1, C82.1, C83.1, C86.1, C89.1, C90.-, C92.1, D18.1 (A1), MD1.4 (DC-), MD3.1 (VI-), MD4.1 (VI-), Q11.2 (S), R90.1, R92.2, R93.1, U10.5 (PGND), U10.8 (AGND), U10.9 (EP), U13.4 (GND), U13.9 (EP), U14.5 (PGND), U14.8 (AGND), U14.9 (EP); no longer C56.1, FT2.1
- net PGND: now also FT3.2, BR1.4 (DC-), C79.1, C91.-; no longer C1.1, FT2.2
- net VDC: now also BR1.1 (DC+), C79.2, C91.+; no longer C1.2
- new net: R83.1, R84.1, R85.1, R88.1
- new net: G2.2, M5.1, M6.1
- new net: C83.2, U14.2 (VCC)
- new net: C84.1, L5.1, U14.6 (SW)
- new net: C32.2, C53.1, F1.2, FT1.3, M4.2, M6.2
- new net: C84.2, U14.7 (BOOST)
- new net: C32.1, C49.1, FT1.1, J1.2, M4.1, M5.2
- new net: C77.2, U13.6 (CDELAY)
- new net: D22.A, Q11.3 (D), RL2.1 (COIL1)
- new net: B1.2, BR1.3 (AC2), RL2.6 (NO)
- new net: C55.2, L4.2, MD4.2 (VI+)
- new net: C62.2, L2.2, L7.2, MD3.2 (VI+)
- new net: C1.2, L1.2, MD1.2 (ACL)
- new net: C85.1, R87.1, R93.2, U14.1 (VFB)
- new net: C66.1, R89.1, R90.2, U10.1 (VFB)
- new net: C63.1, L3.1, U10.6 (SW)
- new net: C57.2, U10.2 (VCC)
- new net: R82.1, U10.3 (EN)
- new net: C63.2, U10.7 (BOOST)
- new net: F1.1, J1.3
- new net: R86.1, U14.3 (EN)
- new net: Q11.1 (G), R91.2, R92.1
- new net: C1.1, L6.2, MD1.1 (ACN)
- new net +24V: C50.2, C54.+, C70.2, C82.2, C92.2, D18.2 (A2), L7.1, MD1.5 (DC+), R82.2, R86.2, U10.4 (VIN), U14.4 (VIN)
- new net AC1: BR1.2 (AC1), C56.1, C59.2, FT1.4, L1.1, M7.2, R83.2, R84.2
- new net AC2: B1.1, C59.1, C61.1, FT1.2, L6.1, M7.1, R85.2, R88.2, RL2.3 (COM), RL2.4 (COM), RL2.5 (NC)
- new net GND1: C64.2, C67.1, C68.-, C75.2, C76.1, C80.1, MD3.3 (DC-), MD4.3 (DC-)
- no-connect marks 0 -> 1
Other:
- note added: "ISOLATED POWER - SAFE-ZONE"
- note removed: "SAFE-ZONE"

Commit message: V1 schematic update 6
Parts:
- removed L3: 22uH/1.5A, SAMPI:IND6045, symbol SAMPI:IND
- removed L6: 4.7uH/100mA, SAMPI:IND0805, symbol SAMPI:IND
- added C99: 10uF, SAMPI:CAP0603, symbol SAMPI:CERCAP
- added D19: 24V, SAMPI:SOD-80C_DO-213AC, symbol SAMPI:DIODE-ZEN
- added D20: 5.1V, Liem:SOD-123, symbol SAMPI:DIODE-ZEN
- added D21: 75V/150mA, SAMPI:SOD-323, symbol SAMPI:DIODE-REC
- added FT5: 10mH/500mA, SAMPI:IND-FL2D, symbol SAMPI:CK_Choke_2
- added Q10: 20V/1A, SAMPI:SOT23, symbol SAMPI:FET_N-CH
- added R94: 100K, SAMPI:RES0603, symbol SAMPI:RES
- added R95: 10K, SAMPI:RES0603, symbol SAMPI:RES
- added RL1: 5V/30A, SAMPI:SLA-12VDC-SL-C, symbol SAMPI:RELAY-SPST-6P
- added U17: LDO 5V±0.4%/250mA, SAMPI:SOT-89, symbol SAMPI:MCP1702
- B1: Checked OK -> (none)
- BR1: Checked OK -> (none); Unit Price 1.32 -> (none)
- C1, C79: Checked OK -> (none); Unit Price 1.5 -> (none)
- C32, C59: Checked OK -> (none); Unit Price 0.72 -> (none)
- C49, C53, C56, C61, C64, C75: Checked OK -> (none); Unit Price 0.19 -> (none)
- C50, C58, C63, C65, C67, C69, C76, C77, C78, C84, C89: Checked OK -> (none); Unit Price 0.0146 -> (none)
- C54, C90: Checked OK -> (none); Unit Price 0.85 -> (none)
- C55, C57, C62, C70, C72, C80, C81, C82, C83, C88: Checked OK -> (none); Unit Price 0.079 -> (none)
- C66, C85: Checked OK -> (none); Unit Price 0.031 -> (none)
- C68: Checked OK -> (none); Unit Price 0.45 -> (none)
- C71: Checked OK -> (none); Unit Price 1.01 -> (none)
- C86, C87: Checked OK -> (none); Unit Price 0.012 -> (none)
- C91: Checked OK -> (none); Unit Price 6.96 -> (none)
- C92: Checked OK -> (none); Unit Price 0.0146 -> (none); now fitted
- D22: Checked OK -> (none); Unit Price 0.068 -> (none)
- F1: Checked OK -> (none); Comment x2 pcs -> (none); Unit Price 0.41 -> (none)
- FT1: value 4.5mH/10A -> 5mH/2.5A; Checked OK -> (none); Unit Price 4 -> (none)
- FT2, FT3, FT4: Checked OK -> (none); Unit Price 0.058 -> (none)
- G2: Checked OK -> (none); Unit Price 0.53 -> (none)
- J1: Checked OK -> (none); Unit Price 0.84 -> (none)
- L1: value 4.7uH/100mA -> 22uH/1A; footprint SAMPI:IND0805 -> SAMPI:IND-8D43-8045; Checked OK -> (none); MFT Eaton -> Bourns Inc.; MNP MCL2012V1-4R7-R -> SRU8043-220Y; Unit Price 0.092 -> (none)
- L2, L4, L7: value 4.7uH/100mA -> 4.7uH/670mA; footprint SAMPI:IND0805 -> SAMPI:IND-R5-2MM-TH; Checked OK -> (none); MFT Eaton -> Bourns Inc.; MNP MCL2012V1-4R7-R -> RLB0608-4R7ML; Unit Price 0.092 -> (none)
- L5: footprint SAMPI:IND6045 -> SAMPI:IND-8D43-8045; Checked OK -> (none); MFT TAI-TECH -> Bourns Inc.; MNP HPC 6045NV-220M -> SRU8043-680Y; Unit Price 0.26 -> (none)
- M4, M5, M6, M7: Checked OK -> (none); Unit Price 0.255 -> (none)
- MD1: value 24V/10W -> AC-DC 24V±2%/10W
- MD3: value DC-DC -> DC-DC 15V/24V-24V/42mA; Checked OK -> (none)
- MD4: value DC-DC -> DC-DC 5V-5V/200mA; Checked OK -> (none)
- Q11: Checked OK -> (none); Unit Price 0.148 -> (none)
- R82, R86, R87, R90, R91, R92, R93: Checked OK -> (none); Unit Price 0.019 -> (none)
- R83, R84, R85, R88: Checked OK -> (none); Unit Price 0.02 -> (none)
- R89: value 53.6K, 1% -> 63.4K, 1%; Checked OK -> (none); Unit Price 0.019 -> (none)
- RL2: Checked OK -> (none); Unit Price 0.8565 -> (none)
- U10: value 5V/1.5A -> SMPS 5V±2%/1.5A; Checked OK -> (none); Comment Vo=5.088V±2%/1.5A -> (none); Unit Price 1.8 -> (none)
- U13: value LDO 3.3V/1.5A -> LDO 3.3V±0.5%/1A; Checked OK -> (none); Comment Vo=3.3V±0.5%/1.5A -> (none); Unit Price 1.11 -> (none)
- U14: value 24V/1A -> SMPS 24V±2%/1A; Checked OK -> (none); Comment Vo=5.088V±2%/1.5A -> (none); Unit Price 1.8 -> (none)
Connections:
- net +24V_ISO: now also D19.K
- net +5V: now also C99.2, U17.3 (VOUT); no longer C66.2, C69.2, C71.+, C72.2, D22.K, R89.2, RL2.2 (COIL2), U13.1 (VIN1), U13.2 (VIN2), U13.3 (~{SHDN})
- net +5V_ISO: now also D20.K
- net AC1: now also FT5.3; no longer L1.1
- net AC2: now also FT5.1; no longer B1.1
- net DEV_RELAY: now also R95.1; no longer R91.1
- net GND: now also C99.1, Q10.2 (S), R94.2, U17.1 (GND)
- net GND1: now also D19.A, D20.A
- net at B1.2, BR1.3 (AC2): now also RL1.6 (NO); no longer RL2.6 (NO)
- net at C1.2, MD1.2 (ACL): now also FT5.4; no longer L1.2
- net at C63.1, U10.6 (SW): now also L1.1
- net at C1.1, MD1.1 (ACN): now also FT5.2
- new net: D21.A, Q10.3 (D), RL1.1 (COIL1)
- new net: Q10.1 (G), R94.1, R95.2
- new net: B1.1, RL1.3 (COM), RL1.4 (COM), RL1.5 (NC), RL2.6 (NO)
- new net +6V: C66.2, C69.2, C71.+, C72.2, D21.K, D22.K, L1.2, R89.2, RL1.2 (COIL2), RL2.2 (COIL2), U13.1 (VIN1), U13.2 (VIN2), U13.3 (~{SHDN}), U17.2 (VIN)
- new net PWR_RELAY: R91.1
Other:
- note added: "For DC-DC 15-24V option: mount L2, unmount L7 For DC-DC 24-24V option: mount L7, unmount L2"
- moved on the sheet: B1, BR1, C55, C58, C62, C64, C65, C67, C68, C75, C76, C78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
