File: V1/Design/HW.ACIM-INV/Power.kicad_sch (KiCad schematic)
At the start: 98 parts, among them J1 AC POWER INPUT, J2 FAN, M4 470V/1.2kA, M5 470V/1.2kA, M6 470V/1.2kA, M7 470V/1.2kA, Q10 20V/1A, Q11 20V/1A, U10 SMPS 12V±2%/0.8A, U13 LDO 3.3V±0.5%/1A, U14 SMPS 15V±2%/0.6A, U17 LDO 5V±0.4%/250mA, U2 LDO 3.3V 250mV, U20 SMPS 5V±2%/1.2A

Commit message: V1 schematic update 12
Parts:
- MD1: value AC-DC 24V±2%/10W -> 24V±2%/10W
Changed lines of the file:
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@@
 			)
 		)
-		(property "Value" "AC-DC 24V±2%/10W"
-			(at 189.23 75.565 0)
+		(property "Value" "24V±2%/10W"
+			(at 182.245 75.565 0)
 			(effects
 				(font
