File: V1/Design/HW.ACIM-INV/VI_Measurement.kicad_sch (KiCad schematic)
At the start: 59 parts, among them Q1 20V/1A, U12 OP-1CH, U15 OP-1CH, U16 OP-1CH, U2 OP-1CH, U4 CMP-1CH

Commit message: V1 schematic update 2
Parts:
- removed C37: 1nF, SAMPI:CAP0603, symbol SAMPI:CERCAP
- removed C38, C39, C40, C41: 100nF, SAMPI:CAP0603, symbol SAMPI:CERCAP
- removed D1, D4: GP DIODE, SAMPI:SOT23, symbol SAMPI:DIODE_ARR2
- removed R4, R48, R49, R51: 100K, SAMPI:RES0603, symbol SAMPI:RES
- removed R5, R52: 10R, SAMPI:RES0603, symbol SAMPI:RES
- removed R50, R53, R6: 1.1K, SAMPI:RES0603, symbol SAMPI:RES
- removed U15, U16: OP-1CH, SAMPI:SOT353, symbol SAMPI:OPAMP-1CH
- added C18, C30: 1nF, SAMPI:CAP0603, symbol SAMPI:CERCAP
- added C29: 100nF, SAMPI:CAP0603, symbol SAMPI:CERCAP
- added D1, D5: GP DIODE, SAMPI:SOT23, symbol SAMPI:DIODE_ARR1
- added R40, R41, R42: 10R, SAMPI:RES0603, symbol SAMPI:RES
- added U3, U5: ISEN 50mV/V, SAMPI:SOT363, symbol SAMPI:ZXCT199Q
- C10: value 100nF -> 1nF; MNP CL10B104KB8NNNC -> CL10B102KB8NNNC; Unit Price 0.0146 -> 0.027
- R1, R2: value 100K -> 10R; MNP RC0603FR-07100KL -> RC0603FR-0710RL; Unit Price 0.019 -> 0.029
- R3: value 1.1K -> 10R; MNP AC0603FR-071K1L -> RC0603FR-0710RL; Unit Price 0.021 -> 0.029
Connections:
- net VDC is gone; now on an unnamed net: R1.1
- net VREF is gone; now on net AVDD: R28.2
- net AGND: now also C10.1, C9.1, C29.1, C30.1, U3.1 (REF), U3.2 (GND), U5.1 (REF), U5.2 (GND); no longer C10.2, C9.2
- net at C8.1: now also R2.1, D1.3 (COM), U5.5 (IN-); no longer R3.1
- net MC_IU_SEN_N: now reaches R2.2
- net at C8.2: now also D1.1 (A1), D1.2 (K2), U5.4 (IN+)
- net MC_IU_SEN_P: now reaches R1.2
- net MC_IU_SEN_P: no longer R2.1
- net INV_FLT_OC renamed MC_PWM_FLT
- net MC_IDC_SENSE renamed MC_IDC_SEN
- net MC_VDC_SENSE renamed MC_IV_SEN
- net MC_IV_SEN: now also C10.2, C30.2, R42.2; no longer C9.1
- net MC_VU_SENSE renamed MC_VU_DIV
- net MC_VV_SENSE renamed MC_VV_DIV
- net ~{INV_FLT_OC} renamed ~{MC_PWM_FLT}
- new net: C18.1, D5.3 (COM), R41.1, U3.5 (IN-)
- new net: R42.1, U3.6 (OUT)
- new net: C18.2, D5.1 (A1), D5.2 (K2), R40.1, U3.4 (IN+)
- new net: R3.1, U5.6 (OUT)
- new net +5V: C29.2, C9.2, U3.3 (V+), U5.3 (V+)
- new net MC_IV_SEN_N: R41.2
- new net MC_IV_SEN_P: R40.2
Other:
- note added: "VOUT=(ILoad*RSen)*Gain+Vref Gain=50, Vref=0, RSen=5mR, Imax=13A, Vout=3.25V"
- note removed: "VDC=(VDC_SENSE/1.1K)*(3*100K+1.1K) =VDC_SENSE*3011/11"
- moved on the sheet: C19, C20, C21, C22, C23, C24, C25, C26, C27, C28, C42, D2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

Commit message: V1 schematic update 3
Parts:
- added C37, C39, C43, C47: 1nF, SAMPI:CAP0603, symbol SAMPI:CERCAP
- added C38, C40, C41, C44, C45, C46, C48: 100nF, SAMPI:CAP0603, symbol SAMPI:CERCAP
- added D16, D17: GP DIODE, SAMPI:SOT23, symbol SAMPI:DIODE_ARR2
- added D9: GP DIODE, SAMPI:SOT23, symbol SAMPI:DIODE_ARR1
- added R50, R51, R52, R59, R78: 10R, SAMPI:RES0603, symbol SAMPI:RES
- added R53, R56, R57, R62, R67, R73: 100K, SAMPI:RES0603, symbol SAMPI:RES
- added R58, R60, R77, R79: 1.1K, SAMPI:RES0603, symbol SAMPI:RES
- added U6: ISEN 50mV/V, SAMPI:SOT363, symbol SAMPI:ZXCT199Q
- added U7, U8: OP-1CH, SAMPI:SOT353, symbol SAMPI:OPAMP-1CH
Connections:
- net +5V: now also C38.2, U6.3 (V+)
- net AGND: now also C38.1, C39.1, C40.2, C41.1, C44.2, C45.2, C46.1, C48.2, D16.1 (A1), D17.1 (A1), R58.2, R77.2, U6.1 (REF), U6.2 (GND), U7.2 (VSS), U8.2 (VSS)
- net AVDD: now also C41.2, C46.2, D16.2 (K2), D17.2 (K2), U7.5 (VDD), U8.5 (VDD)
- net MC_IDC_SEN: now also C39.2, R52.2
- net MC_IV_SEN: no longer C10.2, R3.2
- net MC_VU renamed MC_UU
- net MC_VU_DIV renamed MC_UU_DIV
- net MC_VV renamed MC_UV
- net MC_VV_DIV renamed MC_UV_DIV
- new net: R56.2, R57.1
- new net: C40.1, D16.3 (COM), R57.2, R58.1, U7.3 (VIN+)
- new net: C43.1, R60.1, U7.4 (VIN-)
- new net: C43.2, R59.2, U7.1 (VOUT)
- new net: C37.1, D9.3 (COM), R51.1, U6.5 (IN-)
- new net: R53.2, R56.1
- new net: C45.1, D17.3 (COM), R73.2, R77.1, U8.3 (VIN+)
- new net: C47.2, R78.2, U8.1 (VOUT)
- new net: C47.1, R79.1, U8.4 (VIN-)
- new net: C37.2, D9.1 (A1), D9.2 (K2), R50.1, U6.4 (IN+)
- new net: R67.2, R73.1
- new net: R62.2, R67.1
- new net: R52.1, U6.6 (OUT)
- new net MC_IDC_SEN_N: R51.2
- new net MC_IDC_SEN_P: R50.2
- new net MC_IU_SEN: C10.2, R3.2
- new net MC_UDC_DIV: C48.1, R78.1, R79.2
- new net MC_UW: R53.1
- new net MC_UW_DIV: C44.1, R59.1, R60.2
- new net VDC: R62.1
Other:
- moved on the sheet: C10, C18, C19, C20, C21, C22, C23, C24, C25, C26, C27, C28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

Commit message: V1 schematic update 5
Other:
- moved on the sheet: C25, C26, C27, C28, D3, R34, R35, R36, R37, R38, R39, U12

Commit message: V1 schematic update 6
Parts:
- added C100, C101, C102, C103, C105, C106, C98: 1nF, SAMPI:CAP0603, symbol SAMPI:CERCAP
- added C104, C95: 100nF, SAMPI:CAP0603, symbol SAMPI:CERCAP
- added R100, R80: 10R, SAMPI:RES0603, symbol SAMPI:RES
- added R101, R81: 1.1K, SAMPI:RES0603, symbol SAMPI:RES
- added R102: 10K, SAMPI:RES0603, symbol SAMPI:RES
- added R96, R97, R98, R99: 100K, SAMPI:RES0603, symbol SAMPI:RES
- added U18, U19: OP-1CH, SAMPI:SOT353, symbol SAMPI:NCV21871SQ3T2G
- C10, C18, C19, C21, C25, C30, C37, C39, C43, C47, C8: Checked OK -> (none); Unit Price 0.027 -> (none)
- C20, C22, C23, C24, C26, C27, C28, C29, C38, C40, C41, C42, C44, C45, C46, C48, C9: Checked OK -> (none); Unit Price 0.0146 -> (none)
- D1, D16, D17, D2, D3, D5, D9: Checked OK -> (none); Unit Price 0.11 -> (none)
- Q1: Checked OK -> (none); Unit Price 0.148 -> (none)
- R1, R2, R27, R32, R38, R40, R41, R50, R51, R52, R59, R78: Checked OK -> (none); Unit Price 0.029 -> (none)
- R10, R29, R33, R36, R39, R58, R60, R77, R79: Checked OK -> (none); Unit Price 0.021 -> (none)
- R26, R28, R31, R34, R35, R37, R53, R54, R56, R57, R62, R67, R73, R8, R9: Checked OK -> (none); Unit Price 0.019 -> (none)
- R3, R42: value 10R -> 5.2K; Checked OK -> (none); Unit Price 0.029 -> (none)
- R30: Checked OK -> (none); Unit Price 0.02 -> (none)
- U12, U2, U7, U8: symbol SAMPI:OPAMP-1CH -> SAMPI:NCV21871SQ3T2G; Checked OK -> (none); Unit Price 0.633 -> (none)
- U3, U5, U6: Checked OK -> (none); Unit Price 0.079 -> (none)
- U4: Checked OK -> (none); Unit Price 0.36 -> (none)
Connections:
- net +3V3: now also R102.1
- net AGND: now also C102.1, C103.1, C104.1, C106.1, C95.1, C98.1, R96.2, R99.2, U18.2 (VSS), U19.2 (VSS); no longer C29.1, C38.1, C9.1, U3.1 (REF), U3.2 (GND), U5.1 (REF), U5.2 (GND), U6.1 (REF), U6.2 (GND)
- net AVDD: now also C104.2, C95.2, U18.5 (VDD), U19.5 (VDD)
- net GND: now also C29.1, C38.1, C9.1, U3.1 (REF), U3.2 (GND), U5.1 (REF), U5.2 (GND), U6.1 (REF), U6.2 (GND), C100.1
- net MC_IU_SEN: now also C98.2; no longer C10.2
- net at C40.1, D16.3 (COM), R57.2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: now also U7.1 (IN+); no longer U7.3 (VIN+)
- net at C25.1, R36.1: now also U12.3 (IN-); no longer U12.4 (VIN-)
- net at C25.2, R38.2: now also U12.4 (OUT); no longer U12.1 (VOUT)
- net at C43.1, R60.1: now also U7.3 (IN-); no longer U7.4 (VIN-)
- net at C43.2, R59.2: now also U7.4 (OUT); no longer U7.1 (VOUT)
- net at C28.1, D3.3 (COM), R37.2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: now also U12.1 (IN+); no longer U12.3 (VIN+)
- net at C45.1, D17.3 (COM), R73.2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: now also U8.1 (IN+); no longer U8.3 (VIN+)
- net at C47.2, R78.2: now also U8.4 (OUT); no longer U8.1 (VOUT)
- net at C47.1, R79.1: now also U8.3 (IN-); no longer U8.4 (VIN-)
- net at C23.1, D2.3 (COM), R26.2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: now also U2.1 (IN+); no longer U2.3 (VIN+)
- net at R27.1, R30.1, U4.4 (VOUT): now also R102.2
- net at C19.2, R32.2: now also U2.4 (OUT); no longer U2.1 (VOUT)
- net at C19.1, R10.1: now also U2.3 (IN-); no longer U2.4 (VIN-)
- net at R52.1, U6.6 (OUT): now also C100.2
- new net: C105.2, R100.2, U19.4 (OUT)
- new net: C103.2, R98.2, R99.1, U19.1 (IN+)
- new net: C105.1, R101.1, U19.3 (IN-)
- new net: C101.2, R80.2, U18.4 (OUT)
- new net: C102.2, R96.1, R97.2, U18.1 (IN+)
- new net: C101.1, R81.1, U18.3 (IN-)
- new net MC_ALT_IU_SEN: C10.2, R80.1, R81.2
- new net MC_ALT_IV_SEN: C106.2, R100.1, R101.2
- new net MC_IU_HAL: R97.1
- new net MC_IV_HAL: R98.1
Other:
- moved on the sheet: C18, C19, C20, C24, C25, C26, C27, C29, C30, C39, C41, C43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

Commit message: V1 schematic update 7
Connections:
- net +5V renamed VREF
Changed lines of the file:
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@@
 	)
 	(symbol
+		(lib_id "SAMPI:VREF")
+		(at 52.07 59.69 90)
+		(unit 1)
+		(exclude_from_sim no)
+		(in_bom yes)
+		(on_board yes)
+		(dnp no)
+		(property "Reference" "#PWR076"
+			(at 55.88 59.69 0)
+			(effects
+				(font
+					(size 1.27 1.27)
+				)
+				(hide yes)
+			)
+		)
+		(property "Value" "VREF"
+			(at 46.99 59.69 90)
+			(effects
+				(font
+					(size 1.27 1.27)
+					(bold yes)
+				)
+			)
+		)
+		(property "Footprint" ""
+			(at 52.07 59.69 0)
+			(effects
+				(font
+					(size 1.27 1.27)
+				)
+				(hide yes)
+			)
+		)
+		(property "Datasheet" ""
+			(at 52.07 59.69 0)
+			(effects
+				(font
+					(size 1.27 1.27)
+				)
+				(hide yes)
+			)
+		)
+		(property "Description" "Power symbol creates a global label with name \"VREF\""
+			(at 52.07 59.69 0)
+			(effects
+				(font
+					(size 1.27 1.27)
+				)
+				(hide yes)
+			)
+		)
+		(pin "1"
+		)
+		(instances
+			(project "HW.ACIM-INV"
+				(path "/20f80521-75f2-4ccc-bb34-c9566e70ef5c/7de2aa19-8f84-4f41-81e1-8fc4a5d38687"
+					(reference "#PWR076")
+					(unit 1)
+				)
+			)
+		)
+	)
+	(symbol
 		(lib_id "SAMPI:RES")
 		(at 209.55 101.6 90)
@@
 	)
 	(symbol
+		(lib_id "SAMPI:VREF")
+		(at 168.91 142.875 90)
+		(unit 1)
+		(exclude_from_sim no)
+		(in_bom yes)
+		(on_board yes)
+		(dnp no)
+		(property "Reference" "#PWR025"
+			(at 172.72 142.875 0)
+			(effects
+				(font
+					(size 1.27 1.27)
+				)
+				(hide yes)
+			)
+		)
+		(property "Value" "VREF"
+			(at 163.83 142.875 90)
+			(effects
+				(font
+					(size 1.27 1.27)
+					(bold yes)
+				)
+			)
+		)
+		(property "Footprint" ""
+			(at 168.91 142.875 0)
+			(effects
+				(font
+					(size 1.27 1.27)
+				)
+				(hide yes)
+			)
+		)
+		(property "Datasheet" ""
+			(at 168.91 142.875 0)
+			(effects
+				(font
+					(size 1.27 1.27)
+				)
+				(hide yes)
+			)
+		)
+		(property "Description" "Power symbol creates a global label with name \"VREF\""
+			(at 168.91 142.875 0)
+			(effects
+				(font
+					(size 1.27 1.27)
+				)
+				(hide yes)
+			)
+		)
+		(pin "1"
+		)
+		(instances
+			(project "HW.ACIM-INV"
+				(path "/20f80521-75f2-4ccc-bb34-c9566e70ef5c/7de2aa19-8f84-4f41-81e1-8fc4a5d38687"
+					(reference "#PWR025")
+					(unit 1)
+				)
+			)
+		)
+	)
+	(symbol
 		(lib_id "SAMPI:CERCAP")
 		(at 38.735 187.96 270)
@@
 	)
 	(symbol
-		(lib_id "power:+5V")
-		(at 168.91 142.875 90)
-		(unit 1)
-		(exclude_from_sim no)
-		(in_bom yes)
-		(on_board yes)
-		(dnp no)
-		(property "Reference" "#PWR025"
-			(at 172.72 142.875 0)
-			(effects
-				(font
-					(size 1.27 1.27)
-				)
-				(hide yes)
-			)
-		)
-		(property "Value" "+5V"
-			(at 163.83 142.875 90)
-			(effects
-				(font
-					(size 1.27 1.27)
-					(bold yes)
-				)
-			)
-		)
-		(property "Footprint" ""
-			(at 168.91 142.875 0)
-			(effects
-				(font
-					(size 1.27 1.27)
-				)
-				(hide yes)
-			)
-		)
-		(property "Datasheet" ""
-			(at 168.91 142.875 0)
-			(effects
-				(font
-					(size 1.27 1.27)
-				)
-				(hide yes)
-			)
-		)
-		(property "Description" ""
-			(at 168.91 142.875 0)
-			(effects
-				(font
-					(size 1.27 1.27)
-				)
-				(hide yes)
-			)
-		)
-		(pin "1"
-		)
-		(instances
-			(project "HW.ACIM-INV"
-				(path "/20f80521-75f2-4ccc-bb34-c9566e70ef5c/7de2aa19-8f84-4f41-81e1-8fc4a5d38687"
-					(reference "#PWR025")
-					(unit 1)
-				)
-			)
-		)
-	)
-	(symbol
 		(lib_id "SAMPI:AGND")
 		(at 210.82 139.065 0)
@@
 	)
 	(symbol
+		(lib_id "SAMPI:VREF")
+		(at 52.07 142.24 90)
+		(unit 1)
+		(exclude_from_sim no)
+		(in_bom yes)
+		(on_board yes)
+		(dnp no)
+		(property "Reference" "#PWR032"
+			(at 55.88 142.24 0)
+			(effects
+				(font
+					(size 1.27 1.27)
+				)
+				(hide yes)
+			)
+		)
+		(property "Value" "VREF"
+			(at 46.99 142.24 90)
+			(effects
+				(font
+					(size 1.27 1.27)
+					(bold yes)
+				)
+			)
+		)
+		(property "Footprint" ""
+			(at 52.07 142.24 0)
+			(effects
+				(font
+					(size 1.27 1.27)
+				)
+				(hide yes)
+			)
+		)
+		(property "Datasheet" ""
+			(at 52.07 142.24 0)
+			(effects
+				(font
+					(size 1.27 1.27)
+				)
+				(hide yes)
+			)
+		)
+		(property "Description" "Power symbol creates a global label with name \"VREF\""
+			(at 52.07 142.24 0)
+			(effects
+				(font
+					(size 1.27 1.27)
+				)
+				(hide yes)
+			)
+		)
+		(pin "1"
+		)
+		(instances
+			(project "HW.ACIM-INV"
+				(path "/20f80521-75f2-4ccc-bb34-c9566e70ef5c/7de2aa19-8f84-4f41-81e1-8fc4a5d38687"
+					(reference "#PWR032")
+					(unit 1)
+				)
+			)
+		)
+	)
+	(symbol
 		(lib_id "power:GND")
 		(at 53.34 68.58 0)
@@
 	)
 	(symbol
-		(lib_id "power:+5V")
-		(at 52.07 59.69 90)
-		(unit 1)
-		(exclude_from_sim no)
-		(in_bom yes)
-		(on_board yes)
-		(dnp no)
-		(property "Reference" "#PWR076"
-			(at 55.88 59.69 0)
-			(effects
-				(font
-					(size 1.27 1.27)
-				)
-				(hide yes)
-			)
-		)
-		(property "Value" "+5V"
-			(at 46.99 59.69 90)
-			(effects
-				(font
-					(size 1.27 1.27)
-					(bold yes)
-				)
-			)
-		)
-		(property "Footprint" ""
-			(at 52.07 59.69 0)
-			(effects
-				(font
-					(size 1.27 1.27)
-				)
-				(hide yes)
-			)
-		)
-		(property "Datasheet" ""
-			(at 52.07 59.69 0)
-			(effects
-				(font
-					(size 1.27 1.27)
-				)
-				(hide yes)
-			)
-		)
-		(property "Description" ""
-			(at 52.07 59.69 0)
-			(effects
-				(font
-					(size 1.27 1.27)
-				)
-				(hide yes)
-			)
-		)
-		(pin "1"
-		)
-		(instances
-			(project "HW.ACIM-INV"
-				(path "/20f80521-75f2-4ccc-bb34-c9566e70ef5c/7de2aa19-8f84-4f41-81e1-8fc4a5d38687"
-					(reference "#PWR076")
-					(unit 1)
-				)
-			)
-		)
-	)
-	(symbol
 		(lib_id "SAMPI:AVDD")
 		(at 203.2 54.61 0)
@@
 					(unit 1)
 				)
-			)
-		)
-	)
-	(symbol
-		(lib_id "power:+5V")
-		(at 52.07 142.24 90)
-		(unit 1)
-		(exclude_from_sim no)
-		(in_bom yes)
-		(on_board yes)
-		(dnp no)
-		(property "Reference" "#PWR032"
-			(at 55.88 142.24 0)
-			(effects
-				(font
-					(size 1.27 1.27)
-				)
-				(hide yes)
-			)
-		)
-		(property "Value" "+5V"
-			(at 46.99 142.24 90)
-			(effects
-				(font
-					(size 1.27 1.27)
-					(bold yes)
-				)
-			)
-		)
-		(property "Footprint" ""
-			(at 52.07 142.24 0)
-			(effects
-				(font
-					(size 1.27 1.27)
-				)
-				(hide yes)
-			)
-		)
-		(property "Datasheet" ""
-			(at 52.07 142.24 0)
-			(effects
-				(font
-					(size 1.27 1.27)
-				)
-				(hide yes)
-			)
-		)
-		(property "Description" ""
-			(at 52.07 142.24 0)
-			(effects
-				(font
-					(size 1.27 1.27)
-				)
-				(hide yes)
-			)
-		)
-		(pin "1"
-		)
-		(instances
-			(project "HW.ACIM-INV"
-				(path "/20f80521-75f2-4ccc-bb34-c9566e70ef5c/7de2aa19-8f84-4f41-81e1-8fc4a5d38687"
-					(reference "#PWR032")
-					(unit 1)
-				)

Commit message: V1 schematic update 8
Parts:
- removed C101, C105, C19, C25, C43, C47: 1nF, SAMPI:CAP0603, symbol SAMPI:CERCAP
- removed R101, R36, R60, R79, R81: 1.1K, SAMPI:RES0603, symbol SAMPI:RES
Connections:
- net MC_IDC_SEN: now also R10.2; no longer U4.1 (VIN-)
- net MC_UU_DIV: no longer R10.2
- net at U12.3 (IN-): now also R38.2, U12.4 (OUT)
- net at U7.3 (IN-): now also R59.2, U7.4 (OUT)
- net at R100.2, U19.4 (OUT): now also U19.3 (IN-)
- net at U8.3 (IN-): now also R78.2, U8.4 (OUT)
- net at R80.2, U18.4 (OUT): now also U18.3 (IN-)
- net at U2.3 (IN-): now also R32.2, U2.4 (OUT); no longer R10.1
- new net: R10.1, U4.1 (VIN-)

Commit message: V1 schematic update 11
Parts:
- removed C18, C30, C8, C98: 1nF, SAMPI:CAP0603, symbol SAMPI:CERCAP
- removed C20, C23, C24, C26, C27, C28, C29, C40, C41, C44, C9: 100nF, SAMPI:CAP0603, symbol SAMPI:CERCAP
- removed D1, D5: GP DIODE, SAMPI:SOT23, symbol SAMPI:DIODE_ARR1
- removed D16, D2, D3: GP DIODE, SAMPI:SOT23, symbol SAMPI:DIODE_ARR2
- removed R1, R2, R32, R38, R40, R41, R59: 10R, SAMPI:RES0603, symbol SAMPI:RES
- removed R26, R28, R34, R35, R37, R53, R56, R57, R8, R9: 100K, SAMPI:RES0603, symbol SAMPI:RES
- removed R3, R42: 5.2K, SAMPI:RES0603, symbol SAMPI:RES
- removed R31: 470K, SAMPI:RES0603, symbol SAMPI:RES
- removed R33, R39, R58: 1.1K, SAMPI:RES0603, symbol SAMPI:RES
- removed R54: 10K, SAMPI:RES0603, symbol SAMPI:RES
- removed U12, U2, U7: OP-1CH, SAMPI:SOT353, symbol SAMPI:NCV21871SQ3T2G
- removed U3, U5: ISEN 50mV/V, SAMPI:SOT363, symbol SAMPI:ZXCT199Q
- added OP1: OPTO-BJT-1CH, SAMPI:OPTO_SO4_7.6MM, symbol SAMPI:OPTO-BJT-1CH
- added RV2: 100K, SAMPI:TC33X-2, symbol SAMPI:POT
Connections:
- net MC_ALT_IU_SEN is gone; now on net MC_IU_SEN: C10.2, R80.1
- net MC_ALT_IV_SEN is gone; now on net MC_IV_SEN: C106.2, R100.1
- net VREF is gone; now on net +3V3_ISO: C38.2, U6.3 (V+)
- net AGND: no longer C22.1, C39.1, C42.1, U4.2 (VSS)
- net AVDD: no longer C42.2, U4.5 (VDD)
- net MC_PWM_FLT: no longer Q1.3 (D)
- net at R102.2, R27.1, U4.4 (VOUT): now also R30.2; no longer R30.1
- net at R29.1, U4.3 (VIN+): now also R30.1; no longer R30.2
- net at C22.2, R29.2: now also RV2.2 (WIPER)
- net +3V3 renamed +3V3_ISO
- net +3V3_ISO: now also C42.2, U4.5 (VDD), RV2.1 (CCW)
- net GND renamed GND_ISO
- net GND_ISO: now also C22.1, C39.1, C42.1, U4.2 (VSS), RV2.3 (CW)
Other:
- moved on the sheet: C10, C102, C103, C104, C106, C21, C22, C42, C95, Q1, R10, R100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

Commit message: V1 schematic update 12
Parts:
- added R1: 1.1K, SAMPI:RES0603, symbol SAMPI:RES
- added R2: 10K, SAMPI:RES0603, symbol SAMPI:RES
- added U7: ISO OPAMP 1-CH, symbol SAMPI:ISO-OPAMP
Connections:
- net +3V3_ISO: now also C46.2, D17.2 (K2), U8.5 (VDD), R1.1
- net AGND: no longer C45.2, C46.1, C48.2, D17.1 (A1), R77.2, U8.2 (VSS)
- net AVDD: no longer C46.2, D17.2 (K2), U8.5 (VDD)
- net GND_ISO: now also C45.2, C46.1, C48.2, D17.1 (A1), R77.2, U8.2 (VSS), U7.4 (GND1)
- net MC_PWM_FLT: now also C21.2, Q1.1 (G), R27.2
- net ~{MC_PWM_FLT}: now also OP1.4 (C), R2.2; no longer C21.2, Q1.1 (G), R27.2
- net at R29.2, RV2.2 (WIPER): no longer C22.2
- net at R102.2, R27.1, U4.4 (VOUT): now also R30.1; no longer R30.2
- net at OP1.1 (A): now also R1.2
- net at OP1.2 (K): now also Q1.3 (D)
- net GND: now reaches OP1.3 (E)
- net GND: now also U7.5 (GND2)
- net at R10.1: now also R30.2, U4.3 (VIN+); no longer U4.1 (VIN-)
- net MC_UDC_DIV renamed MC_VDC_DIV
- new net: C22.2, R29.1, U4.1 (VIN-)
- new net +3V3: R2.1
Other:
- moved on the sheet: C10, C102, C103, C104, C106, C21, C22, C42, C45, C46, C48, C95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
