File: V1/Design/HW.ACIM-INV/Inverter.kicad_sch (KiCad schematic)
At the start: 70 parts, among them J3 MOTOR, M1 560V/1.75kA, M2 560V/1.75kA, M3 560V/1.75kA, Q4 20V/1A, Q5 20V/1A, Q6 20V/1A, U1 IPM 600V/15A, U10 I=±10A, U3 ISEN 50mV/V, U7 I=±10A, U9 I=±10A

Commit message: V1 schematic update 2
Parts:
- removed C18, C29, C30, C62, C64, C65, C67, C68: 1nF, SAMPI:CAP0603, symbol SAMPI:CERCAP
- removed C31, C61, C63, C66: 100nF, SAMPI:CAP0603, symbol SAMPI:CERCAP
- removed D20: GP DIODE, SAMPI:SOT23, symbol SAMPI:DIODE_ARR1
- removed R40, R41, R42: 10R, SAMPI:RES0603, symbol SAMPI:RES
- removed U10, U7, U9: I=±10A, SAMPI:SOIC8_ALL, symbol SAMPI:ACS724
- removed U3: ISEN 50mV/V, SAMPI:SOT363, symbol SAMPI:ZXCT199Q
- added R75: 100K, SAMPI:RES0603, symbol SAMPI:RES
- added R76: 10mR/3W/1%, SAMPI:SHU2512, symbol SAMPI:SHUNT
- C15: value 1nF -> 22pF; MFT Samsung -> Walsin; MNP CL10B102KB8NNNC -> 0603N220J500CT; Unit Price 0.027 -> 0.012
- R43: value 5mR/3W/1% -> 10mR/3W/1%
- R7: value 0R -> 1.1K; MNP RC0603JR-070RL -> AC0603FR-071K1L; Unit Price 0.015 -> 0.021
Connections:
- net MC_IPM_TEMP is gone; now on net MC_TEMP_SEN: R11.2
- net MC_VW is gone; now on net MC_VV: U1.20 (W)
- net GND: now also R75.1
- net MC_VU: now also C13.1, J3.4, M3.2, R69.2
- net MC_VV: now also C12.1, J3.2, M1.2, R68.2; no longer U1.21 (V)
- net PGND: now also U1.17 (NW), R76.1
- net at C11.2, J3.3, M2.2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: now also U1.21 (V)
- net MC_IV_SEN_P: now reaches R43.4
- net IPM_PWM_FLT: now reaches R7.1, U1.15 (ITR)
- net IPM_PWM_FLT: now also R75.2
- net at R43.2, U1.18 (NV): no longer U1.17 (NW), U1.19 (NU)
- net MC_IV_SEN_N: now reaches R43.3
- net MC_TEMP_SEN: now reaches C15.2
- net INV_FLT_OC renamed MC_PWM_FLT
- net VREF renamed AVDD
- new net: R76.2, U1.19 (NU)
- new net MC_IU_SEN_N: R76.3
- new net MC_IU_SEN_P: R76.4
Other:
- note removed: "VOUT=(ILoad*RSen)*Gain+Vref Gain=50, Vref=0, RSen=5mR, Imax=13A, Vout=3.25V"
- moved on the sheet: C11, C12, C13, C16, C17, C2, C3, C4, C5, C6, C7, D10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

Commit message: V1 schematic update 3
Parts:
- added R49: 10mR/3W/1%, SAMPI:SHU2512, symbol SAMPI:SHUNT
Connections:
- net PGND: now also R49.1; no longer R43.1, R76.1, U1.17 (NW)
- net MC_UW: now reaches C11.2, J3.3, M2.2, R63.2, U1.21 (V)
- net MC_VU renamed MC_UU
- net MC_VV renamed MC_UV
- new net: R43.1, R49.2, R76.1, U1.17 (NW)
- new net MC_IDC_SEN_N: R49.3
- new net MC_IDC_SEN_P: R49.4
Changed lines of the file:
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@@
 	)
 	(junction
+		(at 154.305 17.78)
+		(diameter 0)
+		(color 0 0 0 0)
+	)
+	(junction
 		(at 154.305 45.72)
 		(diameter 0)
@@
 	(wire
 		(pts
-			(xy 117.475 93.98) (xy 117.475 95.25)
-		)
-		(stroke
-			(width 0.381)
-			(type default)
-		)
-	)
-	(wire
-		(pts
 			(xy 91.44 144.78) (xy 100.33 144.78)
 		)
@@
 	(wire
 		(pts
+			(xy 117.475 93.98) (xy 117.475 95.25)
+		)
+		(stroke
+			(width 0.381)
+			(type default)
+		)
+	)
+	(wire
+		(pts
 			(xy 114.3 19.05) (xy 114.3 20.32)
 		)
@@
 	(wire
 		(pts
+			(xy 117.475 106.68) (xy 117.475 107.95)
+		)
+		(stroke
+			(width 0.381)
+			(type default)
+		)
+	)
+	(wire
+		(pts
 			(xy 107.95 45.72) (xy 154.305 45.72)
 		)
@@
 	(wire
 		(pts
+			(xy 154.305 17.78) (xy 155.575 17.78)
+		)
+		(stroke
+			(width 0)
+			(type default)
+		)
+	)
+	(wire
+		(pts
 			(xy 55.245 33.02) (xy 55.245 34.29)
 		)
@@
 		)
 	)
+	(hierarchical_label "MC_IDC_SEN_P"
+		(shape output)
+		(at 120.65 99.06 0)
+		(fields_autoplaced yes)
+		(effects
+			(font
+				(size 1.27 1.27)
+				(color 0 200 100 1)
+			)
+			(justify left)
+		)
+	)
 	(hierarchical_label "MC_PWM_UH"
 		(shape input)
@@
 		)
 	)
+	(hierarchical_label "MC_IDC_SEN_N"
+		(shape output)
+		(at 120.65 102.87 0)
+		(fields_autoplaced yes)
+		(effects
+			(font
+				(size 1.27 1.27)
+				(color 0 200 100 1)
+			)
+			(justify left)
+		)
+	)
 	(hierarchical_label "IPM_PWM_UH"
 		(shape input)
@@
 		)
 	)
+	(hierarchical_label "MC_UW"
+		(shape output)
+		(at 155.575 17.78 0)
+		(fields_autoplaced yes)
+		(effects
+			(font
+				(size 1.27 1.27)
+				(color 0 200 100 1)
+			)
+			(justify left)
+		)
+	)
 	(hierarchical_label "IPM_PWM_UH"
 		(shape input)
@@
 		)
 	)
-	(hierarchical_label "MC_VV"
+	(hierarchical_label "MC_UV"
 		(shape output)
 		(at 172.085 17.78 0)
@@
 		)
 	)
-	(hierarchical_label "MC_VU"
+	(hierarchical_label "MC_UU"
 		(shape output)
 		(at 187.96 17.78 0)
@@
 	(symbol
 		(lib_id "SAMPI:PGND")
-		(at 117.475 95.25 0)
+		(at 117.475 107.95 0)
 		(unit 1)
 		(exclude_from_sim no)
@@
 		(dnp no)
 		(property "Reference" "#PWR05"
-			(at 117.475 100.33 0)
+			(at 117.475 113.03 0)
 			(effects
 				(font
@@
 		)
 		(property "Value" "PGND"
-			(at 117.475 99.06 0)
+			(at 117.475 111.76 0)
 			(effects
 				(font
@@
 		)
 		(property "Footprint" ""
-			(at 117.475 95.25 0)
+			(at 117.475 107.95 0)
 			(effects
 				(font
@@
 		)
 		(property "Datasheet" ""
-			(at 117.475 95.25 0)
+			(at 117.475 107.95 0)
 			(effects
 				(font
@@
 		)
 		(property "Description" ""
-			(at 117.475 95.25 0)
+			(at 117.475 107.95 0)
 			(effects
 				(font
@@
 					(unit 1)
 				)
+			)
+		)
+	)
+	(symbol
+		(lib_id "SAMPI:SHUNT")
+		(at 113.03 104.14 90)
+		(unit 1)
+		(exclude_from_sim no)
+		(in_bom yes)
+		(on_board yes)
+		(dnp no)
+		(property "Reference" "R49"
+			(at 113.665 98.425 90)
+			(effects
+				(font
+					(size 1.5 1.5)
+					(bold yes)
+				)
+			)
+		)
+		(property "Value" "10mR/3W/1%"
+			(at 111.125 100.965 90)
+			(effects
+				(font
+					(size 1.27 1.27)
+				)
+			)
+		)
+		(property "Footprint" "SAMPI:SHU2512"
+			(at 113.03 104.14 0)
+			(effects
+				(font
+					(size 1.27 1.27)
+				)
+				(hide yes)
+			)
+		)
+		(property "Datasheet" ""
+			(at 113.03 104.14 0)
+			(effects
+				(font
+					(size 1.27 1.27)
+				)
+				(hide yes)
+			)
+		)
+		(property "Description" "RES 0.005 OHM 1% 3W 2512"
+			(at 113.03 104.14 0)
+			(effects
+				(font
+					(size 1.27 1.27)
+				)
+				(hide yes)
+			)
+		)
+		(property "MNP" "MSMA2512R0050FGM"
+			(at 108.585 104.14 90)
+			(effects
+				(font
+					(size 1.27 1.27)
+				)
+				(hide yes)
+			)
+		)
+		(property "Comment" ""
+			(at 113.03 104.14 0)
+			(effects
+				(font
+					(size 1.27 1.27)
+				)
+				(hide yes)
+			)
+		)
+		(property "Unit Price" "0.6"
+			(at 113.03 104.14 0)
+			(effects
+				(font
+					(size 1.27 1.27)
+				)
+				(hide yes)
+			)
+		)
+		(property "MFT" "Eaton"
+			(at 113.03 104.14 0)
+			(effects
+				(font
+					(size 1.27 1.27)
+				)
+				(hide yes)
+			)
+		)
+		(property "Checked" "OK"
+			(at 113.03 104.14 0)
+			(effects
+				(font
+					(size 1.27 1.27)
+				)
+				(hide yes)
+			)
+		)
+		(pin "1"
+		)
+		(pin "2"
+		)
+		(pin "3"
+		)
+		(pin "4"
+		)
+		(instances
+			(project "HW.ACIM-INV"
+				(path "/20f80521-75f2-4ccc-bb34-c9566e70ef5c/220ce183-b27e-490b-828f-5201e8e92b41"
+					(reference "R49")
+					(unit 1)
+				)

Commit message: V1 schematic update 6
Parts:
- added C93, C96: 100nF, SAMPI:CAP0603, symbol SAMPI:CERCAP
- added C94, C97: 1nF, SAMPI:CAP0603, symbol SAMPI:CERCAP
- added U15, U16: I=±10A, SAMPI:SOIC8_ALL, symbol SAMPI:ACS724
- C11, C12, C13, C14: Checked OK -> (none); Unit Price 0.19 -> (none)
- C15: Checked OK -> (none); Unit Price 0.012 -> (none)
- C16: Checked OK -> (none); Unit Price 0.85 -> (none)
- C17, C2, C5, C7: Checked OK -> (none); Unit Price 0.0146 -> (none)
- C3, C4, C6: Checked OK -> (none); Unit Price 0.45 -> (none)
- D10, D11, D13, D15: Checked OK -> (none)
- D12, D14: Checked OK -> (none); Unit Price 0.1 -> (none)
- G1: Checked OK -> (none); Unit Price 0.53 -> (none)
- J3: Checked OK -> (none); Unit Price 0.84 -> (none)
- M1, M2, M3: Checked OK -> (none); Unit Price 0.255 -> (none)
- Q4, Q5, Q6: Checked OK -> (none); Unit Price 0.148 -> (none)
- R11, R13, R14, R15, R19, R20, R21, R22, R64, R66, R7: Checked OK -> (none); Unit Price 0.021 -> (none)
- R12, R16, R17, R18, R23, R24, R25, R75: Checked OK -> (none); Unit Price 0.019 -> (none)
- R43, R49, R76: Checked OK -> (none); Unit Price 0.6 -> (none)
- R63, R68, R69: Checked OK -> (none); Unit Price 0.035 -> (none)
- U1: Checked OK -> (none); Unit Price 11.37 -> (none)
Connections:
- net GND: now also C93.1, C94.1, C96.1, C97.1, U15.5 (GND), U16.5 (GND)
- net MC_UU: now also U15.3 (IPN1), U15.4 (IPN2); no longer U1.22 (U)
- net MC_UW: now also U16.3 (IPN1), U16.4 (IPN2); no longer U1.21 (V)
- new net: C97.2, U16.6 (FILTER)
- new net: C94.2, U15.6 (FILTER)
- new net: U1.21 (V), U16.1 (IPP1), U16.2 (IPP2)
- new net: U1.22 (U), U15.1 (IPP1), U15.2 (IPP2)
- new net +5V: C93.2, C96.2, U15.8 (VCC), U16.8 (VCC)
- new net MC_IU_HAL: U15.7 (VIOUT)
- new net MC_IV_HAL: U16.7 (VIOUT)
Other:
- moved on the sheet: C11, C12, C13, C14, C15, C16, C17, C2, C3, C4, C5, C6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

Commit message: V1 schematic update 7
Connections:
- net +5V renamed VREF
Changed lines of the file:
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@@
 	)
 	(symbol
-		(lib_id "power:+5V")
-		(at 157.48 80.01 0)
-		(unit 1)
-		(exclude_from_sim no)
-		(in_bom yes)
-		(on_board yes)
-		(dnp no)
-		(property "Reference" "#PWR0181"
-			(at 157.48 83.82 0)
-			(effects
-				(font
-					(size 1.5 1.5)
-					(bold yes)
-				)
-				(hide yes)
-			)
-		)
-		(property "Value" "+5V"
-			(at 157.48 76.2 0)
-			(effects
-				(font
-					(size 1.27 1.27)
-					(bold yes)
-				)
-			)
-		)
-		(property "Footprint" ""
-			(at 157.48 80.01 0)
-			(effects
-				(font
-					(size 1.27 1.27)
-				)
-				(hide yes)
-			)
-		)
-		(property "Datasheet" ""
-			(at 157.48 80.01 0)
-			(effects
-				(font
-					(size 1.27 1.27)
-				)
-				(hide yes)
-			)
-		)
-		(property "Description" ""
-			(at 157.48 80.01 0)
-			(effects
-				(font
-					(size 1.27 1.27)
-				)
-				(hide yes)
-			)
-		)
-		(pin "1"
-		)
-		(instances
-			(project "HW.ACIM-INV"
-				(path "/20f80521-75f2-4ccc-bb34-c9566e70ef5c/220ce183-b27e-490b-828f-5201e8e92b41"
-					(reference "#PWR0181")
-					(unit 1)
-				)
-			)
-		)
-	)
-	(symbol
 		(lib_id "SAMPI:IKCM15H60GAXKMA2")
 		(at 55.88 12.7 0)
@@
 	)
 	(symbol
+		(lib_id "SAMPI:VREF")
+		(at 195.58 80.01 0)
+		(unit 1)
+		(exclude_from_sim no)
+		(in_bom yes)
+		(on_board yes)
+		(dnp no)
+		(property "Reference" "#PWR0200"
+			(at 195.58 83.82 0)
+			(effects
+				(font
+					(size 1.27 1.27)
+				)
+				(hide yes)
+			)
+		)
+		(property "Value" "VREF"
+			(at 195.58 76.2 0)
+			(effects
+				(font
+					(size 1.27 1.27)
+					(bold yes)
+				)
+			)
+		)
+		(property "Footprint" ""
+			(at 195.58 80.01 0)
+			(effects
+				(font
+					(size 1.27 1.27)
+				)
+				(hide yes)
+			)
+		)
+		(property "Datasheet" ""
+			(at 195.58 80.01 0)
+			(effects
+				(font
+					(size 1.27 1.27)
+				)
+				(hide yes)
+			)
+		)
+		(property "Description" "Power symbol creates a global label with name \"VREF\""
+			(at 195.58 80.01 0)
+			(effects
+				(font
+					(size 1.27 1.27)
+				)
+				(hide yes)
+			)
+		)
+		(pin "1"
+		)
+		(instances
+			(project "HW.ACIM-INV"
+				(path "/20f80521-75f2-4ccc-bb34-c9566e70ef5c/220ce183-b27e-490b-828f-5201e8e92b41"
+					(reference "#PWR0200")
+					(unit 1)
+				)
+			)
+		)
+	)
+	(symbol
 		(lib_id "SAMPI:CERCAP")
 		(at 110.49 24.13 270)
@@
 	)
 	(symbol
-		(lib_id "power:+5V")
-		(at 195.58 80.01 0)
-		(unit 1)
-		(exclude_from_sim no)
-		(in_bom yes)
-		(on_board yes)
-		(dnp no)
-		(property "Reference" "#PWR0200"
-			(at 195.58 83.82 0)
-			(effects
-				(font
-					(size 1.5 1.5)
-					(bold yes)
-				)
-				(hide yes)
-			)
-		)
-		(property "Value" "+5V"
-			(at 195.58 76.2 0)
-			(effects
-				(font
-					(size 1.27 1.27)
-					(bold yes)
-				)
-			)
-		)
-		(property "Footprint" ""
-			(at 195.58 80.01 0)
-			(effects
-				(font
-					(size 1.27 1.27)
-				)
-				(hide yes)
-			)
-		)
-		(property "Datasheet" ""
-			(at 195.58 80.01 0)
-			(effects
-				(font
-					(size 1.27 1.27)
-				)
-				(hide yes)
-			)
-		)
-		(property "Description" ""
-			(at 195.58 80.01 0)
-			(effects
-				(font
-					(size 1.27 1.27)
-				)
-				(hide yes)
-			)
-		)
-		(pin "1"
-		)
-		(instances
-			(project "HW.ACIM-INV"
-				(path "/20f80521-75f2-4ccc-bb34-c9566e70ef5c/220ce183-b27e-490b-828f-5201e8e92b41"
-					(reference "#PWR0200")
-					(unit 1)
-				)
-			)
-		)
-	)
-	(symbol
 		(lib_id "power:GND")
 		(at 100.33 158.75 0)
@@
 					(unit 1)
 				)
+			)
+		)
+	)
+	(symbol
+		(lib_id "SAMPI:VREF")
+		(at 157.48 80.01 0)
+		(unit 1)
+		(exclude_from_sim no)
+		(in_bom yes)
+		(on_board yes)
+		(dnp no)
+		(property "Reference" "#PWR0181"
+			(at 157.48 83.82 0)
+			(effects
+				(font
+					(size 1.27 1.27)
+				)
+				(hide yes)
+			)
+		)
+		(property "Value" "VREF"
+			(at 157.48 76.2 0)
+			(effects
+				(font
+					(size 1.27 1.27)
+					(bold yes)
+				)
+			)
+		)
+		(property "Footprint" ""
+			(at 157.48 80.01 0)
+			(effects
+				(font
+					(size 1.27 1.27)
+				)
+				(hide yes)
+			)
+		)
+		(property "Datasheet" ""
+			(at 157.48 80.01 0)
+			(effects
+				(font
+					(size 1.27 1.27)
+				)
+				(hide yes)
+			)
+		)
+		(property "Description" "Power symbol creates a global label with name \"VREF\""
+			(at 157.48 80.01 0)
+			(effects
+				(font
+					(size 1.27 1.27)
+				)
+				(hide yes)
+			)
+		)
+		(pin "1"
+		)
+		(instances
+			(project "HW.ACIM-INV"
+				(path "/20f80521-75f2-4ccc-bb34-c9566e70ef5c/220ce183-b27e-490b-828f-5201e8e92b41"
+					(reference "#PWR0181")
+					(unit 1)
+				)

Commit message: V1 schematic update 8
Changed lines of the file:
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@@
 	(wire
 		(pts
-			(xy 254 45.72) (xy 274.955 45.72)
+			(xy 254 45.72) (xy 276.225 45.72)
 		)
 		(stroke
@@
 	(wire
 		(pts
-			(xy 274.955 45.72) (xy 276.225 45.72)
-		)
-		(stroke
-			(width 0.254)
-			(type default)
-		)
-	)
-	(wire
-		(pts
 			(xy 157.48 80.01) (xy 157.48 81.28)
 		)
@@
 	)
 	(hierarchical_label "IPM_PWM_UH"
-		(shape input)
+		(shape output)
 		(at 52.07 139.7 0)
 		(fields_autoplaced yes)
@@
 	)
 	(hierarchical_label "IPM_PWM_VH"
-		(shape input)
+		(shape output)
 		(at 52.07 144.78 0)
 		(fields_autoplaced yes)
@@
 	)
 	(hierarchical_label "IPM_PWM_VL"
-		(shape input)
+		(shape output)
 		(at 109.22 144.78 0)
 		(fields_autoplaced yes)
@@
 	)
 	(hierarchical_label "IPM_PWM_WL"
-		(shape input)
+		(shape output)
 		(at 109.22 149.86 0)
 		(fields_autoplaced yes)
@@
 	)
 	(hierarchical_label "IPM_PWM_UL"
-		(shape input)
+		(shape output)
 		(at 109.22 139.7 0)
 		(fields_autoplaced yes)
@@
 	)
 	(hierarchical_label "IPM_PWM_WH"
-		(shape input)
+		(shape output)
 		(at 52.07 149.86 0)
 		(fields_autoplaced yes)

Commit message: V1 schematic update 11
Parts:
- removed D10, D11: TVS 5.5V 3-CH, SAMPI:SOT143B_NEXT, symbol SAM1:TVS_3CH
- removed Q4, Q5, Q6: 20V/1A, SAMPI:SOT23, symbol SAMPI:FET_N-CH
- removed R13, R14, R15, R19, R21, R22, R7: 1.1K, SAMPI:RES0603, symbol SAMPI:RES
- removed R16, R17, R18, R23, R24, R25, R75: 100K, SAMPI:RES0603, symbol SAMPI:RES
- removed R43, R76: 10mR/3W/1%, SAMPI:SHU2512, symbol SAMPI:SHUNT
- added C18, C19, C20, C23, C24, C25: 10uF, SAMPI:CAP0603, symbol SAMPI:CERCAP
- added D1, D2: TVS 5.5V 3-CH, SAMPI:SOT143B_NEXT, symbol SAM1:TVS_3CH
- added U3, U5, U9: DIGI ISO 2-CH, SAMPI:SOIC8_ALL, symbol SAMPI:ADUM1200
Connections:
- net +3V3: now also C18.2, C19.2, C23.2, U3.1 (VDD1), U5.1 (VDD1), U9.1 (VDD1); no longer D15.4 (CH3), R20.2, R64.2, R66.2
- net GND: now also D12.K, D13.K, D14.K, C18.1, C19.1, C23.1, U3.4 (GND1), U5.4 (GND1), U9.4 (GND1); no longer D15.1 (GND)
- net IPM_PWM_UH: now also D15.2 (CH1), U9.7 (VOA)
- net IPM_PWM_UL: now also D15.3 (CH2), U9.6 (VOB)
- net IPM_PWM_VH: now also D1.2 (CH1), U3.7 (VOA)
- net IPM_PWM_VL: now also D1.3 (CH2), U3.6 (VOB)
- net IPM_PWM_WH: now also D2.2 (CH1), U5.7 (VOA)
- net IPM_PWM_WL: now also D2.3 (CH2), U5.6 (VOB)
- net MC_PWM_UH: now also R20.2, U9.2 (VIA)
- net MC_PWM_UL: now also U9.3 (VIB)
- net MC_PWM_VH: now also R64.2, U3.2 (VIA)
- net MC_PWM_VL: now also U3.3 (VIB)
- net MC_PWM_WH: now also R66.2, U5.2 (VIA); no longer D15.3 (CH2)
- net MC_PWM_WL: now also U5.3 (VIB); no longer D15.2 (CH1)
- net at R49.2, U1.17 (NW): now also U1.18 (NV), U1.19 (NU)
- net MC_UU renamed MC_U
- net MC_UV renamed MC_W
- net MC_UW renamed MC_V
- new net +3V3_ISO: C20.2, C24.2, C25.2, D1.4 (CH3), D15.4 (CH3), D2.4 (CH3), U3.8 (VDD2), U5.8 (VDD2), U9.8 (VDD2)
- new net GND_ISO: C20.1, C24.1, C25.1, D1.1 (GND), D15.1 (GND), D2.1 (GND), U3.5 (GND2), U5.5 (GND2), U9.5 (GND2)
Other:
- moved on the sheet: C11, C12, C13, C14, C15, C16, C17, C2, C3, C4, C5, C6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

Commit message: V1 schematic update 13
Parts:
- removed C15: 22pF, SAMPI:CAP0603, symbol SAMPI:CERCAP
- removed R11: 1.1K, SAMPI:RES0603, symbol SAMPI:RES
- added OP1: OPTO-BJT-1CH, SAMPI:OPTO_SO4_7.6MM, symbol SAMPI:OPTO-BJT-1CH
- added R1: 10K, SAMPI:RES0603, symbol SAMPI:RES
- added R2: 75K, SAMPI:RES0603, symbol SAMPI:RES
Connections:
- net GND: no longer C16.-, C17.2, U1.16 (VSS)
- net GND_ISO: now also C16.-, C17.2, U1.16 (VSS), R2.2
- net MC_TEMP_P: now reaches R12.2, U1.14 (VFO)
- net MC_TEMP_P: now also R1.1
- new net MC_TEMP_N: R1.2, R2.1
Other:
- moved on the sheet: C93, C94, C96, C97, R12, U15, U16

Commit message: V1 schematic update 14
Parts:
- added R17: 1.1K, SAMPI:RES0603, symbol SAMPI:RES
- added R18: 10K, SAMPI:RES0603, symbol SAMPI:RES
- U3, U5, U9: value DIGI ISO 2-CH -> DIGI ISO
Connections:
- net CHASSIS: now also G1.2; no longer G1.1
- net GND: now also OP1.2 (K); no longer C93.1, C94.1, C96.1, C97.1, U15.5 (GND), U16.5 (GND)
- net GND_ISO: no longer C16.-, C17.2, R2.2, U1.16 (VSS)
- net IPM_PWM_FLT: now also OP1.4 (C), R18.2
- net at J3.1, M1.1, M2.1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: now also G1.1; no longer G1.2
- net at OP1.1 (A): now also R17.1
- net GND_INV: now reaches OP1.3 (E)
- net GND_INV: now also C16.-, C17.2, R2.2, U1.16 (VSS)
- net +15V renamed +16V_INV
- net MC_IDC_SEN_N renamed MC_IDC_N
- net MC_IDC_SEN_P renamed MC_IDC_P
- net VREF renamed +5V_ADC
- new net GND_ADC: C93.1, C94.1, C96.1, C97.1, U15.5 (GND), U16.5 (GND)
Other:
- note added: "HIGH VOLTAGE ZONE"
- note added: "LOW VOLTAGE ZONE"
- moved on the sheet: C18, C19, C20, C23, C24, C25, D1, D12, D13, D14, D15, D2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
