File: V1/Design/HW.ACIM-INV/Inverter.kicad_sch (KiCad schematic)
At the start: 52 parts, among them J3 MOTOR, M1 560V/1.75kA, M2 560V/1.75kA, M3 560V/1.75kA, U1 IPM 600V/15A, U15 I=±10A, U16 I=±10A, U3 DIGI ISO, U5 DIGI ISO, U9 DIGI ISO

Commit message: V1 schematic update 15
Parts:
- removed OP1: OPTO-BJT-1CH, SAMPI:OPTO_SO4_7.6MM, symbol SAMPI:OPTO-BJT-1CH
- removed R1, R18: 10K, SAMPI:RES0603, symbol SAMPI:RES
- removed R17: 1.1K, SAMPI:RES0603, symbol SAMPI:RES
- removed R2: 75K, SAMPI:RES0603, symbol SAMPI:RES
- added C78, C80, C81: 100nF, SAMPI:CAP0603, symbol SAMPI:CERCAP
- added OP2: OPTO-BJT-1CH, SAMPI:OPTO_SO4_7.6MM, symbol SAMPI:OPTO-BJT-1CH
- added Q1: 20V/1A, SAMPI:SOT23, symbol SAMPI:FET_N-CH
- added R30: 10K, SAMPI:RES0603, symbol SAMPI:RES
- added R31: 1.1K, SAMPI:RES0603, symbol SAMPI:RES
- added R37: 1M, SAMPI:RES1206, symbol SAMPI:RES
- added RV2: 100K, SAMPI:TC33X-2, symbol SAMPI:POT
- added U20: CMP-1CH, SAMPI:SOT25_DIODES, symbol SAMPI:CMP-1CH
- D1, D15, D2: value TVS 5.5V 3-CH -> TVS 5.5V
Connections:
- net AVDD is gone; now on net +5V_INV: R12.1
- net GND_ADC is gone; now on net GND_MCU: C93.1, C94.1, C96.1, C97.1, U15.5 (GND), U16.5 (GND)
- net GND_ISO is gone; now on net GND_INV: C20.1, C24.1, C25.1, D1.1 (GND), D15.1 (GND), D2.1 (GND), U3.5 (GND2), U5.5 (GND2), U9.5 (GND2)
- net GND_INV: now also C78.1, C80.1, C81.1, OP2.2 (K), Q1.2 (S), RV2.3 (CW), U20.2 (VSS)
- net IPM_PWM_FLT: now also OP2.1 (A), Q1.3 (D), R31.1
- net +3V3 renamed +3V3_MCU
- net +3V3_MCU: now also R30.1
- net +3V3_ISO renamed +5V_INV
- net +5V_INV: now also C78.2, R31.2, RV2.1 (CCW), U20.5 (VDD)
- net +5V_ADC renamed +5V_MCU
- net GND renamed GND_MCU
- net GND_MCU: now also OP2.3 (E)
- net MC_TEMP_P renamed IPM_TEMP_SEN
- net IPM_TEMP_SEN: now also C81.2, R37.1, U20.1 (VIN-)
- new net: C80.2, RV2.2 (WIPER), U20.3 (VIN+)
- new net: Q1.1 (G), R37.2, U20.4 (VOUT)
- new net MC_TEMP_FLT: OP2.4 (C), R30.2
Other:
- company: TON DUC THANG UNIVERSITY -> (none)
- moved on the sheet: C11, C12, C13, C14, C16, C17, C18, C19, C2, C20, C23, C24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

Commit message: V1 schematic update 16
Parts:
- C78, C80, C81: Checked OK -> (none); Unit Price 0.0146 -> (none)
- Q1: Checked OK -> (none); Unit Price 0.148 -> (none)
- R12: value 100K -> 10K; MFT YAGEO -> (none); MNP RC0603FR-07100KL -> (none)
- R20, R31, R64, R66: value 1.1K -> 1K; MFT YAGEO -> (none); MNP AC0603FR-071K1L -> (none)
- R30: MFT YAGEO -> (none); MNP RC0603FR-07100KL -> (none)
- R37: value 1M -> 1.2M; footprint SAMPI:RES1206 -> SAMPI:RES0603; Checked OK -> (none); MFT Walsin -> (none); MNP WR12X105 JTL -> (none); Unit Price 0.02 -> (none)
- RV2: value 100K -> 20K; MNP TC33X-2-104E -> TC33X-2-203E
- U20: Checked OK -> (none); Unit Price 0.36 -> (none)
Connections:
- net GND_INV: no longer OP2.2 (K)
- net IPM_PWM_FLT: now also Q1.1 (G), R37.2, U20.4 (VOUT); no longer OP2.1 (A), Q1.3 (D), R31.1
- new net: OP2.1 (A), R31.1
- new net: OP2.2 (K), Q1.3 (D)
Other:
- moved on the sheet: C78, C80, C81, Q1, R37, RV2, U20

Commit message: V1 schematic update 17
Parts:
- added C50: 470nF/630V, SAMPI:FCAP-15MM, symbol SAMPI:CERCAP
- added J6: U, symbol SAMPI:BANANA
- added J7: V, symbol SAMPI:BANANA
- added J8: W, symbol SAMPI:BANANA
- added J9: N, symbol SAMPI:BANANA
- C41: renamed from C16; value 470uF -> 470uF/25V
- OP1: renamed from OP2; MFT Everlight Electronics Co Ltd -> Everlight
- R16: renamed from R12; MFT (none) -> YAGEO; MNP (none) -> RC0603JR-0710KL
- R18: renamed from R20; MFT (none) -> YAGEO; MNP (none) -> RC0603JR-071KL
- R19: renamed from R64; MFT (none) -> YAGEO; MNP (none) -> RC0603JR-071KL
- R20: renamed from R66; MFT (none) -> YAGEO; MNP (none) -> RC0603JR-071KL
- R22: renamed from R30; MFT (none) -> YAGEO; MNP (none) -> RC0603JR-0710KL
- R24: renamed from R31; MFT (none) -> YAGEO; MNP (none) -> RC0603JR-071KL
- R25: renamed from R37; MFT (none) -> YAGEO; MNP (none) -> RC0603JR-071M2L
- RV1: renamed from RV2; MFT Bourns Inc. -> Bourns
- U10: renamed from U5; MFT Analog Devices Inc. -> Analog Devices
- U8: renamed from U9; MFT Analog Devices Inc. -> Analog Devices
- U9: renamed from U3; MFT Analog Devices Inc. -> Analog Devices
- renumbered C3 to C38, C4 to C39, C6 to C40, C17 to C42, C2 to C43, C5 to C44, C7 to C45, C25 to C46, C20 to C47, C24 to C48, C14 to C49, C93 to C51, C94 to C52, C19 to C53, C18 to C54, C23 to C55, C96 to C56, C97 to C57, C13 to C58, C11 to C59, C12 to C60, C78 to C61, C80 to C62, C81 to C63, D2 to D10, D13 to D11, D14 to D12, D12 to D13, D15 to D8, D1 to D9, G1 to G2, J3 to J5, M3 to M5, M2 to M6, M1 to M7, Q1 to Q3, R49 to R17, R63 to R21, R68 to R23, R69 to R26, U15 to U11, U16 to U12, U20 to U13, U1 to U7
Connections:
- net PGND: now also C50.2
- net VDC: now also C50.1

Commit message: V1 schematic update 18
Parts:
- removed J5: MOTOR, SAMPI:TMB4_9.5, symbol SAMPI:SIL04
- added C88: 100uF/450V, SAMPI:CAP_ELEC-18.0x51.5-LS7.5, symbol SAMPI:ELECCAP
- added J16: HIGH VOLTAGE OUTPUTS, SAMPI:HDF1x10x2.54_TH_RA, symbol SAMPI:SIL10
- added J2: U, SAMPI:QC-6.3, symbol SAMPI:SIL01
- added J3: V, SAMPI:QC-6.3, symbol SAMPI:SIL01
- added J4: W, SAMPI:QC-6.3, symbol SAMPI:SIL01
- added J5: N, SAMPI:QC-6.3, symbol SAMPI:SIL01
Connections:
- net CHASSIS: now also J16.1, J16.2
- net MC_U: now also J2.1
- net MC_V: now also J3.1
- net MC_W: now also J4.1
- net PGND: now also C88.-, J16.4, J16.5, J16.6
- net VDC: now also C88.+, J16.10, J16.8, J16.9
- net at G2.1, M5.1, M6.1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: now also J5.1
Other:
- moved on the sheet: C49, C50, J6, J7, J8, J9

Commit message: V1 schematic update 20
Connections:
- net CHASSIS: now also J16.10, J16.9; no longer J16.1, J16.2
- net PGND: now also J16.1, J16.2, J16.3; no longer J16.4, J16.5, J16.6
- net VDC: now also J16.5, J16.6, J16.7; no longer J16.10, J16.8, J16.9
Changed lines of the file:
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@@
 	)
 	(junction
-		(at 268.605 21.59)
-		(diameter 0)
-		(color 0 0 0 0)
-	)
-	(junction
 		(at 245.11 131.445)
 		(diameter 0)
@@
 	)
 	(junction
-		(at 268.605 31.75)
-		(diameter 0)
-		(color 0 0 0 0)
-	)
-	(junction
 		(at 202.565 46.99)
 		(diameter 0)
@@
 	(wire
 		(pts
-			(xy 267.335 31.75) (xy 268.605 31.75)
-		)
-		(stroke
-			(width 0.3)
-			(type default)
-		)
-	)
-	(wire
-		(pts
 			(xy 219.075 66.04) (xy 219.075 67.31)
 		)
@@
 	(wire
 		(pts
-			(xy 267.335 21.59) (xy 268.605 21.59)
-		)
-		(stroke
-			(width 0.3)
-			(type default)
-		)
-	)
-	(wire
-		(pts
 			(xy 207.01 57.15) (xy 219.075 57.15)
 		)
@@
 	(wire
 		(pts
+			(xy 267.335 34.29) (xy 268.605 34.29)
+		)
+		(stroke
+			(width 0.3)
+			(type default)
+		)
+	)
+	(wire
+		(pts
 			(xy 81.28 145.415) (xy 74.93 145.415)
 		)
@@
 	(wire
 		(pts
+			(xy 267.335 24.13) (xy 268.605 24.13)
+		)
+		(stroke
+			(width 0.3)
+			(type default)
+		)
+	)
+	(wire
+		(pts
 			(xy 40.005 34.29) (xy 40.005 35.56)
 		)
@@
 	(symbol
 		(lib_id "SAMPI:SIL10")
-		(at 269.875 48.26 0)
-		(mirror x)
+		(at 269.875 17.78 0)
 		(unit 1)
 		(exclude_from_sim no)
@@
 		)
 		(property "Value" "HIGH VOLTAGE OUTPUTS"
-			(at 276.225 22.86 90)
+			(at 276.225 43.18 90)
 			(effects
 				(font
@@
 		)
 		(property "Footprint" "SAMPI:HDF1x10x2.54_TH_RA"
-			(at 269.875 48.26 0)
+			(at 269.875 17.78 0)
 			(effects
 				(font
@@
 		)
 		(property "Datasheet" ""
-			(at 269.875 48.26 0)
+			(at 269.875 17.78 0)
 			(effects
 				(font
@@
 		)
 		(property "Description" "CONN HDR 10POS 0.1 TIN PCB R/A"
-			(at 269.875 48.26 0)
+			(at 269.875 17.78 0)
 			(effects
 				(font
@@
 		)
 		(property "MFT" "Sullins"
-			(at 269.875 48.26 0)
+			(at 269.875 17.78 0)
 			(effects
 				(font
@@
 		)
 		(property "MNP" "PPTC101LGBN-RC"
-			(at 269.875 48.26 0)
+			(at 269.875 17.78 0)
 			(effects
 				(font
@@
 		)
 		(property "Checked" "OK"
-			(at 269.875 48.26 0)
+			(at 269.875 17.78 0)
 			(effects
 				(font
@@
 		(pin "6"
 		)
-		(pin "8"
-		)
 		(pin "1"
 		)
@@
 		(pin "10"
 		)
-		(pin "4"
-		)
 		(pin "9"
 		)
 		(pin "5"
 		)
+		(pin "3"
+		)
+		(pin "7"
+		)
 		(instances
 			(project "HW.ACIM-INV"
@@
 	(symbol
 		(lib_id "power:VDC")
-		(at 267.335 21.59 90)
+		(at 267.335 34.29 90)
 		(unit 1)
 		(exclude_from_sim no)
@@
 		(dnp no)
 		(property "Reference" "#PWR0209"
-			(at 269.875 21.59 0)
+			(at 269.875 34.29 0)
 			(effects
 				(font
@@
 		)
 		(property "Value" "VDC"
-			(at 262.89 21.59 90)
+			(at 262.89 34.29 90)
 			(effects
 				(font
@@
 					(size 1.016 1.016)
 					(thickness 0.127)
+					(bold yes)
 				)
 			)
 		)
 		(property "Footprint" ""
-			(at 267.335 21.59 0)
+			(at 267.335 34.29 0)
 			(effects
 				(font
@@
 		)
 		(property "Datasheet" ""
-			(at 267.335 21.59 0)
+			(at 267.335 34.29 0)
 			(effects
 				(font
@@
 		)
 		(property "Description" ""
-			(at 267.335 21.59 0)
+			(at 267.335 34.29 0)
 			(effects
 				(font
@@
 	(symbol
 		(lib_id "SAMPI:PGND")
-		(at 267.335 31.75 270)
+		(at 267.335 24.13 270)
 		(mirror x)
 		(unit 1)
@@
 		(dnp no)
 		(property "Reference" "#PWR0207"
-			(at 262.255 31.75 0)
+			(at 262.255 24.13 0)
 			(effects
 				(font
@@
 		)
 		(property "Value" "PGND"
-			(at 262.89 31.75 90)
+			(at 262.89 24.13 90)
 			(effects
 				(font
@@
 		)
 		(property "Footprint" ""
-			(at 267.335 31.75 0)
+			(at 267.335 24.13 0)
 			(effects
 				(font
@@
 		)
 		(property "Datasheet" ""
-			(at 267.335 31.75 0)
+			(at 267.335 24.13 0)
 			(effects
 				(font
@@
 		)
 		(property "Description" ""
-			(at 267.335 31.75 0)
+			(at 267.335 24.13 0)
 			(effects
 				(font

Commit message: V1 schematic update 22
Parts:
- removed R17: 10mR/3W/1%, SAMPI:SHU2512, symbol SAMPI:SHUNT
- added C3: 100nF, SAMPI:CAP0603, symbol SAMPI:CERCAP
- added C4: 1nF, SAMPI:CAP0603, symbol SAMPI:CERCAP
- added C8: 100pF/2kV, SAMPI:CAP1206, symbol SAMPI:CERCAP
- added C9: 680uF/450V, SAMPI:ESMQ451VSN681MA50S, symbol SAMPI:ELECCAP
- added FT1: 120R@100MHz, SAMPI:FT0603, symbol SAMPI:FerriteBead
- added U1: I=±10A, SAMPI:SOIC8_ALL, symbol SAMPI:ACS724
Connections:
- net +5V_MCU: now also C3.2, U1.8 (VCC)
- net GND_INV: now also FT1.1
- net GND_MCU: now also C3.1, C4.1, U1.5 (GND)
- net PGND: now also C9.-, FT1.2, U1.3 (IPN1), U1.4 (IPN2)
- net VDC: now also C8.1, C9.+
- net at U7.17 (NW), U7.18 (NV), U7.19 (NU): now also C8.2, U1.1 (IPP1), U1.2 (IPP2)
- new net: C4.2, U1.6 (FILTER)
- new net MC_IDC_HAL: U1.7 (VIOUT)
Other:
- moved on the sheet: C49, C50, C88

Commit message: V1 schematic update 23
Connections:
- net MC_V: now also U7.21 (V); no longer U12.3 (IPN1), U12.4 (IPN2)
- net MC_W: now also U12.3 (IPN1), U12.4 (IPN2); no longer U7.20 (W)
- net at U12.1 (IPP1), U12.2 (IPP2): now also U7.20 (W); no longer U7.21 (V)
Changed lines of the file:
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@@
 	)
 	(junction
-		(at 186.055 36.83)
+		(at 158.75 69.85)
 		(diameter 0)
 		(color 0 0 0 0)
 	)
 	(junction
-		(at 219.075 57.15)
+		(at 186.055 36.83)
 		(diameter 0)
 		(color 0 0 0 0)
 	)
 	(junction
-		(at 86.995 127.635)
+		(at 219.075 57.15)
 		(diameter 0)
 		(color 0 0 0 0)
 	)
 	(junction
-		(at 168.91 69.85)
+		(at 86.995 127.635)
 		(diameter 0)
 		(color 0 0 0 0)
@@
 	)
 	(junction
-		(at 158.75 69.85)
+		(at 168.91 69.85)
 		(diameter 0)
 		(color 0 0 0 0)
@@
 	(wire
 		(pts
-			(xy 168.91 69.85) (xy 170.18 69.85)
+			(xy 167.64 69.85) (xy 168.91 69.85)
 		)
 		(stroke
@@
 	(wire
 		(pts
-			(xy 158.75 46.99) (xy 158.75 69.85)
+			(xy 245.11 131.445) (xy 252.73 131.445)
 		)
 		(stroke
-			(width 0.381)
+			(width 0)
 			(type default)
 		)
@@
 	(wire
 		(pts
-			(xy 245.11 131.445) (xy 252.73 131.445)
+			(xy 132.715 104.14) (xy 133.985 104.14)
 		)
 		(stroke
@@
 	(wire
 		(pts
-			(xy 132.715 104.14) (xy 133.985 104.14)
+			(xy 168.91 69.85) (xy 170.18 69.85)
 		)
 		(stroke
-			(width 0)
+			(width 0.381)
 			(type default)
 		)
@@
 	(wire
 		(pts
-			(xy 92.71 46.99) (xy 158.75 46.99)
+			(xy 92.71 46.99) (xy 168.91 46.99)
 		)
 		(stroke
@@
 	(wire
 		(pts
-			(xy 158.75 69.85) (xy 160.02 69.85)
+			(xy 157.48 69.85) (xy 158.75 69.85)
 		)
 		(stroke
@@
 	(wire
 		(pts
+			(xy 168.91 57.15) (xy 168.91 69.85)
+		)
+		(stroke
+			(width 0.381)
+			(type default)
+		)
+	)
+	(wire
+		(pts
 			(xy 124.46 130.175) (xy 124.46 136.525)
 		)
@@
 	(wire
 		(pts
-			(xy 167.64 69.85) (xy 168.91 69.85)
-		)
-		(stroke
-			(width 0.381)
-			(type default)
-		)
-	)
-	(wire
-		(pts
 			(xy 226.06 117.475) (xy 224.79 117.475)
 		)
@@
 	(wire
 		(pts
-			(xy 157.48 69.85) (xy 158.75 69.85)
-		)
-		(stroke
-			(width 0.381)
-			(type default)
-		)
-	)
-	(wire
-		(pts
 			(xy 27.305 35.56) (xy 27.305 34.29)
 		)
@@
 	(wire
 		(pts
-			(xy 168.91 46.99) (xy 168.91 69.85)
-		)
-		(stroke
-			(width 0.381)
-			(type default)
-		)
-	)
-	(wire
-		(pts
 			(xy 45.72 99.06) (xy 45.72 95.25)
 		)
@@
 	(wire
 		(pts
+			(xy 158.75 69.85) (xy 160.02 69.85)
+		)
+		(stroke
+			(width 0.381)
+			(type default)
+		)
+	)
+	(wire
+		(pts
 			(xy 268.605 41.91) (xy 269.875 41.91)
 		)
@@
 	(wire
 		(pts
-			(xy 92.71 57.15) (xy 207.01 57.15)
+			(xy 92.71 57.15) (xy 158.75 57.15)
 		)
 		(stroke
@@
 	(wire
 		(pts
+			(xy 168.91 57.15) (xy 207.01 57.15)
+		)
+		(stroke
+			(width 0.3)
+			(type default)
+		)
+	)
+	(wire
+		(pts
 			(xy 96.52 155.575) (xy 86.995 155.575)
 		)
@@
 	(wire
 		(pts
+			(xy 158.75 57.15) (xy 158.75 69.85)
+		)
+		(stroke
+			(width 0.381)
+			(type default)
+		)
+	)
+	(wire
+		(pts
 			(xy 132.715 155.575) (xy 132.715 156.845)
 		)
@@
 		)
 		(property "Value" "470uF/25V"
-			(at 29.845 96.52 90)
+			(at 29.21 96.52 90)
 			(effects
 				(font

Commit message: V1 schematic update 24
Parts:
- removed D10, D8, D9: TVS 5.5V, SAMPI:SOT143B_NEXT, symbol SAM1:TVS_3CH
- added D1, D2, D3, D4, D5, D6: 5VZ, Liem:SOD-123FL_12, symbol SAMPI:TVS
Connections:
- net +5V_INV: now also OP1.1 (A); no longer R24.2
- net GND_INV: now also D1.2, D2.2, D3.2, D4.2, D5.2, D6.2
- net IPM_PWM_UH: now also D2.1
- net IPM_PWM_UL: now also U9.6 (VOB), D4.1; no longer U8.6 (VOB)
- net IPM_PWM_VH: now also U8.6 (VOB), D1.1; no longer U9.7 (VOA)
- net IPM_PWM_VL: now also U10.7 (VOA), D5.1; no longer U9.6 (VOB)
- net IPM_PWM_WH: now also U9.7 (VOA), D3.1; no longer U10.7 (VOA)
- net IPM_PWM_WL: now also D6.1
- net MC_PWM_UL: now also U9.3 (VIB); no longer U8.3 (VIB)
- net MC_PWM_VH: now also U8.3 (VIB); no longer U9.2 (VIA)
- net MC_PWM_VL: now also U10.2 (VIA); no longer U9.3 (VIB)
- net MC_PWM_WH: now also U9.2 (VIA); no longer U10.2 (VIA)
- net at R24.1: now also Q3.3 (D); no longer OP1.1 (A)
- net at OP1.2 (K): now also R24.2; no longer Q3.3 (D)
Other:
- moved on the sheet: D11, D12, D13, OP1, R18, R19, R20, R22, R24
