File: V1/Design/HW.ACIM-INV/Inverter.kicad_sch (KiCad schematic)
At the start: 75 parts, among them J16 HIGH VOLTAGE OUTPUTS, J2 U, J3 V, J4 W, J5 N, J6 U, J7 V, J8 W, J9 N, M5 560V/1.75kA, M6 560V/1.75kA, M7 560V/1.75kA, Q3 20V/1A, U1 I=±10A, U10 DIGI ISO, U11 I=±10A, U12 I=±10A, U13 CMP-1CH, U7 IPM 600V/15A, U8 DIGI ISO, U9 DIGI ISO

Commit message: V1 schematic update 27
Parts:
- added D7: PV, SAMPI:LED0603, symbol SAMPI:YLED
- added D8: PU, SAMPI:LED0603, symbol SAMPI:RLED
- added D9: PW, SAMPI:LED0603, symbol SAMPI:BLED
- added R4, R5, R6: 1K, SAMPI:RES0603, symbol SAMPI:RES
Connections:
- net GND_MCU: now also D7.K, D8.K, D9.K
- net MC_PWM_UL: now also R4.2
- net MC_PWM_VL: now also R5.2
- net MC_PWM_WL: now also R6.2
- new net: D7.A, R5.1
- new net: D9.A, R6.1
- new net: D8.A, R4.1
Other:
- moved on the sheet: D11, D12, D13, R18, R19, R20

Commit message: V1 schematic update 28
Parts:
- D11: value PV -> VH
- D12: value PW -> WH
- D13: value PU -> UH
- D7: value PV -> VL
- D8: value PU -> UL
- D9: value PW -> WL
Changed lines of the file:
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@@
 			)
 		)
-		(property "Value" "PV"
+		(property "Value" "VL"
 			(at 170.815 154.94 90)
 			(effects
@@
 			)
 		)
-		(property "Value" "PU"
+		(property "Value" "UL"
 			(at 161.29 154.94 90)
 			(effects
@@
 			)
 		)
-		(property "Value" "PU"
+		(property "Value" "UH"
 			(at 184.15 154.94 90)
 			(effects
@@
 		(pin "23"
 		)
-		(pin "24"
-		)
 		(pin "3"
 		)
@@
 			)
 		)
-		(property "Value" "PW"
+		(property "Value" "WL"
 			(at 178.435 154.94 90)
 			(effects
@@
 			)
 		)
-		(property "Value" "PV"
+		(property "Value" "VH"
 			(at 193.675 154.94 90)
 			(effects
@@
 			)
 		)
-		(property "Value" "PW"
+		(property "Value" "WH"
 			(at 201.295 154.94 90)
 			(effects

Commit message: Label & Case
Parts:
- C3, C38, C39, C4, C40, C41, C42, C43, C44, C45, C46, C47, C48, C49, C50, C51, C52, C53, C54, C55, C56, C57, C58, C59, C60, C61, C62, C63, C8, C88, D1, D11, D12, D13, D2, D3, D4, D5, D6, D7, D8, D9, FT1, G2, J2, J3, J4, J5, J6, J7, J8, J9, M5, M6, M7, OP1, Q3, R16, R18, R19, R20, R21, R22, R23, R24, R25, R26, R4, R5, R6, RV1, U1, U10, U11, U12, U13, U8, U9: now not fitted

Commit message: Update schematic
Parts:
- C3, C38, C39, C4, C40, C41, C42, C43, C44, C45, C46, C47, C48, C49, C50, C51, C52, C53, C54, C55, C56, C57, C58, C59, C60, C61, C62, C63, C8, C88, D1, D11, D12, D13, D2, D3, D4, D5, D6, D7, D8, D9, FT1, G2, J2, J3, J4, J5, J6, J7, J8, J9, M5, M6, M7, OP1, Q3, R16, R18, R19, R20, R21, R22, R23, R24, R25, R26, R4, R5, R6, RV1, U1, U10, U11, U12, U13, U8, U9: now fitted
- C9: now fitted; now in the parts list
