File: V1/Design/HW.ACIM-INV/ENCODER.kicad_sch (KiCad schematic)
At the start: 29 parts, among them J8 ENCODER, Q2 60V/265mA, Q7 60V/265mA, Q8 60V/265mA, Q9 60V/265mA, U17 DIGI ISO 2-CH, U19 DIGI ISO 2-CH

Commit message: V1 schematic update 2
Parts:
- removed R44, R56, R62, R67: 1.1K, SAMPI:RES0603, symbol SAMPI:RES
Connections:
- net ENC_A: now also Q8.3 (D), R65.2
- net ENC_B: now also Q9.3 (D), R70.2
- net HOME: now also Q2.3 (D), R55.2
- net INDEX: now also Q7.3 (D), R45.2

Commit message: V1 schematic update 4
Parts:
- removed C77, C80: 100nF, SAMPI:CAP0603, symbol SAMPI:CERCAP
- removed U17, U19: DIGI ISO 2-CH, SAMPI:SOIC8_ALL, symbol SAMPI:ADUM120N
- added U9: ISO6740, SAMPI:SOIC16-W, symbol SAMPI:ISO6740
Connections:
- net +3V3: now also U9.10 (EN2), U9.16 (VCC2)
- net ENC_A: now also U9.11 (OUTD)
- net ENC_B: now also U9.12 (OUTC)
- net ENC_HOME: now also U9.14 (OUTA)
- net ENC_INDEX: now also U9.13 (OUTB)
- net GND: now also U9.15 (GND2), U9.9 (GND2)
- net GND_ISO: now also U9.2 (GND1), U9.8 (GND1)
- net at Q2.2 (S), R61.2: now also U9.3 (INA)
- net at Q8.2 (S), R71.2: now also U9.6 (IND)
- net at Q7.2 (S), R46.2: now also U9.4 (INB)
- net at Q9.2 (S), R72.2: now also U9.5 (INC)
- net +3V3_ISO renamed +5V_ISO
- net +5V_ISO: now also U9.1 (VCC1)
Other:
- moved on the sheet: C36, C51, C52, C60, C82, C84, Q2, Q7, Q8, Q9, R45, R46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

Commit message: V1 schematic update 5
Parts:
- removed C73: 47uF/35V, SAMPI:CAP_ELEC-6.6x6.6-DIA6.3, symbol SAMPI:ELECCAP
- removed C82, C84: 100nF, SAMPI:CAP0603, symbol SAMPI:CERCAP
- added C73: 10uF, SAMPI:CAP0603, symbol SAMPI:CERCAP
- C74: value 100nF -> 10uF; MNP CL10B104KB8NNNC -> CL10A106MQ8NNNC; Unit Price 0.0146 -> 0.079
Connections:
- net +24V_ISO: no longer C74.2, J8.7
- net +3V3: now also C74.2
- net +5V_ISO: now also J8.7, C73.2
- net GND: now also C74.1
- net GND_ISO: now also C73.1; no longer C74.1
Other:
- note added: "ISOLATED POWER - SAFE-ZONE"
- note removed: "ISOLATED POWER SAFE-ZONE"
- moved on the sheet: J8

Commit message: V1 schematic update 6
Parts:
- C36, C51, C52, C60: Checked OK -> (none); Unit Price 0.012 -> (none)
- C73, C74: Checked OK -> (none); Unit Price 0.079 -> (none)
- J8: Checked OK -> (none); Unit Price 0.44 -> (none)
- R45, R46, R55, R61, R65, R70, R71, R72: Checked OK -> (none); Unit Price 0.021 -> (none)
Connections:
- net ENC_A: no longer J8.1, Q8.3 (D), R65.2
- net ENC_B: no longer J8.2, Q9.3 (D), R70.2
- new net PULSE_A: J8.1, Q8.3 (D), R65.2
- new net PULSE_B: J8.2, Q9.3 (D), R70.2

Commit message: V1 schematic update 8
Parts:
- added CB3: CABLE1, symbol SAMPI:CABLE1
Changed lines of the file:
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@@
 	)
 	(rectangle
-		(start 36.83 19.05)
+		(start 20.955 19.05)
 		(end 118.11 115.57)
 		(stroke
@@
 					(unit 1)
 				)
+			)
+		)
+	)
+	(symbol
+		(lib_id "SAMPI:CABLE1")
+		(at 33.655 32.385 0)
+		(mirror y)
+		(unit 1)
+		(exclude_from_sim no)
+		(in_bom yes)
+		(on_board no)
+		(dnp no)
+		(property "Reference" "CB3"
+			(at 28.575 37.4649 0)
+			(effects
+				(font
+					(size 1.5 1.5)
+					(bold yes)
+				)
+				(justify left)
+			)
+		)
+		(property "Value" "CABLE1"
+			(at 28.575 40.0049 0)
+			(effects
+				(font
+					(size 1.27 1.27)
+				)
+				(justify left)
+			)
+		)
+		(property "Footprint" ""
+			(at 33.655 32.385 0)
+			(effects
+				(font
+					(size 1.27 1.27)
+				)
+				(hide yes)
+			)
+		)
+		(property "Datasheet" ""
+			(at 33.655 32.385 0)
+			(effects
+				(font
+					(size 1.27 1.27)
+				)
+				(hide yes)
+			)
+		)
+		(property "Description" ""
+			(at 33.655 32.385 0)
+			(effects
+				(font
+					(size 1.27 1.27)
+				)
+				(hide yes)
+			)
+		)
+		(instances
+			(project "HW.ACIM-INV"
+				(path "/20f80521-75f2-4ccc-bb34-c9566e70ef5c/3b393387-96f5-4b8b-8a59-d8739719ea08"
+					(reference "CB3")
+					(unit 1)
+				)

Commit message: V1 schematic update 11
Parts:
- removed C73, C74: 10uF, SAMPI:CAP0603, symbol SAMPI:CERCAP
- removed U9: ISO6740, SAMPI:SOIC16-W, symbol SAMPI:ISO6740
- added C35: 10uF/35V, SAMPI:CAP0603, symbol SAMPI:CERCAP
- added D19, D23: TVS 5.5V 3-CH, SAMPI:SOT143B_NEXT, symbol SAM1:TVS_3CH
Connections:
- net +3V3: now also Q2.1 (G), Q7.1 (G), Q8.1 (G), Q9.1 (G), R46.1, R61.1, R71.1, R72.1, D19.4 (CH3), D23.4 (CH3)
- net ENC_A: now also Q8.2 (S), R71.2, D23.2 (CH1)
- net ENC_B: now also Q9.2 (S), R72.2, D23.3 (CH2)
- net ENC_HOME: now also Q2.2 (S), R61.2, D19.3 (CH2)
- net ENC_INDEX: now also Q7.2 (S), R46.2, D19.2 (CH1)
- net GND: now also J8.5, C35.1, D19.1 (GND), D23.1 (GND)
- net +24V_ISO renamed V_ENC
- net V_ENC: now also J8.6, C35.2; no longer J8.8
- removed net +5V_ISO: J8.7, Q2.1 (G), Q7.1 (G), Q8.1 (G), Q9.1 (G), R46.1, R61.1, R71.1, R72.1
- net CHASSIS renamed +24V
- removed net GND_ISO: J8.5, J8.6
- new net +12V: J8.8
- new net +5V: J8.7
Other:
- note removed: "ISOLATED POWER - SAFE-ZONE"
- moved on the sheet: C36, C51, C52, C60, CB3, J8, Q2, Q7, Q8, Q9, R45, R46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

Commit message: V1 schematic update 14
Parts:
- removed D19: TVS 5.5V 3-CH, SAMPI:SOT143B_NEXT, symbol SAM1:TVS_3CH
- added D10: TVS 5.5V 3-CH, SAMPI:SOT143B_NEXT, symbol SAM1:TVS_3CH
Connections:
- net ENC_HOME: now also D10.3 (CH2)
- net ENC_INDEX: now also D10.2 (CH1)
- net +12V renamed +12V_MCU
- net +24V renamed +24V_MCU
- net +3V3 renamed +3V3_MCU
- net +3V3_MCU: now also D10.4 (CH3)
- net +5V renamed +5V_MCU
- net GND renamed GND_MCU
- net GND_MCU: now also D10.1 (GND)
Other:
- moved on the sheet: CB3, J8

Commit message: V1 schematic update 15
Other:
- company: TON DUC THANG UNIVERSITY -> (none)
Changed lines of the file:
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@@
 		(date "2024-09-24")
 		(rev "1.0")
-		(company "TON DUC THANG UNIVERSITY")
-		(comment 1 "Schematic Designed by ...")
-		(comment 2 "PCB Designed by ...")
-		(comment 3 "Approved by ...")
 	)
 	(junction
