File: V1/Design/HW.ACIM-INV/ENCODER.kicad_sch (KiCad schematic)
At the start: 21 parts, among them J8 ENCODER, Q2 60V/265mA, Q7 60V/265mA, Q8 60V/265mA, Q9 60V/265mA

Commit message: V1 schematic update 16
Parts:
- C35: footprint SAMPI:CAP0603 -> SAMPI:CAP1206; MFT Samsung -> (none); MNP CL10A106MQ8NNNC -> (none)
- R45, R46, R55, R61, R65, R70, R71, R72: value 4.3K -> 2.2K; MFT YAGEO -> (none); MNP AC0603FR-074K3L -> (none)

Commit message: V1 schematic update 17
Parts:
- added J10: ENCODER PORT, symbol SAMPI:FREE_HANGING_CONN
- C83: renamed from C35; MFT (none) -> Murata; MNP (none) -> GRT31CR6YA106ME01L
- CB2: renamed from CB3; value CABLE1 -> ENCODER CABLE; MFT (none) -> OEM; MNP (none) -> PH2.0-1x8-1-20CM
- D19: renamed from D10; value TVS 5.5V 3-CH -> TVS 5.5V
- D20: renamed from D23; value TVS 5.5V 3-CH -> TVS 5.5V
- Q4: renamed from Q2; MFT Nexperia USA Inc. -> Nexperia
- Q5: renamed from Q7; MFT Nexperia USA Inc. -> Nexperia
- Q6: renamed from Q9; MFT Nexperia USA Inc. -> Nexperia
- Q7: renamed from Q8; MFT Nexperia USA Inc. -> Nexperia
- R51: renamed from R55; MFT (none) -> YAGEO; MNP (none) -> RC0603JR-132K2L
- R52: renamed from R45; MFT (none) -> YAGEO; MNP (none) -> RC0603JR-132K2L
- R53: renamed from R70; MFT (none) -> YAGEO; MNP (none) -> RC0603JR-132K2L
- R54: renamed from R65; MFT (none) -> YAGEO; MNP (none) -> RC0603JR-132K2L
- R55: renamed from R61; MFT (none) -> YAGEO; MNP (none) -> RC0603JR-132K2L
- R56: renamed from R46; MFT (none) -> YAGEO; MNP (none) -> RC0603JR-132K2L
- R57: renamed from R72; MFT (none) -> YAGEO; MNP (none) -> RC0603JR-132K2L
- R58: renamed from R71; MFT (none) -> YAGEO; MNP (none) -> RC0603JR-132K2L
- renumbered C36 to C84, C60 to C85, C52 to C86, C51 to C87, J8 to J11
Connections:
- net +5V_MCU is gone; now on net +12V_MCU: J11.7
- net +12V_MCU: no longer J11.8
- net +24V_MCU: now also J11.8; no longer J11.9
- net GND_MCU: now also J11.9
Other:
- moved on the sheet: C83, C84, C85, C86, C87, CB2, D19, D20, Q4, Q5, Q6, Q7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

Commit message: V1 schematic update 18
Parts:
- added Q1, Q2, Q8, Q9: 60V/265mA, SAMPI:SOT23, symbol SAMPI:FET_N-CH
Connections:
- net HOME: now also Q9.2 (S); no longer Q4.3 (D)
- net INDEX: now also Q8.2 (S); no longer Q5.3 (D)
- net PULSE_A: now also Q1.2 (S); no longer Q7.3 (D)
- net PULSE_B: now also Q2.2 (S); no longer Q6.3 (D)
- net V_ENC: now also Q1.1 (G), Q2.1 (G), Q8.1 (G), Q9.1 (G)
- new net: Q4.3 (D), Q9.3 (D)
- new net: Q1.3 (D), Q7.3 (D)
- new net: Q2.3 (D), Q6.3 (D)
- new net: Q5.3 (D), Q8.3 (D)
Other:
- moved on the sheet: C84, C85, C86, C87, D19, D20, Q4, Q5, Q6, Q7, R55, R56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

Commit message: V1 schematic update 20
Parts:
- added C1, C2: 10uF/35V, SAMPI:CAP1206, symbol SAMPI:CERCAP
Connections:
- net +12V_MCU: now also J11.2, C2.2; no longer J11.7
- net +24V_MCU: now also J11.1, C1.2; no longer J11.8
- net GND_MCU: now also J11.4, C1.1, C2.1; no longer J11.5
- net HOME: now also J11.5; no longer J11.4
- net INDEX: now also J11.6; no longer J11.3
- net PULSE_A: now also J11.8; no longer J11.1
- net PULSE_B: now also J11.7; no longer J11.2
- net V_ENC: now also J11.3; no longer J11.6
Other:
- moved on the sheet: CB2, J10, J11

Commit message: V1 schematic update 23
Connections:
- net ENC_A: now also D20.3 (CH2); no longer D20.2 (CH1)
- net ENC_B: now also D20.2 (CH1); no longer D20.3 (CH2)
- net ENC_HOME: now also D19.2 (CH1); no longer D19.3 (CH2)
- net ENC_INDEX: now also D19.3 (CH2); no longer D19.2 (CH1)
Changed lines of the file:
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@@
-	)
-	(junction
-		(at 149.86 140.97)
-		(diameter 0)
-		(color 0 0 0 0)
-	)
-	(junction
-		(at 152.4 109.22)
-		(diameter 0)
-		(color 0 0 0 0)
 	)
 	(junction
@@
 	)
 	(junction
+		(at 152.4 140.97)
+		(diameter 0)
+		(color 0 0 0 0)
+	)
+	(junction
 		(at 109.855 140.97)
 		(diameter 0)
@@
 	)
 	(junction
+		(at 149.86 45.72)
+		(diameter 0)
+		(color 0 0 0 0)
+	)
+	(junction
 		(at 139.7 130.81)
 		(diameter 0)
@@
 	)
 	(junction
+		(at 152.4 77.47)
+		(diameter 0)
+		(color 0 0 0 0)
+	)
+	(junction
 		(at 109.855 45.72)
 		(diameter 0)
@@
 	)
 	(junction
-		(at 149.86 77.47)
-		(diameter 0)
-		(color 0 0 0 0)
-	)
-	(junction
 		(at 109.855 77.47)
 		(diameter 0)
@@
 	)
 	(junction
-		(at 152.4 45.72)
+		(at 149.86 109.22)
 		(diameter 0)
 		(color 0 0 0 0)
@@
 	(wire
 		(pts
-			(xy 156.21 45.72) (xy 152.4 45.72)
+			(xy 139.7 45.72) (xy 149.86 45.72)
 		)
 		(stroke
@@
 	(wire
 		(pts
-			(xy 149.86 140.97) (xy 139.7 140.97)
+			(xy 139.7 140.97) (xy 152.4 140.97)
 		)
 		(stroke
@@
 	(wire
 		(pts
-			(xy 149.86 140.97) (xy 149.86 142.24)
-		)
-		(stroke
-			(width 0)
-			(type default)
-		)
-	)
-	(wire
-		(pts
 			(xy 98.425 99.06) (xy 109.855 99.06)
 		)
@@
 	(wire
 		(pts
+			(xy 149.86 45.72) (xy 149.86 78.74)
+		)
+		(stroke
+			(width 0)
+			(type default)
+		)
+	)
+	(wire
+		(pts
 			(xy 132.08 137.16) (xy 132.08 130.81)
 		)
@@
 	(wire
 		(pts
-			(xy 152.4 109.22) (xy 139.7 109.22)
+			(xy 139.7 109.22) (xy 149.86 109.22)
 		)
 		(stroke
@@
 	(wire
 		(pts
-			(xy 152.4 45.72) (xy 152.4 78.74)
-		)
-		(stroke
-			(width 0)
-			(type default)
-		)
-	)
-	(wire
-		(pts
 			(xy 98.425 130.81) (xy 109.855 130.81)
 		)
@@
 	(wire
 		(pts
+			(xy 149.86 109.22) (xy 156.21 109.22)
+		)
+		(stroke
+			(width 0)
+			(type default)
+		)
+	)
+	(wire
+		(pts
+			(xy 149.86 109.22) (xy 149.86 142.24)
+		)
+		(stroke
+			(width 0)
+			(type default)
+		)
+	)
+	(wire
+		(pts
 			(xy 134.62 109.22) (xy 139.7 109.22)
 		)
@@
 	(wire
 		(pts
-			(xy 156.21 109.22) (xy 152.4 109.22)
-		)
-		(stroke
-			(width 0)
-			(type default)
-		)
-	)
-	(wire
-		(pts
 			(xy 134.62 45.72) (xy 139.7 45.72)
 		)
@@
 	(wire
 		(pts
-			(xy 152.4 109.22) (xy 152.4 142.24)
+			(xy 149.86 45.72) (xy 156.21 45.72)
 		)
 		(stroke
@@
 	(wire
 		(pts
-			(xy 149.86 77.47) (xy 149.86 78.74)
+			(xy 152.4 140.97) (xy 152.4 142.24)
 		)
 		(stroke
@@
 	(wire
 		(pts
-			(xy 149.86 77.47) (xy 139.7 77.47)
-		)
-		(stroke
-			(width 0)
-			(type default)
-		)
-	)
-	(wire
-		(pts
 			(xy 139.7 99.06) (xy 139.7 100.33)
 		)
@@
 	(wire
 		(pts
-			(xy 152.4 45.72) (xy 139.7 45.72)
-		)
-		(stroke
-			(width 0)
-			(type default)
-		)
-	)
-	(wire
-		(pts
 			(xy 132.08 105.41) (xy 132.08 99.06)
 		)
@@
 	(wire
 		(pts
+			(xy 152.4 77.47) (xy 152.4 78.74)
+		)
+		(stroke
+			(width 0)
+			(type default)
+		)
+	)
+	(wire
+		(pts
 			(xy 108.585 77.47) (xy 109.855 77.47)
 		)
@@
 	(wire
 		(pts
+			(xy 139.7 77.47) (xy 152.4 77.47)
+		)
+		(stroke
+			(width 0)
+			(type default)
+		)
+	)
+	(wire
+		(pts
 			(xy 98.425 130.81) (xy 98.425 132.08)
 		)
@@
 	(wire
 		(pts
-			(xy 156.21 77.47) (xy 149.86 77.47)
+			(xy 156.21 77.47) (xy 152.4 77.47)
 		)
 		(stroke
@@
 	(wire
 		(pts
-			(xy 156.21 140.97) (xy 149.86 140.97)
-		)
-		(stroke
+			(xy 156.21 140.97) (xy 152.4 140.97)
+		)
+		(stroke

Commit message: Label & Case
Parts:
- C1, C2, C83, C84, C85, C86, C87, CB2, D19, D20, J10, J11, Q1, Q2, Q4, Q5, Q6, Q7, Q8, Q9, R51, R52, R53, R54, R55, R56, R57, R58: now not fitted
Changed lines of the file:
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@@
 (kicad_sch
-	(version 20231120)
+	(version 20250114)
 	(generator "eeschema")
-	(generator_version "8.0")
+	(generator_version "9.0")
 	(paper "A4")
 	(title_block
@@
 		(in_bom yes)
 		(on_board yes)
-		(dnp no)
+		(dnp yes)
 		(property "Reference" "Q9"
 			(at 118.11 40.64 90)
@@
 		(in_bom yes)
 		(on_board yes)
-		(dnp no)
+		(dnp yes)
 		(property "Reference" "C2"
 			(at 73.66 139.6999 90)
@@
 		(in_bom yes)
 		(on_board yes)
-		(dnp no)
+		(dnp yes)
 		(fields_autoplaced yes)
 		(property "Reference" "C86"
@@
 		(in_bom yes)
 		(on_board yes)
-		(dnp no)
+		(dnp yes)
 		(property "Reference" "R55"
 			(at 136.525 39.37 90)
@@
 		(in_bom yes)
 		(on_board yes)
-		(dnp no)
+		(dnp yes)
 		(fields_autoplaced yes)
 		(property "Reference" "C84"
@@
 		(in_bom yes)
 		(on_board yes)
-		(dnp no)
+		(dnp yes)
 		(property "Reference" "Q7"
 			(at 129.54 135.89 90)
@@
 		(in_bom yes)
 		(on_board yes)
-		(dnp no)
+		(dnp yes)
 		(property "Reference" "R52"
 			(at 106.68 71.12 90)
@@
 		(in_bom yes)
 		(on_board yes)
-		(dnp no)
+		(dnp yes)
 		(property "Reference" "R56"
 			(at 136.525 71.12 90)
@@
 		(in_bom yes)
 		(on_board yes)
-		(dnp no)
+		(dnp yes)
 		(property "Reference" "#PWR05"
 			(at 76.2 151.13 0)
@@
 		(in_bom yes)
 		(on_board yes)
-		(dnp no)
+		(dnp yes)
 		(property "Reference" "Q6"
 			(at 129.54 104.14 90)
@@
 		(in_bom yes)
 		(on_board yes)
-		(dnp no)
+		(dnp yes)
 		(property "Reference" "R53"
 			(at 106.68 102.87 90)
@@
 		(in_bom yes)
 		(on_board yes)
-		(dnp no)
+		(dnp yes)
 		(property "Reference" "#PWR0180"
 			(at 139.7 92.71 0)
@@
 		(in_bom yes)
 		(on_board yes)
-		(dnp no)
+		(dnp yes)
 		(property "Reference" "C1"
 			(at 62.23 139.6999 90)
@@
 		(in_bom yes)
 		(on_board yes)
-		(dnp no)
+		(dnp yes)
 		(property "Reference" "#PWR0179"
 			(at 139.7 69.85 0)
@@
 		(in_bom yes)
 		(on_board yes)
-		(dnp no)
+		(dnp yes)
 		(property "Reference" "#PWR0173"
 			(at 73.66 133.35 0)
@@
 		(in_bom yes)
 		(on_board yes)
-		(dnp no)
+		(dnp yes)
 		(property "Reference" "#PWR0186"
 			(at 152.4 156.21 0)
@@
 		(in_bom yes)
 		(on_board yes)
-		(dnp no)
+		(dnp yes)
 		(property "Reference" "D20"
 			(at 156.845 144.78 0)
@@
 		(in_bom yes)
 		(on_board yes)
-		(dnp no)
+		(dnp yes)
 		(property "Reference" "C83"
 			(at 95.885 134.6199 90)
@@
 		(in_bom yes)
 		(on_board yes)
-		(dnp no)
+		(dnp yes)
 		(property "Reference" "#PWR0176"
 			(at 98.425 146.05 0)
@@
 		(in_bom yes)
 		(on_board yes)
-		(dnp no)
+		(dnp yes)
 		(property "Reference" "R51"
 			(at 106.68 39.37 90)
@@
 		(in_bom yes)
 		(on_board yes)
-		(dnp no)
+		(dnp yes)
 		(property "Reference" "D19"
 			(at 156.845 81.28 0)
@@
 		(in_bom yes)
 		(on_board no)
-		(dnp no)
+		(dnp yes)
 		(property "Reference" "CB2"
 			(at 45.72 120.65 90)
@@
 		(in_bom yes)
 		(on_board yes)
-		(dnp no)
+		(dnp yes)
 		(property "Reference" "#PWR0178"
 			(at 139.7 60.96 0)
@@
 		(in_bom yes)
 		(on_board yes)
-		(dnp no)
+		(dnp yes)
 		(property "Reference" "#PWR0181"
 			(at 139.7 101.6 0)
@@
 		(in_bom yes)
 		(on_board yes)
-		(dnp no)
+		(dnp yes)
 		(property "Reference" "#PWR0182"
 			(at 139.7 124.46 0)
@@
 		(in_bom yes)
 		(on_board yes)
-		(dnp no)
+		(dnp yes)
 		(property "Reference" "#PWR0183"
 			(at 139.7 133.35 0)
@@
 		(in_bom yes)
 		(on_board yes)
-		(dnp no)
+		(dnp yes)
 		(property "Reference" "#PWR04"
 			(at 64.77 151.13 0)
@@
 		(in_bom yes)
 		(on_board yes)
-		(dnp no)
+		(dnp yes)
 		(property "Reference" "Q1"
 			(at 118.11 135.89 90)
@@
 		(in_bom yes)
 		(on_board yes)
-		(dnp no)
+		(dnp yes)
 		(fields_autoplaced yes)
 		(property "Reference" "C85"
@@
 		(in_bom yes)
 		(on_board yes)
-		(dnp no)
+		(dnp yes)
 		(property "Reference" "R58"
 			(at 136.525 134.62 90)
@@
 		(in_bom yes)
 		(on_board yes)
-		(dnp no)
+		(dnp yes)
 		(property "Reference" "J11"
 			(at 55.245 125.73 0)
@@
 		(in_bom yes)
 		(on_board yes)
-		(dnp no)
+		(dnp yes)
 		(property "Reference" "R54"
 			(at 106.68 134.62 90)
@@
 		(in_bom yes)
 		(on_board yes)
-		(dnp no)
+		(dnp yes)
 		(property "Reference" "#PWR0185"
 			(at 152.4 92.71 0)
@@
 		(in_bom yes)
 		(on_board yes)
-		(dnp no)
+		(dnp yes)
 		(property "Reference" "R57"
 			(at 136.525 102.87 90)
@@
 		(in_bom yes)
 		(on_board no)
-		(dnp no)
+		(dnp yes)
 		(property "Reference" "J10"
 			(at 33.02 126.3649 90)
@@
 		(in_bom yes)
 		(on_board yes)
-		(dnp no)
+		(dnp yes)
 		(property "Reference" "Q8"
 			(at 118.11 72.39 90)
@@
 		(in_bom yes)
 		(on_board yes)
-		(dnp no)
+		(dnp yes)
 		(fields_autoplaced yes)
 		(property "Reference" "C87"
@@
 		(in_bom yes)
 		(on_board yes)
-		(dnp no)
+		(dnp yes)
 		(property "Reference" "Q4"
 			(at 129.54 40.64 90)
@@
 		(in_bom yes)
 		(on_board yes)
-		(dnp no)
+		(dnp yes)
 		(property "Reference" "Q5"
 			(at 129.54 72.39 90)
@@
 		(in_bom yes)
 		(on_board yes)
-		(dnp no)
+		(dnp yes)
 		(property "Reference" "#PWR0175"
 			(at 69.85 115.57 0)
@@
 		(in_bom yes)
 		(on_board yes)
-		(dnp no)
+		(dnp yes)
 		(property "Reference" "#PWR0177"
 			(at 139.7 38.1 0)
@@
 		(in_bom yes)
 		(on_board yes)
-		(dnp no)
+		(dnp yes)
 		(property "Reference" "#PWR0172"
 			(at 69.85 128.27 0)
@@
 		(in_bom yes)
 		(on_board yes)
-		(dnp no)
+		(dnp yes)
 		(property "Reference" "Q2"
 			(at 118.11 104.14 90)
@@
 		(in_bom yes)
 		(on_board yes)
-		(dnp no)
+		(dnp yes)
 		(property "Reference" "#PWR0174"
 			(at 73.66 135.89 0)
@@
 		(in_bom yes)
 		(on_board yes)
-		(dnp no)
+		(dnp yes)
 		(property "Reference" "#PWR0184"
 			(at 139.7 156.21 0)

Commit message: Update schematic
Parts:
- C1, C2, C83, C84, C85, C86, C87, CB2, D19, D20, J10, J11, Q1, Q2, Q4, Q5, Q6, Q7, Q8, Q9, R51, R52, R53, R54, R55, R56, R57, R58: now fitted
Changed lines of the file:
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@@
 		(in_bom yes)
 		(on_board yes)
-		(dnp yes)
+		(dnp no)
 		(property "Reference" "Q9"
 			(at 118.11 40.64 90)
@@
 		(in_bom yes)
 		(on_board yes)
-		(dnp yes)
+		(dnp no)
 		(property "Reference" "C2"
 			(at 73.66 139.6999 90)
@@
 		(in_bom yes)
 		(on_board yes)
-		(dnp yes)
+		(dnp no)
 		(fields_autoplaced yes)
 		(property "Reference" "C86"
@@
 		(in_bom yes)
 		(on_board yes)
-		(dnp yes)
+		(dnp no)
 		(property "Reference" "R55"
 			(at 136.525 39.37 90)
@@
 		(in_bom yes)
 		(on_board yes)
-		(dnp yes)
+		(dnp no)
 		(fields_autoplaced yes)
 		(property "Reference" "C84"
@@
 		(in_bom yes)
 		(on_board yes)
-		(dnp yes)
+		(dnp no)
 		(property "Reference" "Q7"
 			(at 129.54 135.89 90)
@@
 		(in_bom yes)
 		(on_board yes)
-		(dnp yes)
+		(dnp no)
 		(property "Reference" "R52"
 			(at 106.68 71.12 90)
@@
 		(in_bom yes)
 		(on_board yes)
-		(dnp yes)
+		(dnp no)
 		(property "Reference" "R56"
 			(at 136.525 71.12 90)
@@
 		(in_bom yes)
 		(on_board yes)
-		(dnp yes)
+		(dnp no)
 		(property "Reference" "#PWR05"
 			(at 76.2 151.13 0)
@@
 		(in_bom yes)
 		(on_board yes)
-		(dnp yes)
+		(dnp no)
 		(property "Reference" "Q6"
 			(at 129.54 104.14 90)
@@
 		(in_bom yes)
 		(on_board yes)
-		(dnp yes)
+		(dnp no)
 		(property "Reference" "R53"
 			(at 106.68 102.87 90)
@@
 		(in_bom yes)
 		(on_board yes)
-		(dnp yes)
+		(dnp no)
 		(property "Reference" "#PWR0180"
 			(at 139.7 92.71 0)
@@
 		(in_bom yes)
 		(on_board yes)
-		(dnp yes)
+		(dnp no)
 		(property "Reference" "C1"
 			(at 62.23 139.6999 90)
@@
 		(in_bom yes)
 		(on_board yes)
-		(dnp yes)
+		(dnp no)
 		(property "Reference" "#PWR0179"
 			(at 139.7 69.85 0)
@@
 		(in_bom yes)
 		(on_board yes)
-		(dnp yes)
+		(dnp no)
 		(property "Reference" "#PWR0173"
 			(at 73.66 133.35 0)
@@
 		(in_bom yes)
 		(on_board yes)
-		(dnp yes)
+		(dnp no)
 		(property "Reference" "#PWR0186"
 			(at 152.4 156.21 0)
@@
 		(in_bom yes)
 		(on_board yes)
-		(dnp yes)
+		(dnp no)
 		(property "Reference" "D20"
 			(at 156.845 144.78 0)
@@
 		(in_bom yes)
 		(on_board yes)
-		(dnp yes)
+		(dnp no)
 		(property "Reference" "C83"
 			(at 95.885 134.6199 90)
@@
 		(in_bom yes)
 		(on_board yes)
-		(dnp yes)
+		(dnp no)
 		(property "Reference" "#PWR0176"
 			(at 98.425 146.05 0)
@@
 		(in_bom yes)
 		(on_board yes)
-		(dnp yes)
+		(dnp no)
 		(property "Reference" "R51"
 			(at 106.68 39.37 90)
@@
 		(in_bom yes)
 		(on_board yes)
-		(dnp yes)
+		(dnp no)
 		(property "Reference" "D19"
 			(at 156.845 81.28 0)
@@
 		(in_bom yes)
 		(on_board no)
-		(dnp yes)
+		(dnp no)
 		(property "Reference" "CB2"
 			(at 45.72 120.65 90)
@@
 		(in_bom yes)
 		(on_board yes)
-		(dnp yes)
+		(dnp no)
 		(property "Reference" "#PWR0178"
 			(at 139.7 60.96 0)
@@
 		(in_bom yes)
 		(on_board yes)
-		(dnp yes)
+		(dnp no)
 		(property "Reference" "#PWR0181"
 			(at 139.7 101.6 0)
@@
 		(in_bom yes)
 		(on_board yes)
-		(dnp yes)
+		(dnp no)
 		(property "Reference" "#PWR0182"
 			(at 139.7 124.46 0)
@@
 		(in_bom yes)
 		(on_board yes)
-		(dnp yes)
+		(dnp no)
 		(property "Reference" "#PWR0183"
 			(at 139.7 133.35 0)
@@
 		(in_bom yes)
 		(on_board yes)
-		(dnp yes)
+		(dnp no)
 		(property "Reference" "#PWR04"
 			(at 64.77 151.13 0)
@@
 		(in_bom yes)
 		(on_board yes)
-		(dnp yes)
+		(dnp no)
 		(property "Reference" "Q1"
 			(at 118.11 135.89 90)
@@
 		(in_bom yes)
 		(on_board yes)
-		(dnp yes)
+		(dnp no)
 		(fields_autoplaced yes)
 		(property "Reference" "C85"
@@
 		(in_bom yes)
 		(on_board yes)
-		(dnp yes)
+		(dnp no)
 		(property "Reference" "R58"
 			(at 136.525 134.62 90)
@@
 		(in_bom yes)
 		(on_board yes)
-		(dnp yes)
+		(dnp no)
 		(property "Reference" "J11"
 			(at 55.245 125.73 0)
@@
 		(in_bom yes)
 		(on_board yes)
-		(dnp yes)
+		(dnp no)
 		(property "Reference" "R54"
 			(at 106.68 134.62 90)
@@
 		(in_bom yes)
 		(on_board yes)
-		(dnp yes)
+		(dnp no)
 		(property "Reference" "#PWR0185"
 			(at 152.4 92.71 0)
@@
 		(in_bom yes)
 		(on_board yes)
-		(dnp yes)
+		(dnp no)
 		(property "Reference" "R57"
 			(at 136.525 102.87 90)
@@
 		(in_bom yes)
 		(on_board no)
-		(dnp yes)
+		(dnp no)
 		(property "Reference" "J10"
 			(at 33.02 126.3649 90)
@@
 		(in_bom yes)
 		(on_board yes)
-		(dnp yes)
+		(dnp no)
 		(property "Reference" "Q8"
 			(at 118.11 72.39 90)
@@
 		(in_bom yes)
 		(on_board yes)
-		(dnp yes)
+		(dnp no)
 		(fields_autoplaced yes)
 		(property "Reference" "C87"
@@
 		(in_bom yes)
 		(on_board yes)
-		(dnp yes)
+		(dnp no)
 		(property "Reference" "Q4"
 			(at 129.54 40.64 90)
@@
 		(in_bom yes)
 		(on_board yes)
-		(dnp yes)
+		(dnp no)
 		(property "Reference" "Q5"
 			(at 129.54 72.39 90)
@@
 		(in_bom yes)
 		(on_board yes)
-		(dnp yes)
+		(dnp no)
 		(property "Reference" "#PWR0175"
 			(at 69.85 115.57 0)
@@
 		(in_bom yes)
 		(on_board yes)
-		(dnp yes)
+		(dnp no)
 		(property "Reference" "#PWR0177"
 			(at 139.7 38.1 0)
@@
 		(in_bom yes)
 		(on_board yes)
-		(dnp yes)
+		(dnp no)
 		(property "Reference" "#PWR0172"
 			(at 69.85 128.27 0)
@@
 		(in_bom yes)
 		(on_board yes)
-		(dnp yes)
+		(dnp no)
 		(property "Reference" "Q2"
 			(at 118.11 104.14 90)
@@
 		(in_bom yes)
 		(on_board yes)
-		(dnp yes)
+		(dnp no)
 		(property "Reference" "#PWR0174"
 			(at 73.66 135.89 0)
@@
 		(in_bom yes)
 		(on_board yes)
-		(dnp yes)
+		(dnp no)
 		(property "Reference" "#PWR0184"
 			(at 139.7 156.21 0)
