File: V1/Design/HW.ACIM-INV/MCU.kicad_sch (KiCad schematic)
At the start: 44 parts, among them J9 USB, U11 256Kbit EEPROM, U13 128Mbit Flash, U5 MIPS 32-bit DSC, U6 12MHz (3225), X1 32.768kHz

Commit message: V1 schematic update 1
Parts:
- removed C100, C35, C89, C93, C94, C95, C96: 100nF, SAMPI:CAP0603, symbol SAMPI:CERCAP
- removed C101, C97: 22pF, SAMPI:CAP0603, symbol SAMPI:CERCAP
- removed C98, C99: 9pF, SAMPI:CAP0603, symbol SAMPI:CERCAP
- removed FT4: 2x 120R@100MHz, SAMPI:IND1210_4P, symbol SAMPI:IND1210_4P
- removed R110: 100K, SAMPI:RES0603, symbol SAMPI:RES
- removed R111: 0R, SAMPI:RES0603, symbol SAMPI:RES
- removed U13: 128Mbit Flash, SAMPI:SO8W_5.3, symbol SAMPI:SPI_MEM
- removed U5: MIPS 32-bit DSC, SAMPI:TQFP64_10x10_MCHP, symbol SAMPI:PIC32MKxxxxMCM064
- removed U6: 12MHz (3225), SAMPI:CDFN3225-4LD-PL-1, symbol SAMPI:OSC
- removed X1: 32.768kHz, SAMPI:SMD4-7015, symbol SAMPI:XTAL-4P
- added MD2: ACIM-MCU, SAMPI:HW.ACIM-MCU, symbol SAMPI:HW.ACIM-MCU
Connections:
- net VBUS: no longer TP23.1
Other:
- note removed: "(CH0)"
- note removed: "(CH1)"
- note removed: "(CH2)"
- note removed: "(CH3)"
- note removed: "(CH4)"
- note removed: "(CH5)"
- moved on the sheet: J9

Commit message: V1 schematic update 2
Parts:
- removed C43, C44, C45, C46, C47, C69, C70, C71, C72, C90, C91: 22pF, SAMPI:CAP0603, symbol SAMPI:CERCAP
- removed C92: 10uF, SAMPI:CAP0603, symbol SAMPI:CERCAP
- removed FT6: 120R@100MHz, SAMPI:FT0603, symbol SAMPI:FerriteBead
- removed TP1: TEMP, SAMPI:TP1MM, symbol SAMPI:TESTPOINT
- removed TP2: IU, SAMPI:TP1MM, symbol SAMPI:TESTPOINT
- removed TP3: IV, SAMPI:TP1MM, symbol SAMPI:TESTPOINT
- removed TP4: IW, SAMPI:TP1MM, symbol SAMPI:TESTPOINT
- removed TP5: IS, SAMPI:TP1MM, symbol SAMPI:TESTPOINT
- removed TP6: VS, SAMPI:TP1MM, symbol SAMPI:TESTPOINT
- removed TP7: VU, SAMPI:TP1MM, symbol SAMPI:TESTPOINT
- removed TP8: VV, SAMPI:TP1MM, symbol SAMPI:TESTPOINT
- removed TP9: VW, SAMPI:TP1MM, symbol SAMPI:TESTPOINT
- added BT1: UBT, SAMPI:HDM-2x2.54-TH, symbol SAMPI:BT3
- added BZ1: BUZZER, SAMPI:SMT-0827-S-HT-R, symbol SAMPI:BUZZER
- added C31: 1nF, SAMPI:CAP0603, symbol SAMPI:CERCAP
- added C33, C35: 22pF, SAMPI:CAP0603, symbol SAMPI:CERCAP
- added D4: 75V/150mA, SAMPI:SOD-323, symbol SAMPI:DIODE-REC
- added D6: ERR, SAMPI:LED0603, symbol SAMPI:RLED
- added D7: RUN, SAMPI:LED0603, symbol SAMPI:GLED
- added D8: PWR, SAMPI:LED0603, symbol SAMPI:WLED
- added Q3: 20V/1A, SAMPI:SOT23, symbol SAMPI:FET_N-CH
- added R4: 10R, SAMPI:RES0603, symbol SAMPI:RES
- added R44, R47, R5, R74: 1.1K, SAMPI:RES0603, symbol SAMPI:RES
- added R48: 10K, SAMPI:RES0603, symbol SAMPI:RES
- added R6: 100K, SAMPI:RES0603, symbol SAMPI:RES
- added RV1: 10K, Liem:HDM-3x2.54-TH, symbol SAMPI:POT
- U11: value 256Kbit EEPROM -> 2Mbit SRAM; MFT ST -> Microchip Technology; MNP M95256-WMN6P -> 23AA02M-I/SN
Connections:
- net USB_D+ is gone; now on net USB_P: J9.3
- net USB_D- is gone; now on net USB_N: J9.2
- net ~{MEM_TMP} is gone; now on net ~{SRAM_CS}: U11.1 (~{CE})
- net +3V3: now also MD2.27R (+3V3), MD2.28R (+3V3), D8.A, R48.1
- net AGND: now also MD2.1L (AGND), MD2.2L (AVDD), C31.1, RV1.3 (CW)
- net ENC_A: now also MD2.28L (ENC_A)
- net ENC_B: now also MD2.30L (ENC_B)
- net ENC_HOME: now also MD2.27L (ENC_HOME)
- net ENC_INDEX: now also MD2.29L (ENC_IDX)
- net GND: now also MD2.29R (GND), MD2.30R (GND), MD2.5L (GND), MD2.6L (GND), BT1.2, BZ1.1 (NC1), BZ1.4 (NC2), C33.1, C35.1, Q3.2 (S), R44.2, R47.2, R6.2
- net IND_ERR: now also MD2.8L (IO2), Q3.1 (G), R6.1
- net IND_RUN: now also MD2.7L (IO1), D7.A
- net MC_PWM_UH: now also MD2.19R (MC_PWM_UH)
- net MC_PWM_UL: now also MD2.20R (MC_PWM_UL)
- net MC_PWM_VH: now also MD2.17R (MC_PWM_VH)
- net MC_PWM_VL: now also MD2.16R (MC_PWM_WL)
- net MC_PWM_WH: now also MD2.15R (MC_PWM_WH)
- net MC_PWM_WL: now also MD2.18R (MC_PWM_VL)
- net PGC: now also MD2.4R (PGC)
- net PGD: now also MD2.2R (PGD)
- net RXD1: now also MD2.7R (DB_RXD)
- net RXD2: now also MD2.9R (DV_RXD)
- net SCK: now also MD2.15L (SCK)
- net SDI: now also MD2.16L (SDI)
- net SDO: now also MD2.14L (SDO)
- net TXD1: now also MD2.8R (DB_TXD)
- net TXD2: now also MD2.10R (DV_TXD)
- net VBUS: now also MD2.1R (VBUS), TP23.1, C35.2, R74.2; no longer J9.1
- net ~{BT_UBT}: now also MD2.14R (~{BUTTON}), BT1.1, C33.2, R48.2
- net ~{MCLR}: now also MD2.6R (~{MCLR})
- net DEV_RELAY: now reaches MD2.10L (DEV_RELAY)
- net ~{SRAM_CS}: now reaches MD2.13L (~{CS})
- net PFC_PWM_ENB: now reaches MD2.17L (PFC_PWM_ENB)
- net PFC_PWM_B: now reaches MD2.18L (PFC_PWM_B)
- net PFC_PWM_ENA: now reaches MD2.19L (PFC_PWM_ENA)
- net PFC_PWM_A: now reaches MD2.20L (PFC_PWM_A)
- net PFC_VAC_DIV: now reaches MD2.21L (VAC_DIV)
- net ~{PFC_FLT}: now reaches MD2.22L (~{PFC_FLT})
- net PFC_VDC_DIV: now reaches MD2.23L (VDC_DIV)
- net PFC_IB_SEN: now reaches MD2.24L (PFC_IB_SEN)
- net PFC_IDC_SEN: now reaches MD2.25L (IDC_SEN)
- net PFC_IA_SEN: now reaches MD2.26L (PFC_IA_SEN)
- net AVDD: now reaches MD2.3L (AVDD)
- net AVDD: now also MD2.4L (AGND), RV1.1 (CCW)
- net PWR_RELAY: now reaches MD2.9L (PWR_RELAY)
- net RTS2: now reaches MD2.11R (DV_RTS)
- net CTS2: now reaches MD2.12R (DV_CTS)
- net ~{MC_PWM_FLT}: now reaches MD2.13R (~{MC_PWM_FLT})
- net MC_TEMP_SEN: now reaches MD2.21R (MC_TEMP_SEN)
- net MC_VR_DIV: now reaches MD2.22R (MC_VR_DIV)
- net MC_VR_DIV: now also C31.2, R4.2
- net MC_VV_DIV: now reaches MD2.23R (MC_VU_DIV)
- net MC_IU_SEN: now reaches MD2.24R (MC_IU_SEN)
- net MC_VU_DIV: now reaches MD2.25R (MC_VV_DIV)
- net MC_IV_SEN: now reaches MD2.26R (MC_IV_SEN)
- net USB_N: now reaches MD2.3R (USB_N)
- net USB_P: now reaches MD2.5R (USB_P)
- new net: J9.1, R74.1
- new net: D8.K, R47.1
- new net: R4.1, RV1.2 (WIPER)
- new net: BZ1.3 (V-), D4.A, D6.K, Q3.3 (D)
- new net: D7.K, R44.1
- new net: D6.A, R5.1
- new net +5V: BZ1.2 (V+), D4.K, R5.2
- no-connect marks 9 -> 2
Other:
- note removed: "(CH7)"
- moved on the sheet: C34, J9, MD2A, MD2B, TP23, U11

Commit message: V1 schematic update 3
Connections:
- net MC_VU_DIV renamed MC_UV_DIV
- net MC_VV_DIV renamed MC_UU_DIV
- net PFC_IA_SEN: no longer names the net of MD2.26L (PFC_IA_SEN)
- net PFC_IB_SEN: no longer names the net of MD2.24L (PFC_IB_SEN)
- net PFC_IDC_SEN renamed MC_IDC_SEN
- net PFC_PWM_A: no longer names the net of MD2.20L (PFC_PWM_A)
- net PFC_PWM_B: no longer names the net of MD2.18L (PFC_PWM_B)
- net PFC_PWM_ENA: no longer names the net of MD2.19L (PFC_PWM_ENA)
- net PFC_PWM_ENB: no longer names the net of MD2.17L (PFC_PWM_ENB)
- net PFC_VAC_DIV renamed MC_UW_DIV
- net PFC_VDC_DIV renamed MC_UDC_DIV
- net ~{PFC_FLT}: no longer names the net of MD2.22L (~{PFC_FLT})
- no-connect marks 2 -> 9
Changed lines of the file:
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@@
 	)
 	(no_connect
+		(at 116.205 77.47)
+	)
+	(no_connect
 		(at 116.205 92.71)
 	)
 	(no_connect
+		(at 88.265 85.09)
+	)
+	(no_connect
 		(at 88.265 92.71)
 	)
+	(no_connect
+		(at 116.205 74.93)
+	)
+	(no_connect
+		(at 88.265 82.55)
+	)
+	(no_connect
+		(at 116.205 85.09)
+	)
+	(no_connect
+		(at 116.205 80.01)
+	)
+	(no_connect
+		(at 116.205 82.55)
+	)
 	(wire
 		(pts
@@
 		)
 	)
-	(hierarchical_label "PFC_IB_SEN"
-		(shape input)
-		(at 116.205 77.47 0)
-		(fields_autoplaced yes)
-		(effects
-			(font
-				(size 1.27 1.27)
-				(color 0 200 100 1)
-			)
-			(justify left)
-		)
-	)
 	(hierarchical_label "MC_PWM_VH"
 		(shape output)
@@
 		)
 	)
-	(hierarchical_label "MC_VU_DIV"
+	(hierarchical_label "MC_UV_DIV"
 		(shape input)
 		(at 154.305 74.93 180)
@@
 		)
 	)
-	(hierarchical_label "PFC_PWM_ENB"
-		(shape output)
-		(at 88.265 85.09 180)
-		(fields_autoplaced yes)
-		(effects
-			(font
-				(size 1.27 1.27)
-			)
-			(justify right)
-		)
-	)
-	(hierarchical_label "PFC_IA_SEN"
-		(shape input)
-		(at 116.205 74.93 0)
-		(fields_autoplaced yes)
-		(effects
-			(font
-				(size 1.27 1.27)
-				(color 0 200 100 1)
-			)
-			(justify left)
-		)
-	)
 	(hierarchical_label "SDO"
 		(shape output)
@@
 		)
 	)
-	(hierarchical_label "PFC_PWM_ENA"
-		(shape output)
-		(at 88.265 82.55 180)
-		(fields_autoplaced yes)
-		(effects
-			(font
-				(size 1.27 1.27)
-			)
-			(justify right)
-		)
-	)
 	(hierarchical_label "ENC_A"
 		(shape input)
@@
 		)
 	)
-	(hierarchical_label "MC_VV_DIV"
+	(hierarchical_label "MC_UU_DIV"
 		(shape input)
 		(at 154.305 77.47 180)
@@
 		)
 	)
-	(hierarchical_label "PFC_PWM_A"
-		(shape output)
-		(at 116.205 82.55 0)
-		(fields_autoplaced yes)
-		(effects
-			(font
-				(size 1.27 1.27)
-			)
-			(justify left)
-		)
-	)
 	(hierarchical_label "~{SRAM_CS}"
 		(shape input)
@@
 		)
 	)
-	(hierarchical_label "PFC_VDC_DIV"
+	(hierarchical_label "MC_UDC_DIV"
 		(shape input)
 		(at 88.265 77.47 180)
@@
 		)
 	)
-	(hierarchical_label "PFC_PWM_B"
-		(shape output)
-		(at 116.205 85.09 0)
-		(fields_autoplaced yes)
-		(effects
-			(font
-				(size 1.27 1.27)
-			)
-			(justify left)
-		)
-	)
 	(hierarchical_label "ENC_INDEX"
 		(shape input)
@@
 		)
 	)
-	(hierarchical_label "PFC_IDC_SEN"
+	(hierarchical_label "MC_IDC_SEN"
 		(shape input)
 		(at 88.265 74.93 180)
@@
 		)
 	)
-	(hierarchical_label "PFC_VAC_DIV"
+	(hierarchical_label "MC_UW_DIV"
 		(shape input)
 		(at 88.265 80.01 180)
@@
 		)
 	)
-	(hierarchical_label "~{PFC_FLT}"
-		(shape input)
-		(at 116.205 80.01 0)
-		(fields_autoplaced yes)
-		(effects
-			(font
-				(size 1.27 1.27)
-			)
-			(justify left)
-		)
-	)
 	(symbol
 		(lib_id "power:+5V")
@@
 	)
 	(symbol
-		(lib_name "HW.ACIM-MCU_1")
 		(lib_id "SAMPI:HW.ACIM-MCU")
 		(at 168.275 64.77 0)

Commit message: V1 schematic update 5
Changed lines of the file:
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@@
 		)
 		(stroke
-			(width 0)
+			(width 0.254)
 			(type default)
 		)
@@
 		)
 		(stroke
-			(width 0)
+			(width 0.254)
 			(type default)
 		)
@@
 		)
 		(stroke
-			(width 0)
+			(width 0.254)
 			(type default)
 		)
@@
 		)
 		(stroke
-			(width 0)
+			(width 0.254)
 			(type default)
 		)
@@
 		)
 		(stroke
-			(width 0)
+			(width 0.254)
 			(type default)
 		)
@@
 		)
 		(stroke
-			(width 0)
+			(width 0.254)
 			(type default)
 		)
@@
 		)
 		(stroke
-			(width 0)
+			(width 0.254)
 			(type default)
 		)
@@
 		)
 		(stroke
-			(width 0)
+			(width 0.254)
 			(type default)
 		)
@@
 		)
 		(stroke
-			(width 0)
+			(width 0.254)
 			(type default)
 		)
@@
 		)
 		(stroke
-			(width 0)
+			(width 0.254)
 			(type default)
 		)
@@
 		)
 		(stroke
-			(width 0)
+			(width 0.254)
 			(type default)
 		)
@@
 	(wire
 		(pts
-			(xy 69.85 144.78) (xy 69.85 138.43)
-		)
-		(stroke
-			(width 0)
-			(type default)
-		)
-	)
-	(wire
-		(pts
 			(xy 179.07 138.43) (xy 180.34 138.43)
 		)
@@
 		)
 		(stroke
-			(width 0)
+			(width 0.254)
 			(type default)
 		)
@@
 		)
 		(stroke
-			(width 0)
+			(width 0.254)
 			(type default)
 		)
@@
 		)
 		(stroke
-			(width 0)
+			(width 0.254)
 			(type default)
 		)
@@
 		)
 		(stroke
-			(width 0)
+			(width 0.254)
 			(type default)
 		)
@@
 	(symbol
 		(lib_id "power:GND")
-		(at 69.85 144.78 0)
+		(at 69.85 138.43 0)
 		(mirror y)
 		(unit 1)
@@
 		(dnp no)
 		(property "Reference" "#PWR074"
-			(at 69.85 151.13 0)
+			(at 69.85 144.78 0)
 			(effects
 				(font
@@
 		)
 		(property "Value" "GND"
-			(at 69.85 148.59 0)
+			(at 69.85 142.24 0)
 			(effects
 				(font
@@
 		)
 		(property "Footprint" ""
-			(at 69.85 144.78 0)
+			(at 69.85 138.43 0)
 			(effects
 				(font
@@
 		)
 		(property "Datasheet" ""
-			(at 69.85 144.78 0)
+			(at 69.85 138.43 0)
 			(effects
 				(font
@@
 		)
 		(property "Description" ""
-			(at 69.85 144.78 0)
+			(at 69.85 138.43 0)
 			(effects
 				(font

Commit message: V1 schematic update 6
Parts:
- BZ1: Checked OK -> (none); Unit Price 0.77 -> (none)
- C31: Checked OK -> (none); Unit Price 0.027 -> (none)
- C33, C35: Checked OK -> (none); Unit Price 0.012 -> (none)
- C34: Checked OK -> (none); Unit Price 0.0146 -> (none)
- D4: Checked OK -> (none); Unit Price 0.068 -> (none)
- D6, D7: Checked OK -> (none); Unit Price 0.1 -> (none)
- D8: Checked OK -> (none)
- Q3: Checked OK -> (none); Unit Price 0.148 -> (none)
- R4: Checked OK -> (none); Unit Price 0.029 -> (none)
- R44, R47, R5, R74: Checked OK -> (none); Unit Price 0.021 -> (none)
- R48, R6: Checked OK -> (none); Unit Price 0.019 -> (none)
- U11: Checked OK -> (none); Comment EEPROM -> (none); Unit Price 0.71 -> (none)
Connections:
- net MC_ALT_IV_SEN: now reaches MD2.24L (PFC_IB_SEN)
- net MC_ALT_IU_SEN: now reaches MD2.26L (PFC_IA_SEN)
- no-connect marks 9 -> 7

Commit message: V1 schematic update 7
Connections:
- net +3V3: now also MD2.R27 (+3V3), MD2.R28 (+3V3); no longer MD2.27R (+3V3), MD2.28R (+3V3)
- net AGND: now also MD2.L1 (AGND), MD2.L2 (AVDD); no longer MD2.1L (AGND), MD2.2L (AVDD)
- net AVDD: now also MD2.L3 (AVDD), MD2.L4 (AGND); no longer MD2.3L (AVDD), MD2.4L (AGND)
- net CTS2: now also MD2.R12 (DV_CTS); no longer MD2.12R (DV_CTS)
- net ENC_A: now also MD2.L28 (ENC_A); no longer MD2.28L (ENC_A)
- net ENC_B: now also MD2.L30 (ENC_B); no longer MD2.30L (ENC_B)
- net ENC_HOME: now also MD2.L27 (ENC_HOME); no longer MD2.27L (ENC_HOME)
- net ENC_INDEX: now also MD2.L29 (ENC_IDX); no longer MD2.29L (ENC_IDX)
- net GND: now also MD2.L5 (GND), MD2.L6 (GND), MD2.R29 (GND), MD2.R30 (GND); no longer MD2.29R (GND), MD2.30R (GND), MD2.5L (GND), MD2.6L (GND)
- net IND_ERR: now also MD2.L8 (IO2); no longer MD2.8L (IO2)
- net IND_RUN: now also MD2.L7 (IO1); no longer MD2.7L (IO1)
- net MC_ALT_IU_SEN: now also MD2.L26 (PFC_IA_SEN); no longer MD2.26L (PFC_IA_SEN)
- net MC_ALT_IV_SEN: now also MD2.L24 (PFC_IB_SEN); no longer MD2.24L (PFC_IB_SEN)
- net MC_IDC_SEN: now also MD2.L25 (IDC_SEN); no longer MD2.25L (IDC_SEN)
- net MC_IU_SEN: now also MD2.R24 (MC_IU_SEN); no longer MD2.24R (MC_IU_SEN)
- net MC_IV_SEN: now also MD2.R26 (MC_IV_SEN); no longer MD2.26R (MC_IV_SEN)
- net MC_PWM_UH: now also MD2.R19 (MC_PWM_UH); no longer MD2.19R (MC_PWM_UH)
- net MC_PWM_UL: now also MD2.R20 (MC_PWM_UL); no longer MD2.20R (MC_PWM_UL)
- net MC_PWM_VH: now also MD2.R17 (MC_PWM_VH); no longer MD2.17R (MC_PWM_VH)
- net MC_PWM_VL: now also MD2.R16 (MC_PWM_WL); no longer MD2.16R (MC_PWM_WL)
- net MC_PWM_WH: now also MD2.R15 (MC_PWM_WH); no longer MD2.15R (MC_PWM_WH)
- net MC_PWM_WL: now also MD2.R18 (MC_PWM_VL); no longer MD2.18R (MC_PWM_VL)
- net MC_TEMP_SEN: now also MD2.R21 (MC_TEMP_SEN); no longer MD2.21R (MC_TEMP_SEN)
- net MC_UDC_DIV: now also MD2.L23 (UDC_DIV); no longer MD2.23L (UDC_DIV)
- net MC_UU_DIV: now also MD2.R23 (MC_UU_DIV); no longer MD2.23R (MC_UU_DIV)
- net MC_UV_DIV: now also MD2.R25 (MC_UV_DIV); no longer MD2.25R (MC_UV_DIV)
- net MC_UW_DIV: now also MD2.L21 (UAC_DIV); no longer MD2.21L (UAC_DIV)
- net MC_VR_DIV: now also MD2.R22 (MC_VR_DIV); no longer MD2.22R (MC_VR_DIV)
- net PGC: now also MD2.R4 (PGC); no longer MD2.4R (PGC)
- net PGD: now also MD2.R2 (PGD); no longer MD2.2R (PGD)
- net PWR_RELAY: now also MD2.L9 (PWR_RELAY); no longer MD2.9L (PWR_RELAY)
- net RTS2: now also MD2.R11 (DV_RTS); no longer MD2.11R (DV_RTS)
- net RXD1: now also MD2.R7 (DB_RXD); no longer MD2.7R (DB_RXD)
- net RXD2: now also MD2.R9 (DV_RXD); no longer MD2.9R (DV_RXD)
- net SCK: now also MD2.L15 (SCK); no longer MD2.15L (SCK)
- net SDI: now also MD2.L16 (SDI); no longer MD2.16L (SDI)
- net SDO: now also MD2.L14 (SDO); no longer MD2.14L (SDO)
- net TXD1: now also MD2.R8 (DB_TXD); no longer MD2.8R (DB_TXD)
- net TXD2: now also MD2.R10 (DV_TXD); no longer MD2.10R (DV_TXD)
- net USB_N: now also MD2.R3 (USB_N); no longer MD2.3R (USB_N)
- net USB_P: now also MD2.R5 (USB_P); no longer MD2.5R (USB_P)
- net VBUS: now also MD2.R1 (VBUS); no longer MD2.1R (VBUS)
- net ~{BT_UBT}: now also MD2.R14 (~{BUTTON}); no longer MD2.14R (~{BUTTON})
- net ~{MCLR}: now also MD2.R6 (~{MCLR}); no longer MD2.6R (~{MCLR})
- net ~{MC_PWM_FLT}: now also MD2.R13 (~{MC_PWM_FLT}); no longer MD2.13R (~{MC_PWM_FLT})
- net ~{SRAM_CS}: now also MD2.L13 (~{CS}); no longer MD2.13L (~{CS})
- removed net DEV_RELAY: MD2.10L (DEV_RELAY)
- new net ~{DEV_RELAY}: MD2.L10 (~{DEV_RELAY})

Commit message: V1 schematic update 8
Parts:
- removed C35: 22pF, SAMPI:CAP0603, symbol SAMPI:CERCAP
- removed J9: USB, SAMPI:HDM-1x4x1.25-TH, symbol SAMPI:SIL04-1
- removed R74: 1.1K, SAMPI:RES0603, symbol SAMPI:RES
- removed TP23: VUSB, SAMPI:TP1MM, symbol SAMPI:TESTPOINT
- added CB1: CABLE1, symbol SAMPI:CABLE1
- added J4: MCDBG, SAMPI:IDC-2x5x2MM-TH, symbol SAMPI:MCDBG
Connections:
- net +3V3: now also J4.4 (VDD)
- net GND: now also J4.6 (GND)
- net PGC: now also J4.10 (PGC/SWIO)
- net PGD: now also J4.8 (PGD/SWCK)
- net ~{MCLR}: now also J4.2 (~{RESET})
- net CTS2 renamed DV_CTS
- net DV_CTS: now also J4.7 (DV_CTS)
- net RTS2 renamed DV_RTS
- net DV_RTS: now also J4.5 (DV_RTS)
- net RXD1: no longer names the net of MD2.R7 (DB_RXD)
- net RXD2 renamed DV_RXD
- net DV_RXD: now also J4.3 (DV_RXD)
- net TXD1 renamed DB_TXD
- net DB_TXD: now also J4.9 (DB_TXD)
- net TXD2 renamed DV_TXD
- net DV_TXD: now also J4.1 (DV_TXD)
- net USB_N: no longer names the net of MD2.R3 (USB_N)
- net USB_P: no longer names the net of MD2.R5 (USB_P)
- net VBUS: no longer names the net of MD2.R1 (VBUS)
- no-connect marks 7 -> 11

Commit message: V1 schematic update 15
Parts:
- removed BZ1: BUZZER, SAMPI:SMT-0827-S-HT-R, symbol SAMPI:BUZZER
- removed C34: 100nF, SAMPI:CAP0603, symbol SAMPI:CERCAP
- removed D4: 75V/150mA, SAMPI:SOD-323, symbol SAMPI:DIODE-REC
- removed Q3: 20V/1A, SAMPI:SOT23, symbol SAMPI:FET_N-CH
- removed R4: 10R, SAMPI:RES0603, symbol SAMPI:RES
- removed R5: 1.1K, SAMPI:RES0603, symbol SAMPI:RES
- removed U11: 2Mbit SRAM, SAMPI:SOIC8_3.9_MCHP, symbol SAMPI:SPI_MEM
- J4: footprint SAMPI:IDC-2x5x2MM-TH -> SAMPI:IDC-2x6x2.54MM_TH; MFT Sullins Connector Solutions -> Samtec Inc.; MNP SBH21-NBPN-D05-ST-BK -> TST-106-01-T-D
Connections:
- net DB_TXD: now also J4.1 (DB_TXD); no longer J4.9 (DB_TXD)
- net DV_RXD: now also J4.7 (DV_RXD); no longer J4.3 (DV_RXD)
- net DV_TXD: now also J4.5 (DV_TXD); no longer J4.1 (DV_TXD)
- net IND_ERR: now also D6.A; no longer R6.1
- net MC_VR_DIV: now also RV1.2 (WIPER)
- net at D6.K: now also R6.1
- removed net +3V3: D8.A, J4.4 (VDD), MD2.R27 (+3V3), MD2.R28 (+3V3), R48.1
- removed net AGND: C31.1, MD2.L1 (AGND), MD2.L2 (AVDD), RV1.3 (CW)
- removed net AVDD: MD2.L3 (AVDD), MD2.L4 (AGND), RV1.1 (CCW)
- net DV_CTS: no longer names the net of MD2.R12 (DV_CTS)
- net DV_CTS: no longer J4.7 (DV_CTS)
- net DV_RTS: no longer names the net of MD2.R11 (DV_RTS)
- net DV_RTS: no longer J4.5 (DV_RTS)
- removed net GND: BT1.2, C33.1, J4.6 (GND), MD2.L5 (GND), MD2.L6 (GND), MD2.R29 (GND), MD2.R30 (GND), R44.2, R47.2, R6.2
- net MC_ALT_IU_SEN: no longer names the net of MD2.L26 (PFC_IA_SEN)
- net MC_ALT_IV_SEN: no longer names the net of MD2.L24 (PFC_IB_SEN)
- net MC_TEMP_SEN: no longer names the net of MD2.R21 (MC_TEMP_SEN)
- net MC_UU_DIV: no longer names the net of MD2.R23 (MC_UU_DIV)
- net MC_UV_DIV: no longer names the net of MD2.R25 (MC_UV_DIV)
- net MC_UW_DIV: no longer names the net of MD2.L21 (UAC_DIV)
- net SCK: no longer names the net of MD2.L15 (SCK)
- net SDI: no longer names the net of MD2.L16 (SDI)
- net SDO: no longer names the net of MD2.L14 (SDO)
- net ~{SRAM_CS}: no longer names the net of MD2.L13 (~{CS})
- new net +3V3_MCU: J4.4 (VDD)
- new net DB_RXD: J4.3 (DB_RXD)
- new net GND_MCU: J4.6 (GND)
- no-connect marks 11 -> 7
Other:
- company: TON DUC THANG UNIVERSITY -> (none)
- moved on the sheet: CB1, D6, RV1
