File: V1/Design/HW.ACIM-INV/MCU.kicad_sch (KiCad schematic)
At the start: 14 parts, among them J4 MCDBG

Commit message: V1 schematic update 16
Parts:
- removed BT1: UBT, SAMPI:HDM-2x2.54-TH, symbol SAMPI:BT3
- removed C31: 1nF, SAMPI:CAP0603, symbol SAMPI:CERCAP
- removed C33: 22pF, SAMPI:CAP0603, symbol SAMPI:CERCAP
- removed CB1: CABLE1, symbol SAMPI:CABLE1
- removed D8: PWR, SAMPI:LED0603, symbol SAMPI:WLED
- removed J4: MCDBG, SAMPI:IDC-2x6x2.54MM_TH, symbol SAMPI:MCDBG
- removed R47: 1.1K, SAMPI:RES0603, symbol SAMPI:RES
- removed R48: 10K, SAMPI:RES0603, symbol SAMPI:RES
- removed RV1: 10K, Liem:HDM-3x2.54-TH, symbol SAMPI:POT
- R44: value 1.1K -> 1K; MFT YAGEO -> (none); MNP AC0603FR-071K1L -> (none)
- R6: value 100K -> 1K; MFT YAGEO -> (none); MNP RC0603FR-07100KL -> (none)
Connections:
- net +3V3_ADC: now also MD2.L3 (AVDD), MD2.L4 (AGND)
- net +3V3_MCU: now also MD2.R27 (+3V3), MD2.R28 (+3V3)
- net DB_RXD: now also MD2.R7 (DB_RXD)
- net GND_ADC: now also MD2.L1 (AGND), MD2.L2 (AVDD)
- net GND_MCU: now also MD2.L5 (GND), MD2.L6 (GND), MD2.R29 (GND), MD2.R30 (GND), R44.2, R6.2
- net VBUS: now reaches MD2.R1 (VBUS)
- net USB_N: now reaches MD2.R3 (USB_N)
- net USB_P: now reaches MD2.R5 (USB_P)
- net MC_VR_DIV: no longer names the net of MD2.R22 (MC_IW_SEN)
- net ~{BT_UBT}: no longer names the net of MD2.R14 (IO05)
- no-connect marks 7 -> 21
Other:
- moved on the sheet: D6, D7, R44, R6

Commit message: V1 schematic update 17
Parts:
- R49: renamed from R6; MFT (none) -> YAGEO; MNP (none) -> RC0603JR-071KL
- R50: renamed from R44; MFT (none) -> YAGEO; MNP (none) -> RC0603JR-071KL
- renumbered D6 to D17, D7 to D18, MD2 to MD3
Changed lines of the file:
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@@
 		(on_board yes)
 		(dnp no)
-		(property "Reference" "#PWR077"
+		(property "Reference" "#PWR0169"
 			(at 178.435 72.39 0)
 			(effects
@@
 			(project "HW.ACIM-INV"
 				(path "/20f80521-75f2-4ccc-bb34-c9566e70ef5c/51ad8afa-91d3-4900-86cd-9e9f0d5dd47e"
-					(reference "#PWR077")
+					(reference "#PWR0169")
 					(unit 1)
 				)
@@
 		(on_board yes)
 		(dnp no)
-		(property "Reference" "#PWR037"
+		(property "Reference" "#PWR0165"
 			(at 122.555 105.41 0)
 			(effects
@@
 			(project "HW.ACIM-INV"
 				(path "/20f80521-75f2-4ccc-bb34-c9566e70ef5c/51ad8afa-91d3-4900-86cd-9e9f0d5dd47e"
-					(reference "#PWR037")
+					(reference "#PWR0165")
 					(unit 1)
 				)
@@
 		(on_board yes)
 		(dnp no)
-		(property "Reference" "#PWR073"
+		(property "Reference" "#PWR0160"
 			(at 81.915 100.33 0)
 			(effects
@@
 			(project "HW.ACIM-INV"
 				(path "/20f80521-75f2-4ccc-bb34-c9566e70ef5c/51ad8afa-91d3-4900-86cd-9e9f0d5dd47e"
-					(reference "#PWR073")
+					(reference "#PWR0160")
 					(unit 1)
 				)
@@
 		(on_board yes)
 		(dnp no)
-		(property "Reference" "#PWR074"
+		(property "Reference" "#PWR0163"
 			(at 122.555 100.33 0)
 			(effects
@@
 			(project "HW.ACIM-INV"
 				(path "/20f80521-75f2-4ccc-bb34-c9566e70ef5c/51ad8afa-91d3-4900-86cd-9e9f0d5dd47e"
-					(reference "#PWR074")
+					(reference "#PWR0163")
 					(unit 1)
 				)
@@
 		(on_board yes)
 		(dnp no)
-		(property "Reference" "#PWR078"
+		(property "Reference" "#PWR0167"
 			(at 158.115 72.39 0)
 			(effects
@@
 			(project "HW.ACIM-INV"
 				(path "/20f80521-75f2-4ccc-bb34-c9566e70ef5c/51ad8afa-91d3-4900-86cd-9e9f0d5dd47e"
-					(reference "#PWR078")
+					(reference "#PWR0167")
 					(unit 1)
 				)
@@
 		(on_board yes)
 		(dnp no)
-		(property "Reference" "#PWR017"
+		(property "Reference" "#PWR0161"
 			(at 92.075 102.87 0)
 			(effects
@@
 			(project "HW.ACIM-INV"
 				(path "/20f80521-75f2-4ccc-bb34-c9566e70ef5c/51ad8afa-91d3-4900-86cd-9e9f0d5dd47e"
-					(reference "#PWR017")
+					(reference "#PWR0161")
 					(unit 1)
 				)
@@
 		(on_board yes)
 		(dnp no)
-		(property "Reference" "MD2"
+		(property "Reference" "MD3"
 			(at 102.87 64.135 0)
 			(effects
@@
 			(project ""
 				(path "/20f80521-75f2-4ccc-bb34-c9566e70ef5c/51ad8afa-91d3-4900-86cd-9e9f0d5dd47e"
-					(reference "MD2")
+					(reference "MD3")
 					(unit 1)
 				)
@@
 		(on_board yes)
 		(dnp no)
-		(property "Reference" "#PWR063"
+		(property "Reference" "#PWR0168"
 			(at 188.595 69.85 0)
 			(effects
@@
 			(project "HW.ACIM-INV"
 				(path "/20f80521-75f2-4ccc-bb34-c9566e70ef5c/51ad8afa-91d3-4900-86cd-9e9f0d5dd47e"
-					(reference "#PWR063")
+					(reference "#PWR0168")
 					(unit 1)
 				)
@@
 		(on_board yes)
 		(dnp no)
-		(property "Reference" "R44"
+		(property "Reference" "R50"
 			(at 217.17 99.06 90)
 			(effects
@@
 			)
 		)
-		(property "Description" ""
+		(property "Description" "RES 1K OHM 5% 1/10W 0603"
 			(at 210.82 99.06 0)
 			(effects
@@
 			)
 		)
-		(property "MFT" ""
+		(property "MFT" "YAGEO"
 			(at 210.82 99.06 0)
 			(effects
@@
 			)
 		)
-		(property "MNP" ""
+		(property "MNP" "RC0603JR-071KL"
 			(at 210.82 99.06 0)
 			(effects
@@
 			(project "HW.ACIM-INV"
 				(path "/20f80521-75f2-4ccc-bb34-c9566e70ef5c/51ad8afa-91d3-4900-86cd-9e9f0d5dd47e"
-					(reference "R44")
+					(reference "R50")
 					(unit 1)
 				)
@@
 		(dnp no)
 		(fields_autoplaced yes)
-		(property "Reference" "D7"
+		(property "Reference" "D18"
 			(at 210.82 91.4399 90)
 			(effects
@@
 			(project "HW.ACIM-INV"
 				(path "/20f80521-75f2-4ccc-bb34-c9566e70ef5c/51ad8afa-91d3-4900-86cd-9e9f0d5dd47e"
-					(reference "D7")
+					(reference "D18")
 					(unit 1)
 				)
@@
 		(on_board yes)
 		(dnp no)
-		(property "Reference" "#PWR079"
+		(property "Reference" "#PWR0170"
 			(at 203.2 110.49 0)
 			(effects
@@
 			(project "HW.ACIM-INV"
 				(path "/20f80521-75f2-4ccc-bb34-c9566e70ef5c/51ad8afa-91d3-4900-86cd-9e9f0d5dd47e"
-					(reference "#PWR079")
+					(reference "#PWR0170")
 					(unit 1)
 				)
@@
 		(on_board yes)
 		(dnp no)
-		(property "Reference" "#PWR036"
+		(property "Reference" "#PWR0162"
 			(at 81.915 105.41 0)
 			(effects
@@
 			(project "HW.ACIM-INV"
 				(path "/20f80521-75f2-4ccc-bb34-c9566e70ef5c/51ad8afa-91d3-4900-86cd-9e9f0d5dd47e"
-					(reference "#PWR036")
+					(reference "#PWR0162")
 					(unit 1)
 				)
@@
 		(on_board yes)
 		(dnp no)
-		(property "Reference" "#PWR080"
+		(property "Reference" "#PWR0171"
 			(at 213.36 110.49 0)
 			(effects
@@
 			(project "HW.ACIM-INV"
 				(path "/20f80521-75f2-4ccc-bb34-c9566e70ef5c/51ad8afa-91d3-4900-86cd-9e9f0d5dd47e"
-					(reference "#PWR080")
+					(reference "#PWR0171")
 					(unit 1)
 				)
@@
 		(on_board yes)
 		(dnp no)
-		(property "Reference" "R6"
+		(property "Reference" "R49"
 			(at 207.01 99.06 90)
 			(effects
@@
 			)
 		)
-		(property "Description" ""
+		(property "Description" "RES 1K OHM 5% 1/10W 0603"
 			(at 200.66 99.06 0)
 			(effects
@@
 			)
 		)
-		(property "MFT" ""
+		(property "MFT" "YAGEO"
 			(at 200.66 99.06 0)
 			(effects
@@
 			)
 		)
-		(property "MNP" ""
+		(property "MNP" "RC0603JR-071KL"
 			(at 200.66 99.06 0)
 			(effects
@@
 			(project "HW.ACIM-INV"
 				(path "/20f80521-75f2-4ccc-bb34-c9566e70ef5c/51ad8afa-91d3-4900-86cd-9e9f0d5dd47e"
-					(reference "R6")
+					(reference "R49")
 					(unit 1)
 				)
@@
 		(on_board yes)
 		(dnp no)
-		(property "Reference" "#PWR050"
+		(property "Reference" "#PWR0164"
 			(at 112.395 102.87 0)
 			(effects
@@
 			(project "HW.ACIM-INV"
 				(path "/20f80521-75f2-4ccc-bb34-c9566e70ef5c/51ad8afa-91d3-4900-86cd-9e9f0d5dd47e"
-					(reference "#PWR050")
+					(reference "#PWR0164")
 					(unit 1)
 				)
@@
 		(on_board yes)
 		(dnp no)
-		(property "Reference" "D6"
+		(property "Reference" "D17"
 			(at 198.12 91.44 90)
 			(effects
@@
 			(project "HW.ACIM-INV"
 				(path "/20f80521-75f2-4ccc-bb34-c9566e70ef5c/51ad8afa-91d3-4900-86cd-9e9f0d5dd47e"
-					(reference "D6")
+					(reference "D17")
 					(unit 1)
 				)
@@
 		(on_board yes)
 		(dnp no)
-		(property "Reference" "#PWR056"
+		(property "Reference" "#PWR0166"
 			(at 147.955 69.85 0)
 			(effects
@@
 			(project "HW.ACIM-INV"
 				(path "/20f80521-75f2-4ccc-bb34-c9566e70ef5c/51ad8afa-91d3-4900-86cd-9e9f0d5dd47e"
-					(reference "#PWR056")
+					(reference "#PWR0166")
 					(unit 1)
 				)
@@
 		(on_board yes)
 		(dnp no)
-		(property "Reference" "MD2"
+		(property "Reference" "MD3"
 			(at 168.275 64.135 0)
 			(effects
@@
 			(project ""
 				(path "/20f80521-75f2-4ccc-bb34-c9566e70ef5c/51ad8afa-91d3-4900-86cd-9e9f0d5dd47e"
-					(reference "MD2")
+					(reference "MD3")
 					(unit 2)
 				)

Commit message: V1 schematic update 21
Connections:
- net GND_MCU: now also D17.K, D18.K; no longer R49.2, R50.2
- net IND_ERR: now also R49.1; no longer D17.A
- net IND_RUN: now also R50.1; no longer D18.A
- new net: D18.A, R50.2
- new net: D17.A, R49.2
Other:
- moved on the sheet: D17, D18, R49, R50
Changed lines of the file:
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@@
 	(hierarchical_label "IND_RUN"
 		(shape input)
-		(at 213.36 88.9 90)
+		(at 213.36 90.805 90)
 		(fields_autoplaced yes)
 		(effects
@@
 	(hierarchical_label "IND_ERR"
 		(shape input)
-		(at 203.2 88.9 90)
+		(at 203.2 90.805 90)
 		(fields_autoplaced yes)
 		(effects
@@
 	(symbol
 		(lib_id "SAMPI:RES")
-		(at 210.82 99.06 90)
+		(at 210.82 93.345 90)
 		(mirror x)
 		(unit 1)
@@
 		(dnp no)
 		(property "Reference" "R50"
-			(at 217.17 99.06 90)
+			(at 217.17 93.345 90)
 			(effects
 				(font
@@
 		)
 		(property "Value" "1K"
-			(at 217.17 101.6 90)
+			(at 217.17 95.885 90)
 			(effects
 				(font
@@
 		)
 		(property "Footprint" "SAMPI:RES0603"
-			(at 210.82 99.06 0)
+			(at 210.82 93.345 0)
 			(effects
 				(font
@@
 		)
 		(property "Datasheet" ""
-			(at 210.82 99.06 0)
+			(at 210.82 93.345 0)
 			(effects
 				(font
@@
 		)
 		(property "Description" "RES 1K OHM 5% 1/10W 0603"
-			(at 210.82 99.06 0)
+			(at 210.82 93.345 0)
 			(effects
 				(font
@@
 		)
 		(property "MFT" "YAGEO"
-			(at 210.82 99.06 0)
+			(at 210.82 93.345 0)
 			(effects
 				(font
@@
 		)
 		(property "MNP" "RC0603JR-071KL"
-			(at 210.82 99.06 0)
+			(at 210.82 93.345 0)
 			(effects
 				(font
@@
 	(symbol
 		(lib_id "SAMPI:GLED")
-		(at 210.82 90.805 90)
+		(at 210.82 100.33 90)
 		(mirror x)
 		(unit 1)
@@
 		(fields_autoplaced yes)
 		(property "Reference" "D18"
-			(at 210.82 91.4399 90)
+			(at 210.82 100.9649 90)
 			(effects
 				(font
@@
 		)
 		(property "Value" "RUN"
-			(at 210.82 93.9799 90)
+			(at 210.82 103.5049 90)
 			(effects
 				(font
@@
 		)
 		(property "Footprint" "SAMPI:LED0603"
-			(at 210.82 90.805 0)
+			(at 210.82 100.33 0)
 			(effects
 				(font
@@
 		)
 		(property "Datasheet" ""
-			(at 210.82 90.805 0)
+			(at 210.82 100.33 0)
 			(effects
 				(font
@@
 		)
 		(property "Description" "LED GREEN DIFFUSED 0603 SMD"
-			(at 210.82 90.805 0)
+			(at 210.82 100.33 0)
 			(effects
 				(font
@@
 		)
 		(property "MFT" "Harvatek"
-			(at 210.82 90.805 0)
+			(at 210.82 100.33 0)
 			(effects
 				(font
@@
 		)
 		(property "MNP" "B1911NG--20D000214U1930"
-			(at 210.82 90.805 0)
+			(at 210.82 100.33 0)
 			(effects
 				(font
@@
 	(symbol
 		(lib_id "SAMPI:GND_MCU")
-		(at 203.2 104.14 0)
+		(at 203.2 106.045 0)
 		(unit 1)
 		(exclude_from_sim no)
@@
 		(dnp no)
 		(property "Reference" "#PWR0170"
-			(at 203.2 110.49 0)
+			(at 203.2 112.395 0)
 			(effects
 				(font
@@
 		)
 		(property "Value" "GND_MCU"
-			(at 203.2 107.95 0)
+			(at 203.2 109.855 0)
 			(effects
 				(font
@@
 		)
 		(property "Footprint" ""
-			(at 203.2 104.14 0)
+			(at 203.2 106.045 0)
 			(effects
 				(font
@@
 		)
 		(property "Datasheet" ""
-			(at 203.2 104.14 0)
+			(at 203.2 106.045 0)
 			(effects
 				(font
@@
 		)
 		(property "Description" "Power symbol creates a global label with name \"GND\" , ground"
-			(at 203.2 104.14 0)
+			(at 203.2 106.045 0)
 			(effects
 				(font
@@
 	(symbol
 		(lib_id "SAMPI:GND_MCU")
-		(at 213.36 104.14 0)
+		(at 213.36 106.045 0)
 		(unit 1)
 		(exclude_from_sim no)
@@
 		(dnp no)
 		(property "Reference" "#PWR0171"
-			(at 213.36 110.49 0)
+			(at 213.36 112.395 0)
 			(effects
 				(font
@@
 		)
 		(property "Value" "GND_MCU"
-			(at 213.36 107.95 0)
+			(at 213.36 109.855 0)
 			(effects
 				(font
@@
 		)
 		(property "Footprint" ""
-			(at 213.36 104.14 0)
+			(at 213.36 106.045 0)
 			(effects
 				(font
@@
 		)
 		(property "Datasheet" ""
-			(at 213.36 104.14 0)
+			(at 213.36 106.045 0)
 			(effects
 				(font
@@
 		)
 		(property "Description" "Power symbol creates a global label with name \"GND\" , ground"
-			(at 213.36 104.14 0)
+			(at 213.36 106.045 0)
 			(effects
 				(font
@@
 	(symbol
 		(lib_id "SAMPI:RES")
-		(at 200.66 99.06 90)
+		(at 200.66 93.345 90)
 		(mirror x)
 		(unit 1)
@@
 		(dnp no)
 		(property "Reference" "R49"
-			(at 207.01 99.06 90)
+			(at 207.01 93.345 90)
 			(effects
 				(font
@@
 		)
 		(property "Value" "1K"
-			(at 207.01 101.6 90)
+			(at 207.01 95.885 90)
 			(effects
 				(font
@@
 		)
 		(property "Footprint" "SAMPI:RES0603"
-			(at 200.66 99.06 0)
+			(at 200.66 93.345 0)
 			(effects
 				(font
@@
 		)
 		(property "Datasheet" ""
-			(at 200.66 99.06 0)
+			(at 200.66 93.345 0)
 			(effects
 				(font
@@
 		)
 		(property "Description" "RES 1K OHM 5% 1/10W 0603"
-			(at 200.66 99.06 0)
+			(at 200.66 93.345 0)
 			(effects
 				(font
@@
 		)
 		(property "MFT" "YAGEO"
-			(at 200.66 99.06 0)
+			(at 200.66 93.345 0)
 			(effects
 				(font
@@
 		)
 		(property "MNP" "RC0603JR-071KL"
-			(at 200.66 99.06 0)
+			(at 200.66 93.345 0)
 			(effects
 				(font
@@
 	(symbol
 		(lib_id "SAMPI:RLED")
-		(at 207.645 91.44 270)
+		(at 207.645 100.965 270)
 		(unit 1)
 		(exclude_from_sim no)
@@
 		(dnp no)
 		(property "Reference" "D17"
-			(at 198.12 91.44 90)
+			(at 198.12 100.965 90)
 			(effects
 				(font
@@
 		)
 		(property "Value" "ERR"
-			(at 198.12 93.98 90)
+			(at 198.12 103.505 90)
 			(effects
 				(font
@@
 		)
 		(property "Footprint" "SAMPI:LED0603"
-			(at 207.645 91.44 0)
+			(at 207.645 100.965 0)
 			(effects
 				(font
@@
 		)
 		(property "Datasheet" ""
-			(at 207.645 91.44 0)
+			(at 207.645 100.965 0)
 			(effects
 				(font
@@
 		)
 		(property "Description" "LED RED DIFFUSED 0603 SMD"
-			(at 207.645 91.44 0)
+			(at 207.645 100.965 0)
 			(effects
 				(font
@@
 		)
 		(property "MFT" "Harvatek"
-			(at 207.645 91.44 0)
+			(at 207.645 100.965 0)
 			(effects
 				(font
@@
 		)
 		(property "MNP" "B1911USD-20D000114U1930"
-			(at 207.645 91.44 0)
-			(effects
-				(font
+			(at 207.645 100.965 0)
+			(effects
+				(font

Commit message: V1 schematic update 24
Parts:
- MD3: footprint SAMPI:HW.ACIM-MCU -> SAMPI:HW.ACIM-MCU_SMD
Connections:
- no-connect marks 21 -> 0
Changed lines of the file:
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@@
 		(rev "1.0")
-	)
-	(no_connect
-		(at 182.245 80.01)
-	)
-	(no_connect
-		(at 182.245 90.17)
-	)
-	(no_connect
-		(at 154.305 92.71)
-	)
-	(no_connect
-		(at 88.265 90.17)
-	)
-	(no_connect
-		(at 116.205 92.71)
-	)
-	(no_connect
-		(at 182.245 92.71)
-	)
-	(no_connect
-		(at 116.205 90.17)
-	)
-	(no_connect
-		(at 154.305 74.93)
-	)
-	(no_connect
-		(at 88.265 87.63)
-	)
-	(no_connect
-		(at 154.305 80.01)
-	)
-	(no_connect
-		(at 88.265 85.09)
-	)
-	(no_connect
-		(at 88.265 92.71)
-	)
-	(no_connect
-		(at 88.265 82.55)
-	)
-	(no_connect
-		(at 116.205 74.93)
-	)
-	(no_connect
-		(at 116.205 77.47)
-	)
-	(no_connect
-		(at 154.305 77.47)
-	)
-	(no_connect
-		(at 88.265 80.01)
-	)
-	(no_connect
-		(at 116.205 85.09)
-	)
-	(no_connect
-		(at 116.205 87.63)
-	)
-	(no_connect
-		(at 116.205 80.01)
-	)
-	(no_connect
-		(at 116.205 82.55)
 	)
 	(hierarchical_label "VBUS"
@@
 			)
 		)
-		(property "Footprint" "SAMPI:HW.ACIM-MCU"
+		(property "Footprint" "SAMPI:HW.ACIM-MCU_SMD"
 			(at 102.87 66.675 0)
 			(effects
@@
 		(pin "R5"
 		)
-		(pin "L11"
-		)
 		(pin "L30"
 		)
@@
 		(pin "L6"
 		)
-		(pin "L16"
-		)
 		(pin "L7"
 		)
-		(pin "R25"
-		)
-		(pin "L26"
-		)
 		(pin "L29"
 		)
-		(pin "R23"
-		)
 		(pin "R18"
 		)
-		(pin "L13"
-		)
 		(pin "R28"
 		)
@@
 		(pin "L3"
 		)
-		(pin "L20"
-		)
 		(pin "R3"
 		)
-		(pin "R22"
-		)
-		(pin "L12"
-		)
 		(pin "L23"
 		)
@@
 		(pin "R27"
 		)
-		(pin "L14"
-		)
 		(pin "R16"
 		)
-		(pin "L24"
-		)
-		(pin "L18"
-		)
 		(pin "R13"
 		)
@@
 		(pin "L28"
 		)
-		(pin "R12"
-		)
 		(pin "R15"
 		)
 		(pin "L2"
 		)
-		(pin "R11"
-		)
 		(pin "L9"
 		)
 		(pin "R29"
 		)
-		(pin "L17"
-		)
 		(pin "R2"
 		)
-		(pin "R14"
-		)
 		(pin "R26"
 		)
-		(pin "R21"
-		)
 		(pin "R19"
 		)
@@
 		)
 		(pin "R24"
-		)
-		(pin "L22"
-		)
-		(pin "L21"
-		)
-		(pin "L19"
-		)
-		(pin "L15"
 		)
 		(pin "R10"
@@
 			)
 		)
-		(property "Footprint" "SAMPI:HW.ACIM-MCU"
+		(property "Footprint" "SAMPI:HW.ACIM-MCU_SMD"
 			(at 168.275 66.675 0)
 			(effects
@@
 			)
 		)
-		(pin "L16"
-		)
-		(pin "L19"
-		)
 		(pin "L7"
 		)
-		(pin "L18"
-		)
 		(pin "R20"
 		)
@@
 		(pin "L29"
 		)
-		(pin "L17"
-		)
 		(pin "L5"
 		)
 		(pin "R2"
 		)
-		(pin "R23"
-		)
 		(pin "L28"
 		)
@@
 		(pin "L8"
 		)
-		(pin "L11"
-		)
 		(pin "L1"
 		)
@@
 		(pin "R18"
 		)
-		(pin "L12"
-		)
-		(pin "R21"
-		)
 		(pin "L23"
 		)
 		(pin "R4"
 		)
-		(pin "R11"
-		)
-		(pin "L13"
-		)
 		(pin "R27"
 		)
-		(pin "L14"
-		)
 		(pin "L4"
 		)
-		(pin "R12"
-		)
-		(pin "R14"
-		)
-		(pin "L26"
-		)
-		(pin "L22"
-		)
 		(pin "L27"
 		)
@@
 		(pin "L9"
 		)
-		(pin "L24"
-		)
-		(pin "L15"
-		)
-		(pin "R25"
-		)
 		(pin "R26"
 		)
-		(pin "R22"
-		)
 		(pin "L3"
 		)
-		(pin "L21"
-		)
 		(pin "R16"
 		)
@@
 		(pin "R6"
 		)
-		(pin "L20"
-		)
 		(pin "R10"

Commit message: V1 schematic update 28
Connections:
- net MC_IU_SEN: now also MD3.R26 (MC_IU_SEN); no longer MD3.R24 (MC_IV_SEN)
- net MC_IV_SEN: now also MD3.R24 (MC_IV_SEN); no longer MD3.R26 (MC_IU_SEN)
Changed lines of the file:
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@@
 	(hierarchical_label "MC_IU_SEN"
 		(shape input)
-		(at 182.245 77.47 0)
+		(at 182.245 74.93 0)
 		(fields_autoplaced yes)
 		(effects
@@
 	(hierarchical_label "MC_IV_SEN"
 		(shape input)
-		(at 182.245 74.93 0)
-		(fields_autoplaced yes)
-		(effects
+		(at 182.245 77.47 0)
+		(fields_autoplaced yes)
+		(effects

Commit message: V1 schematic update 29
Connections:
- net MC_IU_SEN: now also MD3.R24 (MC_IU_SEN); no longer MD3.R26 (MC_IU_SEN)
- net MC_IV_SEN: now also MD3.R26 (MC_IV_SEN); no longer MD3.R24 (MC_IV_SEN)
Changed lines of the file:
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@@
 	(hierarchical_label "MC_IU_SEN"
 		(shape input)
-		(at 182.245 74.93 0)
+		(at 182.245 77.47 0)
 		(fields_autoplaced yes)
 		(effects
@@
 	(hierarchical_label "MC_IV_SEN"
 		(shape input)
-		(at 182.245 77.47 0)
-		(fields_autoplaced yes)
-		(effects
+		(at 182.245 74.93 0)
+		(fields_autoplaced yes)
+		(effects
