File: V1/Design/HW.ACIM-INV/HW.ACIM-INV.kicad_sch (KiCad schematic)
At the start: 7 parts

Commit message: V1 schematic update 2
Connections:
- no-connect marks 15 -> 0
Other:
- removed sheet DEBUGGER
- sheet ENCODER ports: added none; removed ENC_A, ENC_B, ENC_HOME, ENC_INDEX
- sheet Inverter ports: added none; removed INV_FLT_OC, IPM_PWM_UH, IPM_PWM_UL, IPM_PWM_VH, IPM_PWM_VL, IPM_PWM_WH, IPM_PWM_WL, MC_IDC_SENSE, MC_IPM_TEMP, MC_IU_SENSE, MC_IV_SENSE, MC_IW_SENSE, MC_PWM_UH, MC_PWM_UL, MC_PWM_VH, MC_PWM_VL, MC_PWM_WH, MC_PWM_WL, MC_VU, MC_VV, MC_VW
- sheet MCU ports: added none; removed CTS2, ENC_A, ENC_B, ENC_HOME, ENC_INDEX, IND_ERR, IND_RUN, MC_IDC_SENSE, MC_IPM_TEMP, MC_IU_SENSE, MC_IV_SENSE, MC_IW_SENSE, MC_PWM_UH, MC_PWM_UL, MC_PWM_VH, MC_PWM_VL, MC_PWM_WH, MC_PWM_WL, MC_VDC_SENSE, MC_VU_SENSE, MC_VV_SENSE, MC_VW_SENSE, PGC, PGD, RTS2, RXD1, RXD2, SCK, SDI, SDO, SOSCI, SOSCO, SYS_CLK, SYS_CLK_EN, TXD1, TXD2, ~{BT_UBT}, ~{INV_FAULT}, ~{INV_FLT_OC}, ~{MCLR}, ~{MEM_CFG}, ~{MEM_TMP}, ~{PWR_FAULT}
- sheet POWER ports: added none; removed ~{INV_FAULT}, ~{PWR_FAULT}
- sheet VI Measurement ports: added none; removed INV_FLT_OC, MC_IDC_SENSE, MC_VDC_SENSE, MC_VU, MC_VU_SENSE, MC_VV, MC_VV_SENSE, MC_VW, MC_VW_SENSE, ~{INV_FLT_OC}
- note added: "3.3V/0.3A"
- note added: "3.3V/1A"

Commit message: V1 schematic update 6
Other:
- sheet ENCODER ports: added ENC_A, ENC_B, ENC_HOME, ENC_INDEX, HOME, INDEX, PULSE_A, PULSE_B; removed none
- sheet Inverter ports: added IPM_PWM_FLT, IPM_PWM_UH, IPM_PWM_UL, IPM_PWM_VH, IPM_PWM_VL, IPM_PWM_WH, IPM_PWM_WL, MC_IDC_SEN_N, MC_IDC_SEN_P, MC_IU_HAL, MC_IU_SEN_N, MC_IU_SEN_P, MC_IV_HAL, MC_IV_SEN_N, MC_IV_SEN_P, MC_PWM_FLT, MC_PWM_UH, MC_PWM_UL, MC_PWM_VH, MC_PWM_VL, MC_PWM_WH, MC_PWM_WL, MC_TEMP_SEN, MC_UU, MC_UV, MC_UW; removed none
- sheet MCU ports: added CTS2, DEV_RELAY, ENC_A, ENC_B, ENC_HOME, ENC_INDEX, IND_ERR, IND_RUN, MC_ALT_IU_SEN, MC_ALT_IV_SEN, MC_IDC_SEN, MC_IU_SEN, MC_IV_SEN, MC_PWM_UH, MC_PWM_UL, MC_PWM_VH, MC_PWM_VL, MC_PWM_WH, MC_PWM_WL, MC_TEMP_SEN, MC_UDC_DIV, MC_UU_DIV, MC_UV_DIV, MC_UW_DIV, MC_VR_DIV, PGC, PGD, PWR_RELAY, RTS2, RXD1, RXD2, SCK, SDI, SDO, TXD1, TXD2, USB_N, USB_P, VBUS, ~{BT_UBT}, ~{MCLR}, ~{MC_PWM_FLT}, ~{SRAM_CS}; removed none
- sheet POWER ports: added DEV_RELAY, PWR_RELAY; removed none
- sheet VI Measurement ports: added MC_ALT_IU_SEN, MC_ALT_IV_SEN, MC_IDC_SEN, MC_IDC_SEN_N, MC_IDC_SEN_P, MC_IU_HAL, MC_IU_SEN, MC_IU_SEN_N, MC_IU_SEN_P, MC_IV_HAL, MC_IV_SEN, MC_IV_SEN_N, MC_IV_SEN_P, MC_PWM_FLT, MC_UDC_DIV, MC_UU, MC_UU_DIV, MC_UV, MC_UV_DIV, MC_UW, MC_UW_DIV, ~{MC_PWM_FLT}; removed none
- moved on the sheet: SH1, SH2, SH3, SH4, SH5, SH6, SH7

Commit message: V1 schematic update 8
Connections:
- no-connect marks 0 -> 31
Other:
- sheet MCU ports: added DB_TXD, DV_CTS, DV_RTS, DV_RXD, DV_TXD, ~{DEV_RELAY}; removed CTS2, DEV_RELAY, RTS2, RXD2, TXD1, TXD2
- sheet POWER ports: added ~{DEV_RELAY}; removed DEV_RELAY

Commit message: V1 schematic update 9
Other:
- note added: "15V"
- note added: "220VAC"
- note added: "3.3V"
- note added: "5V"
- note added: "AVDD=3.3V"
- note added: "ENCODER"
- note added: "ICSP"
- note added: "ISOLATED 24V"
- note added: "ISOLATED 5V"
- note added: "UART 3MBIT UART 115.2KBIT"
- note added: "VDD=3.3V"
- note added: "VREF=5V"
- note removed: "15V/0.6A"
- note removed: "15V/0.7A 5V/1.5A 3.3V/1.5A ~{INV_FAULT}"
- note removed: "3.3V/0.3A"
- note removed: "3.3V/1.5A"
- note removed: "3.3V/1A"
- note removed: "380VDC"
- note removed: "5V/1.5A"
- note removed: "ISOLATED 24V/0.3A"
- note removed: "SHAFT"
- note removed: "VREF 3.3V/20mA"
- moved on the sheet: SH1, SH2, SH3, SH4, SH5, SH6, SH7

Commit message: V1 schematic update 13
Other:
- sheet Inverter renamed INVERTER
- sheet POWER renamed INVERTER POWER
- sheet VI Measurement renamed POWER MEASUREMENT
- added sheet MCU POWER (MCUPOWER.kicad_sch)
- sheet INVERTER: file Inverter.kicad_sch -> INVERTER.kicad_sch
- sheet INVERTER POWER: file Power.kicad_sch -> INVPOWER.kicad_sch
- sheet POWER MEASUREMENT: file VI_Measurement.kicad_sch -> POWERMEASUREMENT.kicad_sch
Changed lines of the file:
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@@
 	(polyline
 		(pts
-			(xy 35.56 37.465) (xy 36.83 38.735)
+			(xy 30.48 37.465) (xy 31.75 38.735)
 		)
 		(stroke
@@
 	(polyline
 		(pts
-			(xy 35.56 40.005) (xy 36.83 38.735)
+			(xy 30.48 40.005) (xy 31.75 38.735)
 		)
 		(stroke
@@
 	(polyline
 		(pts
-			(xy 25.4 38.735) (xy 36.83 38.735)
+			(xy 21.59 38.735) (xy 31.75 38.735)
 		)
 		(stroke
@@
 	(text_box "POWER SUPPLY"
 		(exclude_from_sim no)
-		(at 17.78 31.75 0)
+		(at 13.97 31.75 0)
 		(size 7.62 12.7)
 		(stroke
@@
 	(text "220VAC"
 		(exclude_from_sim no)
-		(at 31.115 37.465 0)
+		(at 25.4 37.465 0)
 		(effects
 			(font
@@
 			(color 150 255 150 1.0000)
 		)
-		(property "Sheetname" "Inverter"
-			(at 158.75 27.94 0)
+		(property "Sheetname" "INVERTER"
+			(at 158.75 28.575 0)
 			(effects
 				(font
@@
 			)
 		)
-		(property "Sheetfile" "Inverter.kicad_sch"
-			(at 158.75 29.21 0)
+		(property "Sheetfile" "INVERTER.kicad_sch"
+			(at 158.75 29.845 0)
 			(effects
 				(font
@@
 	)
 	(sheet
-		(at 36.83 31.75)
-		(size 20.32 12.7)
+		(at 31.75 31.75)
+		(size 25.4 12.7)
 		(stroke
 			(width 0.1524)
@@
 			(color 150 255 150 1.0000)
 		)
-		(property "Sheetname" "POWER"
-			(at 37.465 30.48 0)
+		(property "Sheetname" "INVERTER POWER"
+			(at 31.75 28.575 0)
 			(effects
 				(font
@@
 			)
 		)
-		(property "Sheetfile" "Power.kicad_sch"
-			(at 36.83 45.72 0)
+		(property "Sheetfile" "INVPOWER.kicad_sch"
+			(at 31.75 29.845 0)
 			(effects
 				(font
@@
 			(effects
 				(font
-					(size 1.27 1.27)
+					(size 1.5 1.5)
 					(bold yes)
 				)
@@
 		)
 		(property "Sheetname" "MCU"
-			(at 69.85 27.94 0)
+			(at 69.85 28.575 0)
 			(effects
 				(font
@@
 		)
 		(property "Sheetfile" "MCU.kicad_sch"
-			(at 69.85 29.21 0)
+			(at 69.85 29.845 0)
 			(effects
 				(font
@@
 			(project "HW.ACIM-INV"
 				(path "/20f80521-75f2-4ccc-bb34-c9566e70ef5c"
-					(page "5")
+					(page "6")
 				)
 			)
@@
 			(color 150 255 150 1.0000)
 		)
-		(property "Sheetname" "VI Measurement"
-			(at 158.75 73.025 0)
+		(property "Sheetname" "POWER MEASUREMENT"
+			(at 158.75 73.66 0)
 			(effects
 				(font
@@
 			)
 		)
-		(property "Sheetfile" "VI_Measurement.kicad_sch"
-			(at 158.75 74.295 0)
+		(property "Sheetfile" "POWERMEASUREMENT.kicad_sch"
+			(at 158.75 74.93 0)
 			(effects
 				(font
@@
 			(project "HW.ACIM-INV"
 				(path "/20f80521-75f2-4ccc-bb34-c9566e70ef5c"
-					(page "4")
+					(page "5")
+				)
+			)
+		)
+	)
+	(sheet
+		(at 31.75 57.15)
+		(size 25.4 12.7)
+		(stroke
+			(width 0.1524)
+			(type solid)
+		)
+		(fill
+			(color 150 255 150 1.0000)
+		)
+		(property "Sheetname" "MCU POWER"
+			(at 31.75 53.975 0)
+			(effects
+				(font
+					(size 1.5 1.5)
+					(thickness 0.254)
+					(bold yes)
+				)
+				(justify left bottom)
+			)
+		)
+		(property "Sheetfile" "MCUPOWER.kicad_sch"
+			(at 31.75 55.245 0)
+			(effects
+				(font
+					(size 1.27 1.27)
+				)
+				(justify left top)
+			)
+		)
+		(instances
+			(project "HW.ACIM-INV"
+				(path "/20f80521-75f2-4ccc-bb34-c9566e70ef5c"
+					(page "3")
 				)
 			)

Commit message: V1 schematic update 14
Connections:
- no-connect marks 31 -> 0
Other:
- sheet ENCODER ports: added none; removed ENC_A, ENC_B, ENC_HOME, ENC_INDEX, HOME, INDEX, PULSE_A, PULSE_B
- sheet INVERTER ports: added none; removed IPM_PWM_FLT, IPM_PWM_UH, IPM_PWM_UL, IPM_PWM_VH, IPM_PWM_VL, IPM_PWM_WH, IPM_PWM_WL, MC_IDC_SEN_N, MC_IDC_SEN_P, MC_IU_HAL, MC_IU_SEN_N, MC_IU_SEN_P, MC_IV_HAL, MC_IV_SEN_N, MC_IV_SEN_P, MC_PWM_FLT, MC_PWM_UH, MC_PWM_UL, MC_PWM_VH, MC_PWM_VL, MC_PWM_WH, MC_PWM_WL, MC_TEMP_SEN, MC_UU, MC_UV, MC_UW
- sheet MCU ports: added none; removed DB_TXD, DV_CTS, DV_RTS, DV_RXD, DV_TXD, ENC_A, ENC_B, ENC_HOME, ENC_INDEX, IND_ERR, IND_RUN, MC_ALT_IU_SEN, MC_ALT_IV_SEN, MC_IDC_SEN, MC_IU_SEN, MC_IV_SEN, MC_PWM_UH, MC_PWM_UL, MC_PWM_VH, MC_PWM_VL, MC_PWM_WH, MC_PWM_WL, MC_TEMP_SEN, MC_UDC_DIV, MC_UU_DIV, MC_UV_DIV, MC_UW_DIV, MC_VR_DIV, PGC, PGD, RXD1, SCK, SDI, SDO, USB_N, USB_P, VBUS, ~{BT_UBT}, ~{MCLR}, ~{MC_PWM_FLT}, ~{SRAM_CS}
- sheet POWER MEASUREMENT ports: added none; removed MC_ALT_IU_SEN, MC_ALT_IV_SEN, MC_IDC_SEN, MC_IDC_SEN_N, MC_IDC_SEN_P, MC_IU_HAL, MC_IU_SEN, MC_IU_SEN_N, MC_IU_SEN_P, MC_IV_HAL, MC_IV_SEN, MC_IV_SEN_N, MC_IV_SEN_P, MC_PWM_FLT, MC_UDC_DIV, MC_UU, MC_UU_DIV, MC_UV, MC_UV_DIV, MC_UW, MC_UW_DIV, ~{MC_PWM_FLT}

Commit message: V1 schematic update 15
Other:
- company: TON DUC THANG UNIVERSITY -> (none)
Changed lines of the file:
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@@
 		(date "2024-09-24")
 		(rev "1.0")
-		(company "TON DUC THANG UNIVERSITY")
-		(comment 1 "Schematic Designed by ...")
-		(comment 2 "PCB Designed by ...")
-		(comment 3 "Approved by ...")
 	)
 	(polyline

Commit message: V1 schematic update 16
Parts:
- added CB1: CABLE1, symbol SAMPI:CABLE1
- added J4: MCDBG, SAMPI:IDC-2x6x2.54MM_TH, symbol SAMPI:MCDBG
Connections:
- new net +3V3_MCU: J4.4 (VDD)
- new net GND_MCU: J4.6 (GND)
- new net MCU/DB_RXD: J4.3 (DB_RXD)
- new net MCU/DB_TXD: J4.1 (DB_TXD)
- new net MCU/DV_RXD: J4.7 (DV_RXD)
- new net MCU/DV_TXD: J4.5 (DV_TXD)
- new net MCU/PGC: J4.10 (PGC/SWDCK)
- new net MCU/PGD: J4.8 (PGD/SWDIO)
- new net MCU/USB_N: J4.11 (USB_DM)
- new net MCU/USB_P: J4.9 (UDB_DP)
- new net MCU/VBUS: J4.12 (VBUS)
- new net MCU/~{MCLR}: J4.2 (~{RESET})
- no-connect marks 0 -> 14
Other:
- sheet ENCODER ports: added ENC_A, ENC_B, ENC_HOME, ENC_INDEX, HOME, INDEX, PULSE_A, PULSE_B; removed none
- sheet INVERTER ports: added IPM_PWM_FLT, IPM_PWM_UH, IPM_PWM_UL, IPM_PWM_VH, IPM_PWM_VL, IPM_PWM_WH, IPM_PWM_WL, IPM_TEMP_SEN, MC_IDC_N, MC_IDC_P, MC_IU_HAL, MC_IV_HAL, MC_PWM_UH, MC_PWM_UL, MC_PWM_VH, MC_PWM_VL, MC_PWM_WH, MC_PWM_WL, MC_TEMP_FLT; removed none
- sheet MCU ports: added DB_RXD, DB_TXD, DV_RXD, DV_TXD, ENC_A, ENC_B, ENC_HOME, ENC_INDEX, IND_ERR, IND_RUN, MC_IDC_SEN, MC_IU_SEN, MC_IV_SEN, MC_PWM_UH, MC_PWM_UL, MC_PWM_VH, MC_PWM_VL, MC_PWM_WH, MC_PWM_WL, MC_UDC_DIV, PGC, PGD, USB_N, USB_P, VBUS, ~{MCLR}, ~{MC_PWM_FLT}; removed none
- sheet POWER MEASUREMENT ports: added MC_IDC_N, MC_IDC_P, MC_IDC_SEN, MC_IU_HAL, MC_IU_SEN, MC_IV_HAL, MC_IV_SEN, MC_UDC_DIV; removed none
- note added: "12V_MCU"
- note added: "16V_INV"
- note added: "24V_MCU"
- note added: "3V3_ADC"
- note added: "3V3_MCU"
- note added: "5V_INV"
- note added: "5V_MCU"
- note added: "VDC (310V)"
- note removed: "15V"
- note removed: "3.3V"
- note removed: "310VDC"
- note removed: "5V"
- note removed: "AVDD=3.3V"
- note removed: "ISOLATED 24V"
- note removed: "ISOLATED 5V"
- note removed: "VDD=3.3V"
- note removed: "VREF=5V"
- moved on the sheet: SH1, SH2, SH3, SH4, SH5, SH6, SH7
