File: V1/Design/HW.ACIM-INV/HW.ACIM-INV.kicad_sch (KiCad schematic)
At the start: 9 parts, among them J4 MCDBG

Commit message: V1 schematic update 17
Parts:
- CB1: value CABLE1 -> MCDBG CABLE; MFT (none) -> Samtec Inc.; MNP (none) -> IDSD-06-D-06.00-T-G
- J1: renamed from J4; MFT Samtec Inc. -> Samtec
- SH1, SH2, SH3, SH4, SH5, SH6, SH7: MFT (none) -> Essentra; MNP (none) -> 50M025045P012; now in the parts list

Commit message: V1 schematic update 18
Other:
- removed sheet INVERTER POWER
- sheet MCU POWER ports: added PWR_RELAY, ~{DEV_RELAY}; removed none
- note removed: "220VAC"
Changed lines of the file:
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@@
 	(polyline
 		(pts
-			(xy 55.88 52.705) (xy 55.88 40.005)
-		)
-		(stroke
-			(width 0)
-			(type default)
-		)
-	)
-	(polyline
-		(pts
 			(xy 232.41 71.755) (xy 233.68 70.485)
 		)
@@
 	)
 	(circle
-		(center 55.88 52.705)
-		(radius 0.635)
-		(stroke
-			(width 0)
-			(type default)
-		)
-		(fill
-			(type color)
-			(color 0 0 0 0)
-		)
-	)
-	(circle
 		(center 107.95 52.705)
 		(radius 0.635)
@@
 		)
 	)
-	(text_box "POWER SUPPLY"
+	(text_box "POWER SUPPLY BOARD"
 		(exclude_from_sim no)
 		(at 13.97 65.405 0)
@@
 		)
 	)
-	(text "220VAC"
-		(exclude_from_sim no)
-		(at 25.4 71.12 0)
-		(effects
-			(font
-				(face "Consolas")
-				(size 1.016 1.016)
-				(thickness 0.127)
-			)
-		)
-	)
 	(text "ENCODER"
 		(exclude_from_sim no)
@@
 	)
 	(sheet
-		(at 31.75 65.405)
-		(size 25.4 12.7)
-		(stroke
-			(width 0.1524)
-			(type solid)
-		)
-		(fill
-			(color 150 255 150 1.0000)
-		)
-		(property "Sheetname" "INVERTER POWER"
-			(at 31.75 62.23 0)
-			(effects
-				(font
-					(face "Consolas")
-					(size 1.27 1.27)
-					(bold yes)
-				)
-				(justify left bottom)
-			)
-		)
-		(property "Sheetfile" "INVPOWER.kicad_sch"
-			(at 31.75 63.5 0)
-			(effects
-				(font
-					(face "Consolas")
-					(size 1.016 1.016)
-					(thickness 0.127)
-				)
-				(justify left top)
-			)
-		)
-		(pin "PWR_RELAY" input
-			(at 57.15 67.31 0)
-			(effects
-				(font
-					(face "Consolas")
-					(size 1.016 1.016)
-					(thickness 0.127)
-				)
-				(justify right)
-			)
-		)
-		(pin "~{DEV_RELAY}" input
-			(at 57.15 69.85 0)
-			(effects
-				(font
-					(face "Consolas")
-					(size 1.016 1.016)
-					(thickness 0.127)
-				)
-				(justify right)
-			)
-		)
-		(instances
-			(project "HW.ACIM-INV"
-				(path "/20f80521-75f2-4ccc-bb34-c9566e70ef5c"
-					(page "2")
-				)
-			)
-		)
-	)
-	(sheet
 		(at 158.75 135.255)
 		(size 59.69 23.495)
@@
 	)
 	(sheet
-		(at 31.75 27.305)
+		(at 31.75 65.405)
 		(size 25.4 12.7)
 		(stroke
@@
 		)
 		(property "Sheetname" "MCU POWER"
-			(at 31.75 24.13 0)
+			(at 31.75 62.23 0)
 			(effects
 				(font
@@
 		)
 		(property "Sheetfile" "MCUPOWER.kicad_sch"
-			(at 31.75 25.4 0)
+			(at 31.75 63.5 0)
 			(effects
 				(font
@@
 			)
 		)
+		(pin "~{DEV_RELAY}" input
+			(at 57.15 69.85 0)
+			(effects
+				(font
+					(size 1.27 1.27)
+				)
+				(justify right)
+			)
+		)
+		(pin "PWR_RELAY" input
+			(at 57.15 67.31 0)
+			(effects
+				(font
+					(size 1.27 1.27)
+				)
+				(justify right)
+			)
+		)

Commit message: V1 schematic update 20
Parts:
- added SH10, SH8, SH9: SCREW HOLDER, SAMPI:SCREWHOLE-2.5M, symbol SAMPI:SCREWHOLDER

Commit message: V1 schematic update 22
Parts:
- removed SH10: SCREW HOLDER, SAMPI:SCREWHOLE-2.5M, symbol SAMPI:SCREWHOLDER
Changed lines of the file:
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@@
-	(symbol
-		(lib_id "SAMPI:SCREWHOLDER")
-		(at 139.7 165.1 0)
-		(unit 1)
-		(exclude_from_sim no)
-		(in_bom yes)
-		(on_board yes)
-		(dnp no)
-		(property "Reference" "SH10"
-			(at 138.43 165.1 0)
-			(effects
-				(font
-					(face "Consolas")
-					(size 1.27 1.27)
-					(thickness 0.254)
-					(bold yes)
-				)
-				(justify left)
-			)
-		)
-		(property "Value" "SCREW HOLDER"
-			(at 142.24 170.1799 0)
-			(effects
-				(font
-					(face "Consolas")
-					(size 1.016 1.016)
-					(thickness 0.127)
-				)
-				(justify left)
-				(hide yes)
-			)
-		)
-		(property "Footprint" "SAMPI:SCREWHOLE-2.5M"
-			(at 139.7 165.1 0)
-			(effects
-				(font
-					(face "Consolas")
-					(size 1.016 1.016)
-					(thickness 0.127)
-				)
-				(hide yes)
-			)
-		)
-		(property "Datasheet" ""
-			(at 139.7 165.1 0)
-			(effects
-				(font
-					(face "Consolas")
-					(size 1.016 1.016)
-					(thickness 0.127)
-				)
-				(hide yes)
-			)
-		)
-		(property "Description" "PAN PHILLIPS SCREW, M2.5 X 4.5 T"
-			(at 139.7 165.1 0)
-			(effects
-				(font
-					(face "Consolas")
-					(size 1.016 1.016)
-					(thickness 0.127)
-				)
-				(hide yes)
-			)
-		)
-		(property "MFT" "Essentra"
-			(at 139.7 165.1 0)
-			(effects
-				(font
-					(face "Consolas")
-					(size 1.016 1.016)
-				)
-				(hide yes)
-			)
-		)
-		(property "MNP" "50M025045P012"
-			(at 139.7 165.1 0)
-			(effects
-				(font
-					(face "Consolas")
-					(size 1.016 1.016)
-				)
-				(hide yes)
-			)
-		)
-		(instances
-			(project "HW.ACIM-INV"
-				(path "/20f80521-75f2-4ccc-bb34-c9566e70ef5c"
-					(reference "SH10")
-					(unit 1)
-				)
-			)
-		)
-	)
 	(symbol
 		(lib_id "SAMPI:SCREWHOLDER")
@@
 			(effects
 				(font
-					(size 1.27 1.27)
+					(face "Consolas")
+					(size 1.016 1.016)
+					(thickness 0.254)
 				)
 				(justify right)
@@
 			(effects
 				(font
-					(size 1.27 1.27)
-				)
-				(justify right)
+					(face "Consolas")
+					(size 1.016 1.016)
+					(thickness 0.254)
+				)
+				(justify right)

Commit message: V1 schematic update 23
Other:
- moved on the sheet: SH1, SH2, SH3, SH4, SH5, SH6, SH7, SH8, SH9

Commit message: V1 schematic update 25
Other:
- sheet INVERTER ports: added MC_IDC_HAL; removed MC_IDC_N, MC_IDC_P
- sheet POWER MEASUREMENT ports: added MC_IDC_HAL; removed MC_IDC_N, MC_IDC_P
Changed lines of the file:
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@@
 		)
 	)
+	(wire
+		(pts
+			(xy 209.55 103.505) (xy 209.55 110.49)
+		)
+		(stroke
+			(width 0)
+			(type default)
+		)
+	)
 	(polyline
 		(pts
@@
 		)
 	)
-	(wire
-		(pts
-			(xy 209.55 103.505) (xy 209.55 110.49)
-		)
-		(stroke
-			(width 0)
-			(type default)
-		)
-	)
 	(polyline
 		(pts
@@
 		)
 	)
-	(wire
-		(pts
-			(xy 207.01 103.505) (xy 207.01 110.49)
-		)
-		(stroke
-			(width 0)
-			(type default)
-		)
-	)
 	(polyline
 		(pts
@@
 			)
 		)
-		(pin "MC_IDC_P" output
-			(at 207.01 103.505 270)
-			(effects
-				(font
-					(face "Consolas")
-					(size 1.016 1.016)
-					(thickness 0.127)
-				)
-				(justify left)
-			)
-		)
-		(pin "MC_IDC_N" output
-			(at 209.55 103.505 270)
-			(effects
-				(font
-					(face "Consolas")
-					(size 1.016 1.016)
-					(thickness 0.127)
-				)
-				(justify left)
-			)
-		)
 		(pin "MC_PWM_UL" input
 			(at 158.75 70.485 180)
@@
 			)
 		)
+		(pin "MC_IDC_HAL" output
+			(at 209.55 103.505 270)
+			(effects
+				(font
+					(size 1.016 1.016)
+				)
+				(justify left)
+			)
+		)
 		(instances
 			(project "HW.ACIM-INV"
@@
 			)
 		)
-		(pin "MC_IDC_P" input
-			(at 207.01 110.49 90)
-			(effects
-				(font
-					(face "Consolas")
-					(size 1.016 1.016)
-					(thickness 0.127)
-				)
-				(justify right)
-			)
-		)
-		(pin "MC_IDC_N" input
-			(at 209.55 110.49 90)
-			(effects
-				(font
-					(face "Consolas")
-					(size 1.016 1.016)
-					(thickness 0.127)
-				)
-				(justify right)
-			)
-		)
 		(pin "MC_IV_HAL" input
 			(at 214.63 110.49 90)
@@
 			)
 		)
+		(pin "MC_IDC_HAL" input
+			(at 209.55 110.49 90)
+			(effects
+				(font
+					(size 1.016 1.016)
+				)
+				(justify right)
+			)
+		)

Commit message: Label & Case
Parts:
- J1: now not fitted
