File: V1/Design/HW.ACIM-INV/INVPOWER.kicad_sch (KiCad schematic)
At the start: 50 parts, among them J1 AC POWER INPUT, M4 470V/1.2kA, M5 470V/1.2kA, M6 470V/1.2kA, M7 470V/1.2kA, Q10 20V/1A, Q11 20V/1A, U4 SMPS 16V±2%/0.6A

Commit message: V1 schematic update 14
Parts:
- added C72: 10uF, SAMPI:CAP0603, symbol SAMPI:CERCAP
- added D11, D16: 6V3, symbol SAMPI:DIODE-ZEN
- added R16: 1M, SAMPI:RES1206, symbol SAMPI:RES
- added U14: LDO 5V±1%, SAMPI:SOT-89, symbol SAMPI:LDO_BDxxFA1FP3
Connections:
- net +16V_INV: now also U14.3 (VCC)
- net GND_INV: now also C72.1, U14.2 (GND)
- net PGND: now also R16.2
- net at D21.A, RL1.1 (COIL1): now also D16.K; no longer Q10.3 (D)
- net at D22.A, RL2.1 (COIL1): now also D11.K; no longer Q11.3 (D)
- net at R106.1, RL2.5 (NC): now also R16.1
- net +5V renamed +12V_MCU
- net GND renamed GND_MCU
- new net: D16.A, Q10.3 (D)
- new net: D11.A, Q11.3 (D)
- new net +5V_INV: C72.2, U14.1 (VO)
Other:
- moved on the sheet: C1, C15, C28, C42, C47, C62, C67, C8, C9, D3, FT3, FT6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

Commit message: V1 schematic update 15
Other:
- company: TON DUC THANG UNIVERSITY -> (none)
Changed lines of the file:
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@@
 		(date "2024-09-24")
 		(rev "1.0")
-		(company "TON DUC THANG UNIVERSITY")
-		(comment 1 "Schematic Designed by ...")
-		(comment 2 "PCB Designed by ...")
-		(comment 3 "Approved by ...")
 	)
 	(junction

Commit message: V1 schematic update 16
Parts:
- C1: footprint SAMPI:CAP0603 -> SAMPI:CAP1206; MFT Samsung -> (none); MNP CL10A106MQ8NNNC -> (none)
- R3, R92, R94: value 100K -> 10K; MFT YAGEO -> (none); MNP RC0603FR-07100KL -> (none)
Other:
- moved on the sheet: C1, C15, C28, C42, C47, C62, C67, C72, C8, C9, D3, FT3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

Commit message: V1 schematic update 17
Parts:
- removed CB2: CABLE1, symbol SAMPI:CABLE1
- removed F1: 10A, SAMPI:01000056Z, symbol SAMPI:FUSE
- added J2: POWER CONN, symbol SAMPI:FREE_HANGING_CONN
- B1: MFT (none) -> OEM
- C1: renamed from C15; MFT KEMET -> KYAVX; MNP A768MS477M1ELAE017 -> APD1012471M035R
- C12: renamed from C67; value 470uF/35V -> 470uF/25V
- C2: renamed from C1; MFT (none) -> Murata; MNP (none) -> GRT31CR6YA106ME01L
- C6: renamed from C47; now not fitted; now left out of the parts list
- D3: renamed from D11; value 6V3 -> 6V2; footprint (none) -> SAMPI:SOD80C-LL34; MFT (none) -> Diotec; MNP (none) -> ZMM6.2
- D4: renamed from D16; value 6V3 -> 6V2; footprint (none) -> SAMPI:SOD80C-LL34; MFT (none) -> Diotec; MNP (none) -> ZMM6.2
- L1: MFT Bourns Inc. -> Bourns
- MD1: renamed from MD3; footprint SAMPI:LD10-23BxxR2-RC -> SAMPI:HLK-PMxx
- R1: renamed from R3; MFT (none) -> YAGEO; MNP (none) -> RC0603JR-0710KL
- R10: renamed from R92; MFT (none) -> YAGEO; MNP (none) -> RC0603JR-0710KL
- R11: renamed from R94; MFT (none) -> YAGEO; MNP (none) -> RC0603JR-0710KL
- R2: renamed from R9; value 190K, 1% -> 191K, 1%; MNP RC0603FR-07100KL -> RC0603FR-07191KL
- U1: renamed from U4; MFT Microchip Technology -> Microchip
- renumbered C62 to C10, C53 to C11, C56 to C13, C72 to C14, C59 to C15, C61 to C16, C79 to C17, C91 to C18, C28 to C3, C9 to C4, C42 to C5, C8 to C7, C32 to C8, C49 to C9, D3 to D1, D22 to D2, D21 to D5, FT6 to FT1, FT1 to FT2, G2 to G1, J1 to J3, M4 to M1, M5 to M2, M6 to M3, M7 to M4, Q11 to Q1, Q10 to Q2, R10 to R3, R83 to R4, R84 to R5, R85 to R6, R88 to R7, R106 to R8, R16 to R9, RL2 to RL1, RL1 to RL2, U14 to U2
Connections:
- net +24V_INV: now also MD1.4 (DC+); no longer MD1.5 (DC+)
- net GND_INV: now also MD1.3 (DC-); no longer MD1.4 (DC-)
- net at C11.1, C8.2, FT2.3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: now also J3.3

Commit message: V1 schematic update 18
Parts:
- added J12: HIGH VOLTAGE OUTPUTS, SAMPI:HDF1x10x2.54_TH_RA, symbol SAMPI:SIL10
- added J13: INV PWR & RELAYS, SAMPI:HDM1x8x2.54_TH_RA, symbol SAMPI:SIL08
Connections:
- net +16V_INV: now also J13.2
- net +5V_INV: now also J13.4
- net CHASSIS: now also J12.1, J12.2
- net GND_INV: now also J13.1, J13.3
- net PGND: now also J12.4, J12.5, J12.6
- net PWR_RELAY: now also J13.8
- net VDC: now also J12.10, J12.8, J12.9
- net ~{DEV_RELAY}: now also J13.7
Other:
- moved on the sheet: B1, BR1, C1, C10, C11, C12, C13, C14, C15, C16, C17, C18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
