File: V1/Design/HW.ACIM-INV/HW.ACIM-INV.kicad_pcb (KiCad board)
At the start: 4 copper layers, 95 x 95 mm, 252 parts, among them J1 HIGH VOLT, J2 ICSP, J3 MOTOR, J4 LOW VOLT, J6 INV DEBUG, J7 INV DEBUG EXT, J8 ENCODER, J9 USB, M1 560V/1.75kA, M2 560V/1.75kA, M3 560V/1.75kA, Q1 20V/1A, Q3 20V/1A, Q4 20V/1A, Q5 20V/1A, Q6 20V/1A, U1 IPM 600V/15A, U10 I=±10A, U11 256Kbit EEPROM, U12 OP-1CH, U13 128Mbit Flash, U14 LDO 3.3V/1.5A, U15 OP-1CH, U16 OP-1CH, U2 OP-1CH, U3 ISEN 50mV/V, U4 CMP-1CH, U5 MIPS 32-bit DSC, U6 12MHz (3225), U7 I=±10A, U8 LDO 3.3V±0.1%/20mA, U9 I=±10A, X1 32.768kHz

Commit message: V1 schematic update 7
Parts:
- removed BT2: UBT, SAMPI:HDM-2x2.54-TH
- removed FT6: 120R@100MHz, SAMPI:FT0603
- removed G*** (x2): LOGO, LOGO
- removed J4: LOW VOLT, SAMPI:HDM1x10x2.54_TH_RA
- removed J6: INV DEBUG, SAMPI:HDM1x10x2.54_TH_RA
- removed J7: INV DEBUG EXT, SAMPI:HDF1x3x2.54_TH_RA
- removed OP1: OPTO-BJT-4CH, SAMPI:OPTO_SO16_6.5MM
- removed R110: 100K, SAMPI:RES0603
- removed R111: 0R, SAMPI:RES0603
- removed TP1: TEMP, SAMPI:TP1MM
- removed TP10: 24V, SAMPI:TP1MM
- removed TP11: GND1, SAMPI:TP1MM
- removed TP12: 15V, SAMPI:TP1MM
- removed TP13: 5V, SAMPI:TP1MM
- removed TP14: 3V3, SAMPI:TP1MM
- removed TP15: VREF, SAMPI:TP1MM
- removed TP16: VDC, SAMPI:TP1MM
- removed TP17: AVDD, SAMPI:TP1MM
- removed TP18: PGND, SAMPI:TP1MM
- removed TP19: GND, SAMPI:TP1MM
- removed TP2: IU, SAMPI:TP1MM
- removed TP20: AGND, SAMPI:TP1MM
- removed TP3: IV, SAMPI:TP1MM
- removed TP4: IW, SAMPI:TP1MM
- removed TP5: IS, SAMPI:TP1MM
- removed TP6: VS, SAMPI:TP1MM
- removed TP7: VU, SAMPI:TP1MM
- removed TP8: VV, SAMPI:TP1MM
- removed TP9: VW, SAMPI:TP1MM
- removed X1: 32.768kHz, SAMPI:SMD4-7015
- added B1: 220V/50W, SAMPI:LAMP_6.35MM, F.Cu at (63.2, 117.1)
- added BR1: 400V/10A, SAMPI:GBJ25xx, F.Cu at (35.3, 122.0)
- added C102: 1nF, SAMPI:CAP0603, F.Cu at (94.2, 148.7)
- added C103: 1nF, SAMPI:CAP0603, F.Cu at (94.2, 151.3)
- added C104: 100nF, SAMPI:CAP0603, F.Cu at (94.2, 153.9)
- added C105: 1nF, SAMPI:CAP0603, F.Cu at (94.2, 156.5)
- added C106: 1nF, SAMPI:CAP0603, F.Cu at (97.9, 127.8)
- added C107: 10uF/35V, SAMPI:CAP0603, F.Cu at (97.8, 109.7)
- added C108: 10uF, SAMPI:CAP0603, F.Cu at (97.8, 112.3)
- added C109: 100nF, SAMPI:CAP0603, F.Cu at (97.8, 114.9)
- added C110: 3.3nF, SAMPI:CAP0603, F.Cu at (97.8, 117.5)
- added C111: 100nF, SAMPI:CAP0603, F.Cu at (101.5, 94.0)
- added C112: 470uF/35V, SAMPI:CAP_ELEC-10.3x10.3-DIA10, F.Cu at (81.1, 95.5)
- added C77: 100nF, SAMPI:CAP0603, F.Cu at (94.1, 101.8)
- added C80: 10uF, SAMPI:CAP0603, F.Cu at (94.1, 107.1)
- added C82: 10uF/35V, SAMPI:CAP0603, F.Cu at (94.1, 109.7)
- added C84: 100nF, SAMPI:CAP0603, F.Cu at (94.1, 114.9)
- added C85: 3.3nF, SAMPI:CAP0603, F.Cu at (94.1, 117.5)
- added C86: 22pF, SAMPI:CAP0603, F.Cu at (97.8, 94.0)
- added C87: 22pF, SAMPI:CAP0603, F.Cu at (97.8, 96.6)
- added C88: 10uF, SAMPI:CAP0603, F.Cu at (97.8, 99.2)
- added D16: GP DIODE, SAMPI:SOT23, F.Cu at (121.8, 138.3)
- added D17: GP DIODE, SAMPI:SOT23, F.Cu at (117.2, 143.0)
- added D18: 24V, SAMPI:DO-214AA-12, F.Cu at (92.9, 121.5)
- added D19: 24V, SAMPI:SOD-80C_DO-213AC, F.Cu at (99.7, 124.6)
- added D21: 75V/150mA, SAMPI:SOD-323, F.Cu at (122.7, 85.2)
- added D22: 75V/150mA, SAMPI:SOD-323, F.Cu at (122.7, 88.2)
- added D5: GP DIODE, SAMPI:SOT23, F.Cu at (121.8, 133.6)
- added F1: 10A, SAMPI:01000056Z, F.Cu at (113.0, 21.7)
- added FT5: 10mH/500mA, SAMPI:IND-FL2D, F.Cu at (88.4, 42.6)
- added G2: 300V, SAMPI:GDT1812_3532, F.Cu at (122.6, 115.4)
- added L1: 56uH/1A, SAMPI:IND-8D43-8045, F.Cu at (113.0, 97.5)
- added L2: 4.7uH/670mA, SAMPI:IND-R5-2MM-TH, F.Cu at (122.1, 96.0)
- added L3: 22uH/1.5A, SAMPI:IND-8D43-8045, F.Cu at (113.0, 107.1)
- added L4: 4.7uH/670mA, SAMPI:IND-R5-2MM-TH, F.Cu at (122.1, 102.6)
- added L5: 68uH/1A, SAMPI:IND-8D43-8045, F.Cu at (113.0, 116.7)
- added L7: 4.7uH/670mA, SAMPI:IND-R5-2MM-TH, F.Cu at (122.1, 109.2)
- added M4: 470V/1.2kA, SAMPI:MOV5MM, F.Cu at (61.6, 84.9)
- added M5: 470V/1.2kA, SAMPI:MOV5MM, F.Cu at (61.6, 92.1)
- added M6: 470V/1.2kA, SAMPI:MOV5MM, F.Cu at (61.6, 99.4)
- added M7: 470V/1.2kA, SAMPI:MOV5MM, F.Cu at (61.6, 106.6)
- added MD1: AC-DC 24V±2%/10W, SAMPI:LD10-23BxxR2-RC, F.Cu at (46.5, 66.9)
- added MD2: ACIM-MCU, SAMPI:HW.ACIM-MCU, F.Cu at (142.9, 137.3)
- added MD3: DC-DC 15V/24V-24V/42mA, SAMPI:B1524S-1WR3, F.Cu at (119.8, 31.1)
- added MD4: DC-DC 5V-5V/200mA, SAMPI:B1524S-1WR3, F.Cu at (119.8, 38.7)
- added Q10: 20V/1A, SAMPI:SOT23, F.Cu at (99.6, 121.2)
- added Q11: 20V/1A, SAMPI:SOT23, F.Cu at (104.2, 121.2)
- added Q2: 60V/265mA, SAMPI:SOT23, F.Cu at (87.2, 174.0)
- added Q7: 60V/265mA, SAMPI:SOT23, F.Cu at (91.8, 174.0)
- added Q8: 60V/265mA, SAMPI:SOT23, F.Cu at (96.4, 174.0)
- added Q9: 60V/265mA, SAMPI:SOT23, F.Cu at (101.0, 174.0)
- added R100: 10R, SAMPI:RES0603, F.Cu at (109.0, 151.3)
- added R101: 1.1K, SAMPI:RES0603, F.Cu at (109.0, 153.9)
- added R102: 10K, SAMPI:RES0603, F.Cu at (109.0, 156.5)
- added R103: 100K, SAMPI:RES0603, F.Cu at (105.3, 104.5)
- added R104: 53.6K, 1%, SAMPI:RES0603, F.Cu at (105.3, 107.1)
- added R105: 10K, 1%, SAMPI:RES0603, F.Cu at (105.3, 109.7)
- added R106: 1M, SAMPI:RES1206, F.Cu at (81.4, 114.8)
- added R55: 4.3K, SAMPI:RES0603, F.Cu at (90.4, 185.5)
- added R56: 100K, SAMPI:RES0603, F.Cu at (105.3, 138.3)
- added R65: 4.3K, SAMPI:RES0603, F.Cu at (94.2, 177.7)
- added R67: 100K, SAMPI:RES0603, F.Cu at (105.3, 153.9)
- added R74: 1.1K, SAMPI:RES0603, F.Cu at (135.4, 157.3)
- added R75: 100K, SAMPI:RES0603, F.Cu at (73.8, 143.5)
- added R76: 10mR/3W/1%, SAMPI:SHU2512, F.Cu at (62.9, 186.7)
- added R77: 1.1K, SAMPI:RES0603, F.Cu at (109.0, 127.8)
- added R78: 10R, SAMPI:RES0603, F.Cu at (109.0, 130.4)
- added R79: 1.1K, SAMPI:RES0603, F.Cu at (109.0, 133.1)
- added R80: 10R, SAMPI:RES0603, F.Cu at (109.0, 135.7)
- added R81: 1.1K, SAMPI:RES0603, F.Cu at (109.0, 138.3)
- added R82: 100K, SAMPI:RES0603, F.Cu at (101.5, 104.5)
- added R83: 1M, SAMPI:RES1206, F.Cu at (81.4, 103.1)
- added R84: 1M, SAMPI:RES1206, F.Cu at (81.4, 106.0)
- added R85: 1M, SAMPI:RES1206, F.Cu at (81.4, 108.9)
- added R86: 100K, SAMPI:RES0603, F.Cu at (101.5, 107.1)
- added R87: 180K, 1%, SAMPI:RES0603, F.Cu at (101.5, 109.7)
- added R88: 1M, SAMPI:RES1206, F.Cu at (81.4, 111.8)
- added R89: 140K, 1%, SAMPI:RES0603, F.Cu at (101.5, 112.3)
- added R90: 10K, 1%, SAMPI:RES0603, F.Cu at (101.5, 114.9)
- added R91: 10K, SAMPI:RES0603, F.Cu at (101.5, 117.5)
- added R92: 100K, SAMPI:RES0603, F.Cu at (105.3, 94.0)
- added R93: 10K, 1%, SAMPI:RES0603, F.Cu at (105.3, 96.6)
- added R94: 100K, SAMPI:RES0603, F.Cu at (105.3, 99.2)
- added R95: 10K, SAMPI:RES0603, F.Cu at (105.3, 101.8)
- added R96: 100K, SAMPI:RES0603, F.Cu at (109.0, 140.9)
- added R97: 100K, SAMPI:RES0603, F.Cu at (109.0, 143.5)
- added R98: 100K, SAMPI:RES0603, F.Cu at (109.0, 146.1)
- added R99: 100K, SAMPI:RES0603, F.Cu at (109.0, 148.7)
- added RL1: 5V/30A, SAMPI:SLA-12VDC-SL-C, F.Cu at (33.8, 47.3)
- added RL2: 5V/30A, SAMPI:SLA-12VDC-SL-C, F.Cu at (63.7, 47.3)
- added RV1: 10K, Liem:HDM-3x2.54-TH, F.Cu at (154.2, 151.9)
- added U17: LDO 5V±0.4%/250mA, SAMPI:SOT-89, F.Cu at (123.5, 75.3)
- added U18: OP-1CH, SAMPI:SOT353, F.Cu at (112.9, 143.7)
- added U19: OP-1CH, SAMPI:SOT353, F.Cu at (112.9, 147.5)
- added U20: SMPS 5V±2%/1.2A, SAMPI:TDFN8_2x3_MCHP, F.Cu at (83.6, 121.8)
- BT1: value RESET -> UBT
- C1: value 1uF/400V -> 100nF/400V; footprint SAMPI:ECWFE2W105 -> SAMPI:CAP_FILM_6.0x12.0x12.5-P10
- C10, C100, C31, C39, C94: value 100nF -> 1nF
- C101, C43, C47, C97: value 22pF -> 1nF
- C15: value 1nF -> 22pF
- C29, C65, C67: value 1nF -> 100nF
- C32: value 220uF/6.3V -> 1uF/400V; footprint SAMPI:CAP1411 -> SAMPI:ECWFE2W105
- C35: value 100nF -> 22pF
- C44, C45, C46, C58, C69, C76: value 22pF -> 100nF
- C48, C92: value 10uF -> 100nF
- C49: value 22pF -> 100pF/2kV; footprint SAMPI:CAP0603 -> SAMPI:CAP1206
- C53, C61: value 100nF -> 100pF/2kV; footprint SAMPI:CAP0603 -> SAMPI:CAP1206
- C54: value 10uF -> 470uF/35V; footprint SAMPI:CAP0603 -> SAMPI:CAP_ELEC-10.3x10.3-DIA10
- C56: value 3.3nF -> 100pF/2kV; footprint SAMPI:CAP0603 -> SAMPI:CAP1206
- C57, C72: value 22pF -> 10uF
- C59: value 10uF -> 1uF/400V; footprint SAMPI:CAP0603 -> SAMPI:ECWFE2W105
- C62: value 1nF -> 10uF/35V
- C64: value 1nF -> 100pF/2kV; footprint SAMPI:CAP0603 -> SAMPI:CAP1206
- C66: value 100nF -> 3.3nF
- C68: value 1nF -> 47uF/35V; footprint SAMPI:CAP0603 -> SAMPI:CAP_ELEC-6.6x6.6-DIA6.3
- C70: value 22pF -> 10uF/35V
- C71: value 22pF -> 220uF/6.3V; footprint SAMPI:CAP0603 -> SAMPI:CAP1411
- C73: value 47uF/35V -> 10uF; footprint SAMPI:CAP_ELEC-6.6x6.6-DIA6.3 -> SAMPI:CAP0603
- C74: value 100nF -> 10uF
- C75: value 100uF/450V -> 100pF/2kV; footprint SAMPI:CAP_ELEC-18.0x51.5-LS7.5 -> SAMPI:CAP1206
- C79: value 100nF -> 100nF/400V; footprint SAMPI:CAP0603 -> SAMPI:CAP_FILM_6.0x12.0x12.5-P10
- C81, C90: value 22pF -> 470uF/35V; footprint SAMPI:CAP0603 -> SAMPI:CAP_ELEC-10.3x10.3-DIA10
- C83: value 220uF/6.3V -> 10uF; footprint SAMPI:CAP1411 -> SAMPI:CAP0603
- C91: value 22pF -> 680uF/450V; footprint SAMPI:CAP0603 -> SAMPI:ESMQ451VSN681MA50S
- C98: value 9pF -> 1nF
- C99: value 9pF -> 10uF
- D20: value GP DIODE -> 5.1V; footprint SAMPI:SOT23 -> Liem:SOD-123
- D4: value GP DIODE -> 75V/150mA; footprint SAMPI:SOT23 -> SAMPI:SOD-323
- D7: value 75V/150mA -> RUN; footprint SAMPI:SOD-323 -> SAMPI:LED0603
- D8: value RUN -> PWR
- D9: value PWR -> GP DIODE; footprint SAMPI:LED0603 -> SAMPI:SOT23
- FT1: value 120R@100MHz -> 5mH/2.5A; footprint SAMPI:FT0603 -> SAMPI:IND-SQ1010
- FT4: value 2x 120R@100MHz -> 120R@100MHz; footprint SAMPI:IND1210_4P -> SAMPI:FT0603
- J1: value HIGH VOLT -> AC POWER INPUT; footprint SAMPI:HDM1x10x2.54_TH_RA -> SAMPI:TMB3_9.5
- J2: value ICSP -> FAN; footprint SAMPI:HDM1x8x2.54_TH_RA -> SAMPI:HDM-2x2.54-TH
- R1, R2, R4, R51: value 100K -> 10R
- R3: value 1.1K -> 5.2K
- R42: value 10R -> 5.2K
- R43: value 5mR/3W/1% -> 10mR/3W/1%
- R44: value 4.3K -> 1.1K
- R47: value 10K -> 1.1K
- R48: value 100K -> 10K
- R49: value 100K -> 10mR/3W/1%; footprint SAMPI:RES0603 -> SAMPI:SHU2512
- R5: value 10R -> 1.1K
- R50, R59: value 1.1K -> 10R
- R53, R57, R6, R62: value 1.1K -> 100K
- R58: value 100K -> 1.1K
- R7: value 0R -> 1.1K
- R70, R71, R72: value 1.1K -> 4.3K
- R73: value 10K -> 100K
- U1: moved to F.Cu
- U10: value I=±10A -> SMPS 12V±2%/0.8A; footprint SAMPI:SOIC8_ALL -> SAMPI:TDFN8_2x3_MCHP
- U11: value 256Kbit EEPROM -> 2Mbit SRAM
- U13: value 128Mbit Flash -> LDO 3.3V±0.5%/1A; footprint SAMPI:SO8W_5.3 -> SAMPI:DFN8_3x3_MCHP
- U14: value LDO 3.3V/1.5A -> SMPS 15V±2%/0.6A; footprint SAMPI:DFN8_3x3_MCHP -> SAMPI:TDFN8_2x3_MCHP
- U15, U16: value OP-1CH -> I=±10A; footprint SAMPI:SOT353 -> SAMPI:SOIC8_ALL
- U5: value MIPS 32-bit DSC -> ISEN 50mV/V; footprint SAMPI:TQFP64_10x10_MCHP -> SAMPI:SOT363
- U6: value 12MHz (3225) -> ISEN 50mV/V; footprint SAMPI:CDFN3225-4LD-PL-1 -> SAMPI:SOT363
- U7: value I=±10A -> OP-1CH; footprint SAMPI:SOIC8_ALL -> SAMPI:SOT353
- U8: value LDO 3.3V±0.1%/20mA -> OP-1CH; footprint SAMPI:SOT-23-6_MCHP -> SAMPI:SOT353
- U9: value I=±10A -> ISO6740; footprint SAMPI:SOIC8_ALL -> SAMPI:SOIC16-W
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Connections:
- net Net-(U1-ITR) renamed /Inverter/IPM_PWM_FLT
- BT1 pad 1: /DEBUGGER/~{MCLR} -> /MCU/~{BT_UBT}
- C1 pad 1: PGND -> Net-(MD1-ACN)
- C1 pad 2: VDC -> Net-(MD1-ACL)
- C10 pad 1: Net-(D1-COM) -> AGND
- C10 pad 2: AGND -> /VI Measurement/MC_ALT_IU_SEN
- C100 pad 2: +3V3 -> Net-(U6-OUT)
- C101 pad 1: GND -> Net-(U18-IN-)
- C101 pad 2: /MCU/SYS_CLK -> Net-(U18-OUT)
- C11 pad 2: Net-(U9-IPN1) -> /Inverter/MC_UW
- C12 pad 1: Net-(U7-IPN1) -> /Inverter/MC_UV
- C13 pad 1: Net-(U10-IPN1) -> /Inverter/MC_UU
- C15 pad 2: Net-(U7-FILTER) -> /Inverter/MC_TEMP_SEN
- C18 pad 1: AGND -> Net-(D5-COM)
- C18 pad 2: /Inverter/MC_IPM_TEMP -> Net-(D5-A1)
- C19 pad 1: Net-(U2-VIN-) -> Net-(U2-IN-)
- C19 pad 2: Net-(U2-VOUT) -> Net-(U2-OUT)
- C20 pad 1: /MCU/MC_VU_SENSE -> /VI Measurement/MC_UU_DIV
- C21 pad 2: /MCU/~{INV_FLT_OC} -> /VI Measurement/~{MC_PWM_FLT}
- C25 pad 1: Net-(U12-VIN-) -> Net-(U12-IN-)
- C25 pad 2: Net-(U12-VOUT) -> Net-(U12-OUT)
- C26 pad 1: /MCU/MC_VV_SENSE -> /VI Measurement/MC_UV_DIV
- C29 pad 1: Net-(D20-COM) -> GND
- C29 pad 2: Net-(D20-A1) -> VREF
- C30 pad 2: /Inverter/MC_IDC_SENSE -> /VI Measurement/MC_IV_SEN
- C31 pad 2: +5V -> /MCU/MC_VR_DIV
- C33 pad 2: /DEBUGGER/~{MCLR} -> /MCU/~{BT_UBT}
- C35 pad 2: +3V3 -> /MCU/VBUS
- C37 pad 1: Net-(U15-VIN-) -> Net-(D9-COM)
- C37 pad 2: Net-(U15-VOUT) -> Net-(D9-A1)
- C38 pad 1: /MCU/MC_VW_SENSE -> GND
- C38 pad 2: AGND -> VREF
- C39 pad 2: AVDD -> /VI Measurement/MC_IDC_SEN
- C40 pad 1: Net-(D4-COM) -> Net-(D16-COM)
- C43 pad 1: AGND -> Net-(U7-IN-)
- C43 pad 2: /Inverter/MC_IDC_SENSE -> Net-(U7-OUT)
- C44 pad 1: AGND -> /VI Measurement/MC_UW_DIV
- C44 pad 2: /Inverter/MC_IW_SENSE -> AGND
- C45 pad 1: AGND -> Net-(D17-COM)
- C45 pad 2: /Inverter/MC_IV_SENSE -> AGND
- C46 pad 2: /Inverter/MC_IU_SENSE -> AVDD
- C47 pad 1: AGND -> Net-(U8-IN-)
- C47 pad 2: /MCU/MC_VDC_SENSE -> Net-(U8-OUT)
- C48 pad 1: GND -> /VI Measurement/MC_UDC_DIV
- C48 pad 2: +5V -> AGND
- C49 pad 1: AGND -> Net-(C32-Pad1)
- C49 pad 2: +5V -> CHASSIS
- C50 pad 1: AGND -> GND
- C50 pad 2: +5V -> +24V
- C53 pad 1: AGND -> Net-(C32-Pad2)
- C53 pad 2: VREF -> CHASSIS
- C55 pad 1: AGND -> GND
- C55 pad 2: VREF -> Net-(MD4-VI+)
- C56 pad 1: GND -> AC1
- C56 pad 2: +3V3 -> CHASSIS
- C57 pad 2: +3V3 -> Net-(U10-VCC)
- C58 pad 1: AGND -> GND
- C58 pad 2: AVDD -> +15V
- C59 pad 1: AGND -> AC2
- C59 pad 2: AVDD -> AC1
- C61 pad 1: AGND -> AC2
- C61 pad 2: VREF -> CHASSIS
- C62 pad 1: AGND -> GND
- C62 pad 2: /Inverter/MC_IW_SENSE -> Net-(MD3-VI+)
- C63 pad 1: AGND -> Net-(U10-SW)
- C63 pad 2: VREF -> Net-(U10-BOOST)
- C64 pad 1: AGND -> GND
- C64 pad 2: Net-(U9-FILTER) -> GND1
- C65 pad 1: AGND -> GND
- C65 pad 2: /Inverter/MC_IV_SENSE -> +5V
- C66 pad 1: AGND -> Net-(U10-VFB)
- C66 pad 2: VREF -> +12V
- C67 pad 1: AGND -> GND1
- C67 pad 2: Net-(U10-FILTER) -> +24V_ISO
- C69 pad 1: AGND -> GND
- C69 pad 2: /MCU/MC_VU_SENSE -> +12V
- C70 pad 1: AGND -> GND
- C70 pad 2: /MCU/MC_VV_SENSE -> +24V
- C72 pad 1: AGND -> GND
- C72 pad 2: /Inverter/MC_IPM_TEMP -> +5V
- C74 pad 1: GND1 -> GND
- C74 pad 2: +24V -> +3V3
- C76 pad 1: GND -> GND1
- C76 pad 2: Net-(C76-Pad2) -> +5V_ISO
- C78 pad 2: +5V -> +3V3
- C79 pad 1: GND -> PGND
- C79 pad 2: Net-(U14-CDELAY) -> VDC
- C8 pad 1: Net-(U16-VIN-) -> Net-(D1-COM)
- C8 pad 2: Net-(U16-VOUT) -> Net-(D1-A1)
- C89 pad 2: Net-(U5-VDD1) -> +15V
- C9 pad 1: /MCU/MC_VDC_SENSE -> GND
- C9 pad 2: AGND -> VREF
- C92 pad 2: Net-(U5-VDD1) -> +24V
- C93 pad 2: Net-(U5-VDD1) -> VREF
- C94 pad 2: Net-(U5-VDD1) -> Net-(U15-FILTER)
- C95 pad 2: VREF -> AVDD
- C96 pad 2: Net-(U5-VDD1) -> VREF
- C97 pad 2: /MCU/VBUS -> Net-(U16-FILTER)
- C98 pad 1: GND -> AGND
- C98 pad 2: /MCU/SOSCI -> /VI Measurement/MC_IU_SEN
- C99 pad 2: /MCU/SOSCO -> VREF
- D1 pad 1: AGND -> Net-(D1-A1)
- D1 pad 2: AVDD -> Net-(D1-A1)
- D10 pad 2: /DEBUGGER/PWM_UH -> /Inverter/MC_PWM_UH
- D10 pad 3: /DEBUGGER/PWM_VH -> /Inverter/MC_PWM_VH
- D11 pad 2: /DEBUGGER/PWM_VL -> /Inverter/MC_PWM_VL
- D11 pad 3: /DEBUGGER/PWM_UL -> /Inverter/MC_PWM_UL
- D15 pad 2: /DEBUGGER/PWM_WL -> /Inverter/MC_PWM_WL
- D15 pad 3: /DEBUGGER/PWM_WH -> /Inverter/MC_PWM_WH
- D7 pad A: Net-(BZ1-V-) -> /MCU/IND_RUN
- D7 pad K: +5V -> Net-(D7-PadK)
- D8 pad A: /DEBUGGER/IND_RUN -> +3V3
- FT1 pad 1: AGND -> Net-(C32-Pad1)
- FT1 pad 2: GND -> AC2
- FT2 pad 1: GND -> AGND
- FT2 pad 2: PGND -> GND
- FT3 pad 1: +3V3 -> GND
- FT3 pad 2: AVDD -> PGND
- FT4 pad 1: /MCU/USB1_P -> +3V3
- FT4 pad 2: /MCU/USB_P -> AVDD
- J1 pad 1: VDC -> CHASSIS
- J1 pad 2: VDC -> Net-(C32-Pad1)
- J1 pad 3: VDC -> Net-(F1-Pad1)
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Routing:
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Other:
- board size 95 x 95 mm -> 154 x 178.5 mm
- board text removed: "HW.ACIM-INV-R0.1"

Commit message: V1 schematic update 8
Parts:
- removed C101, C105, C19, C25, C43, C47: 1nF, SAMPI:CAP0603
- removed R101, R36, R60, R79, R81: 1.1K, SAMPI:RES0603
- FT5: value 10mH/500mA -> 15mH/500mA; footprint SAMPI:IND-FL2D -> SAMPI:EE8.3
- moved FT5 11.8 mm to (94.7, 52.6)
Connections:
- R10 pad 1: Net-(U2-IN-) -> Net-(U4-VIN-)
- R10 pad 2: /VI Measurement/MC_UU_DIV -> /VI Measurement/MC_IDC_SEN
- R100 pad 2: Net-(U19-OUT) -> Net-(U19-IN-)
- R32 pad 2: Net-(U2-OUT) -> Net-(U2-IN-)
- R38 pad 2: Net-(U12-OUT) -> Net-(U12-IN-)
- R59 pad 2: Net-(U7-OUT) -> Net-(U7-IN-)
- R78 pad 2: Net-(U8-OUT) -> Net-(U8-IN-)
- R80 pad 2: Net-(U18-OUT) -> Net-(U18-IN-)
- U12 pad 4: Net-(U12-OUT) -> Net-(U12-IN-)
- U18 pad 4: Net-(U18-OUT) -> Net-(U18-IN-)
- U19 pad 4: Net-(U19-OUT) -> Net-(U19-IN-)
- U2 pad 4: Net-(U2-OUT) -> Net-(U2-IN-)
- U4 pad 1: /VI Measurement/MC_IDC_SEN -> Net-(U4-VIN-)
- U7 pad 4: Net-(U7-OUT) -> Net-(U7-IN-)
- U8 pad 4: Net-(U8-OUT) -> Net-(U8-IN-)

Commit message: V1 schematic update 9
Parts:
- removed C35: 22pF, SAMPI:CAP0603
- removed J9: USB, SAMPI:HDM-1x4x1.25-TH
- removed R74: 1.1K, SAMPI:RES0603
- removed TP23: VUSB, SAMPI:TP1MM
- added J4: MCDBG, SAMPI:IDC-2x5x2MM-TH, F.Cu at (144.8, 98.8)
Connections:
- C10 pad 2: /VI Measurement/MC_ALT_IU_SEN -> /MCU/MC_ALT_IU_SEN
- C106 pad 2: /VI Measurement/MC_ALT_IV_SEN -> /MCU/MC_ALT_IV_SEN
- C20 pad 1: /VI Measurement/MC_UU_DIV -> /MCU/MC_UU_DIV
- C21 pad 2: /VI Measurement/~{MC_PWM_FLT} -> /MCU/~{MC_PWM_FLT}
- C26 pad 1: /VI Measurement/MC_UV_DIV -> /MCU/MC_UV_DIV
- C30 pad 2: /VI Measurement/MC_IV_SEN -> /MCU/MC_IV_SEN
- C39 pad 2: /VI Measurement/MC_IDC_SEN -> /MCU/MC_IDC_SEN
- C44 pad 1: /VI Measurement/MC_UW_DIV -> /MCU/MC_UW_DIV
- C48 pad 1: /VI Measurement/MC_UDC_DIV -> /MCU/MC_UDC_DIV
- C98 pad 2: /VI Measurement/MC_IU_SEN -> /MCU/MC_IU_SEN
- MD2 pad R1: /MCU/VBUS -> unconnected-(MD2B-VBUS-PadR1)
- MD2 pad R10: /MCU/TXD2 -> /MCU/DV_TXD
- MD2 pad R11: /MCU/RTS2 -> /MCU/DV_RTS
- MD2 pad R12: /MCU/CTS2 -> /MCU/DV_CTS
- MD2 pad R15: /MCU/MC_PWM_WH -> /Inverter/MC_PWM_WH
- MD2 pad R16: /MCU/MC_PWM_VL -> /Inverter/MC_PWM_VL
- MD2 pad R17: /MCU/MC_PWM_VH -> /Inverter/MC_PWM_VH
- MD2 pad R18: /MCU/MC_PWM_WL -> /Inverter/MC_PWM_WL
- MD2 pad R19: /MCU/MC_PWM_UH -> /Inverter/MC_PWM_UH
- MD2 pad R20: /MCU/MC_PWM_UL -> /Inverter/MC_PWM_UL
- MD2 pad R21: /MCU/MC_TEMP_SEN -> /Inverter/MC_TEMP_SEN
- MD2 pad R3: /MCU/USB_N -> unconnected-(MD2B-USB_N-PadR3)
- MD2 pad R5: /MCU/USB_P -> unconnected-(MD2B-USB_P-PadR5)
- MD2 pad R7: /MCU/RXD1 -> unconnected-(MD2B-DB_RXD-PadR7)
- MD2 pad R8: /MCU/TXD1 -> /MCU/DB_TXD
- MD2 pad R9: /MCU/RXD2 -> /MCU/DV_RXD
- Q1 pad 1: /VI Measurement/~{MC_PWM_FLT} -> /MCU/~{MC_PWM_FLT}
- Q1 pad 3: /VI Measurement/MC_PWM_FLT -> /Inverter/MC_PWM_FLT
- R1 pad 2: /VI Measurement/MC_IU_SEN_P -> /Inverter/MC_IU_SEN_P
- R10 pad 2: /VI Measurement/MC_IDC_SEN -> /MCU/MC_IDC_SEN
- R100 pad 1: /VI Measurement/MC_ALT_IV_SEN -> /MCU/MC_ALT_IV_SEN
- R2 pad 2: /VI Measurement/MC_IU_SEN_N -> /Inverter/MC_IU_SEN_N
- R27 pad 2: /VI Measurement/~{MC_PWM_FLT} -> /MCU/~{MC_PWM_FLT}
- R3 pad 2: /VI Measurement/MC_IU_SEN -> /MCU/MC_IU_SEN
- R32 pad 1: /VI Measurement/MC_UU_DIV -> /MCU/MC_UU_DIV
- R34 pad 1: /VI Measurement/MC_UV -> /Inverter/MC_UV
- R38 pad 1: /VI Measurement/MC_UV_DIV -> /MCU/MC_UV_DIV
- R40 pad 2: /VI Measurement/MC_IV_SEN_P -> /Inverter/MC_IV_SEN_P
- R41 pad 2: /VI Measurement/MC_IV_SEN_N -> /Inverter/MC_IV_SEN_N
- R42 pad 2: /VI Measurement/MC_IV_SEN -> /MCU/MC_IV_SEN
- R50 pad 2: /VI Measurement/MC_IDC_SEN_P -> /Inverter/MC_IDC_SEN_P
- R51 pad 2: /VI Measurement/MC_IDC_SEN_N -> /Inverter/MC_IDC_SEN_N
- R52 pad 2: /VI Measurement/MC_IDC_SEN -> /MCU/MC_IDC_SEN
- R53 pad 1: /VI Measurement/MC_UW -> /Inverter/MC_UW
- R54 pad 2: /VI Measurement/MC_PWM_FLT -> /Inverter/MC_PWM_FLT
- R59 pad 1: /VI Measurement/MC_UW_DIV -> /MCU/MC_UW_DIV
- R78 pad 1: /VI Measurement/MC_UDC_DIV -> /MCU/MC_UDC_DIV
- R8 pad 1: /VI Measurement/MC_UU -> /Inverter/MC_UU
- R80 pad 1: /VI Measurement/MC_ALT_IU_SEN -> /MCU/MC_ALT_IU_SEN
- R91 pad 1: /POWER/PWR_RELAY -> /MCU/PWR_RELAY
- R95 pad 1: /POWER/~{DEV_RELAY} -> /MCU/~{DEV_RELAY}
- R97 pad 1: /VI Measurement/MC_IU_HAL -> /Inverter/MC_IU_HAL
- R98 pad 1: /VI Measurement/MC_IV_HAL -> /Inverter/MC_IV_HAL

Commit message: V1 schematic update 17
Parts:
- removed BT1: UBT, SAMPI:HDM-2x2.54-TH
- removed BZ1: BUZZER, SAMPI:SMT-0827-S-HT-R
- removed C100, C102, C103, C106, C94, C97, C98: 1nF, SAMPI:CAP0603
- removed C104, C109, C111, C89, C92, C93, C95, C96: 100nF, SAMPI:CAP0603
- removed C107: 10uF/35V, SAMPI:CAP0603
- removed C108, C88, C99: 10uF, SAMPI:CAP0603
- removed C110: 3.3nF, SAMPI:CAP0603
- removed C112, C90: 470uF/35V, SAMPI:CAP_ELEC-10.3x10.3-DIA10
- removed C91: 680uF/450V, SAMPI:ESMQ451VSN681MA50S
- removed D21, D22: 75V/150mA, SAMPI:SOD-323
- removed F1: 10A, SAMPI:01000056Z
- removed J2: FAN, SAMPI:HDM-2x2.54-TH
- removed J8: ENCODER, SAMPI:HDM1x8x2.0_SMA_RA
- removed L3: 22uH/1.5A, SAMPI:IND-8D43-8045
- removed L4, L7: 4.7uH/670mA, SAMPI:IND-R5-2MM-TH
- removed L5: 68uH/1A, SAMPI:IND-8D43-8045
- removed MD4: DC-DC 5V-5V/200mA, SAMPI:B1524S-1WR3
- removed Q10, Q11: 20V/1A, SAMPI:SOT23
- removed Q8, Q9: 60V/265mA, SAMPI:SOT23
- removed R100, R59, R78, R80: 10R, SAMPI:RES0603
- removed R102, R91, R95: 10K, SAMPI:RES0603
- removed R103, R62, R67, R73, R75, R82, R86, R92, R94, R96, R97, R98, R99: 100K, SAMPI:RES0603
- removed R104: 53.6K, 1%, SAMPI:RES0603
- removed R105, R90, R93: 10K, 1%, SAMPI:RES0603
- removed R106, R83, R84, R85, R88: 1M, SAMPI:RES1206
- removed R61, R65, R70, R71, R72: 4.3K, SAMPI:RES0603
- removed R63, R68, R69: 4.7R, SAMPI:RES1206
- removed R64, R66, R77: 1.1K, SAMPI:RES0603
- removed R76: 10mR/3W/1%, SAMPI:SHU2512
- removed R87: 180K, 1%, SAMPI:RES0603
- removed R89: 140K, 1%, SAMPI:RES0603
- removed U20: SMPS 5V±2%/1.2A, SAMPI:TDFN8_2x3_MCHP
- added C19: 10uF/35V, SAMPI:CAP1206, F.Cu at (150.5, 132.1)
- added C25: 470uF/35V, SAMPI:CAP_ELEC-10.3x10.3-DIA10, F.Cu at (122.4, 119.4)
- added C35: 100nF, SAMPI:CAP0603, F.Cu at (109.3, 119.8)
- added C43: 100nF, SAMPI:CAP0603, F.Cu at (147.0, 55.7)
- added C47: 10uF, SAMPI:CAP0603, F.Cu at (147.0, 66.1)
- added J11: ENCODER, SAMPI:HDM1x8x2.0_SMA_RA, F.Cu at (114.6, 146.7)
- added J5: MOTOR, SAMPI:TMB4_9.5, F.Cu at (124.5, 58.5)
- added OP1: OPTO-BJT-1CH, SAMPI:OPTO_SO4_7.6MM, F.Cu at (163.2, 58.1)
- added R36: 10R, 1%, SAMPI:RES0603, F.Cu at (35.6, 128.6)
- C1: value 100nF/400V -> 470uF/35V; footprint SAMPI:CAP_FILM_6.0x12.0x12.5-P10 -> SAMPI:CAP_ELEC-10.3x10.3-DIA10
- C10: value 1nF -> 100nF
- C12: value 100pF/2kV -> 470uF/25V; footprint SAMPI:CAP1206 -> SAMPI:CAP_ELEC-10.3x10.3-DIA10
- C14, C53: value 100pF/2kV -> 10uF; footprint SAMPI:CAP1206 -> SAMPI:CAP0603
- C15: value 22pF -> 1uF/400V; footprint SAMPI:CAP0603 -> SAMPI:ECWFE2W105
- C16: value 470uF -> 100pF/2kV; footprint SAMPI:CAP_ELEC-10.3x10.3-DIA10 -> SAMPI:CAP1206
- C17, C7: value 100nF -> 100nF/400V; footprint SAMPI:CAP0603 -> SAMPI:CAP_FILM_6.0x12.0x12.5-P10
- C18: value 1nF -> 680uF/450V; footprint SAMPI:CAP0603 -> SAMPI:ESMQ451VSN681MA50S
- C2, C28, C29: value 100nF -> 10uF/35V; footprint SAMPI:CAP0603 -> SAMPI:CAP1206
- C20, C46, C48: value 100nF -> 10uF
- C21: value 1nF -> 100nF/400V; footprint SAMPI:CAP0603 -> SAMPI:CAP_FILM_6.0x12.0x12.5-P10
- C23: value 100nF -> 3.3nF
- C27: value 100nF -> 470uF/16V; footprint SAMPI:CAP0603 -> SAMPI:CAP_ELEC-8.3x8.3-DIA8.0
- C3: value 47uF/35V -> 10uF; footprint SAMPI:CAP_ELEC-6.6x6.6-DIA6.3 -> SAMPI:CAP0603
- C30, C31, C37: value 1nF -> 10uF
- C32: value 1uF/400V -> 100nF; footprint SAMPI:ECWFE2W105 -> SAMPI:CAP0603
- C34: value 100nF -> 220uF/6.3V; footprint SAMPI:CAP0603 -> SAMPI:CAP1411
- C36, C51: value 22pF -> 100nF
- C38, C40: value 100nF -> 47uF/35V; footprint SAMPI:CAP0603 -> SAMPI:CAP_ELEC-6.6x6.6-DIA6.3
- C39: value 1nF -> 47uF/35V; footprint SAMPI:CAP0603 -> SAMPI:CAP_ELEC-6.6x6.6-DIA6.3
- C4, C68: value 47uF/35V -> 100nF; footprint SAMPI:CAP_ELEC-6.6x6.6-DIA6.3 -> SAMPI:CAP0603
- C41: value 100nF -> 470uF/25V; footprint SAMPI:CAP0603 -> SAMPI:CAP_ELEC-10.3x10.3-DIA10
- C50: value 100nF -> 470nF/630V; footprint SAMPI:CAP0603 -> SAMPI:FCAP-15MM
- C52: value 22pF -> 1nF
- C54: value 470uF/35V -> 10uF; footprint SAMPI:CAP_ELEC-10.3x10.3-DIA10 -> SAMPI:CAP0603
- C56, C61: value 100pF/2kV -> 100nF; footprint SAMPI:CAP1206 -> SAMPI:CAP0603
- C57, C74: value 10uF -> 1nF
- C58, C9: value 100nF -> 100pF/2kV; footprint SAMPI:CAP0603 -> SAMPI:CAP1206
- C59: value 1uF/400V -> 100pF/2kV; footprint SAMPI:ECWFE2W105 -> SAMPI:CAP1206
- C6: value 47uF/35V -> 3.3nF; footprint SAMPI:CAP_ELEC-6.6x6.6-DIA6.3 -> SAMPI:CAP0603
- C60: value 22pF -> 100pF/2kV; footprint SAMPI:CAP0603 -> SAMPI:CAP1206
- C62: value 10uF/35V -> 100nF
- C64, C75: value 100pF/2kV -> 1nF; footprint SAMPI:CAP1206 -> SAMPI:CAP0603
- C65, C76, C77, C78: value 100nF -> 1nF
- C66: value 3.3nF -> 100nF
- C70, C82: value 10uF/35V -> 1nF
- C71: value 220uF/6.3V -> 1nF; footprint SAMPI:CAP1411 -> SAMPI:CAP0603
- C72, C73, C80: value 10uF -> 100nF
- C79: value 100nF/400V -> 100nF; footprint SAMPI:CAP_FILM_6.0x12.0x12.5-P10 -> SAMPI:CAP0603
- C8: value 1nF -> 1uF/400V; footprint SAMPI:CAP0603 -> SAMPI:ECWFE2W105
- C81: value 470uF/35V -> 1nF; footprint SAMPI:CAP_ELEC-10.3x10.3-DIA10 -> SAMPI:CAP0603
- C83: value 10uF -> 10uF/35V; footprint SAMPI:CAP0603 -> SAMPI:CAP1206
- C84: value 100nF -> 22pF
- C85: value 3.3nF -> 22pF
- D1: value GP DIODE -> 24V; footprint SAMPI:SOT23 -> SAMPI:DO-214AA-12
- D10: value TVS 5.5V 3-CH -> TVS 5.5V
- D11: value TVS 5.5V 3-CH -> PV; footprint SAMPI:SOT143B_NEXT -> SAMPI:LED0603
- D12: value PU -> PW
- D13: value PV -> PU
- D14: value PW -> GP DIODE; footprint SAMPI:LED0603 -> SAMPI:SOT23
- D15: value TVS 5.5V 3-CH -> GP DIODE; footprint SAMPI:SOT143B_NEXT -> SAMPI:SOT23
- D17: value GP DIODE -> ERR; footprint SAMPI:SOT23 -> SAMPI:LED0603
- D18: value 24V -> RUN; footprint SAMPI:DO-214AA-12 -> SAMPI:LED0603
- D19: value 24V -> TVS 5.5V; footprint SAMPI:SOD-80C_DO-213AC -> SAMPI:SOT143B_NEXT
- D2, D5: value GP DIODE -> 75V/150mA; footprint SAMPI:SOT23 -> SAMPI:SOD-323
- D20: value 5.1V -> TVS 5.5V; footprint Liem:SOD-123 -> SAMPI:SOT143B_NEXT
- D3: value GP DIODE -> 6V2; footprint SAMPI:SOT23 -> SAMPI:SOD80C-LL34
- D4: value 75V/150mA -> 6V2; footprint SAMPI:SOD-323 -> SAMPI:SOD80C-LL34
- D6: value ERR -> 24V; footprint SAMPI:LED0603 -> SAMPI:DO-214AA-12
- D7: value RUN -> PWR
- D8: value PWR -> TVS 5.5V; footprint SAMPI:LED0603 -> SAMPI:SOT143B_NEXT
- D9: value GP DIODE -> TVS 5.5V; footprint SAMPI:SOT23 -> SAMPI:SOT143B_NEXT
- FT1: value 5mH/2.5A -> 15mH/500mA; footprint SAMPI:IND-SQ1010 -> SAMPI:EE8.3
- FT2: value 120R@100MHz -> 5mH/2.5A; footprint SAMPI:FT0603 -> SAMPI:IND-SQ1010
- FT4: value 120R@100MHz -> 15mH/500mA; footprint SAMPI:FT0603 -> SAMPI:EE8.3
- FT5: value 15mH/500mA -> 120R@100MHz; footprint SAMPI:EE8.3 -> SAMPI:FT0603
- J1: value AC POWER INPUT -> MCDBG; footprint SAMPI:TMB3_9.5 -> SAMPI:IDC-2x6x2.54MM_TH
- J3: value MOTOR -> AC POWER INPUT; footprint SAMPI:TMB4_9.5 -> SAMPI:TMB3_9.5
- J4: value MCDBG -> FAN; footprint SAMPI:IDC-2x5x2MM-TH -> SAMPI:HDM-2x2.54-TH
- L1: value 56uH/1A -> 68uH/1A
- L2: value 4.7uH/670mA -> 56uH/1A; footprint SAMPI:IND-R5-2MM-TH -> SAMPI:IND-8D43-8045
- M1, M2, M3: value 560V/1.75kA -> 470V/1.2kA
- M5, M6, M7: value 470V/1.2kA -> 560V/1.75kA
- MD1: value AC-DC 24V±2%/10W -> 24V±2%/3W; footprint SAMPI:LD10-23BxxR2-RC -> SAMPI:HLK-PMxx
- MD2: value ACIM-MCU -> 24V±2%/10W; footprint SAMPI:HW.ACIM-MCU -> SAMPI:HLK-10M
- MD3: value DC-DC 15V/24V-24V/42mA -> ACIM-MCU; footprint SAMPI:B1524S-1WR3 -> SAMPI:HW.ACIM-MCU
- Q2: value 60V/265mA -> 20V/1A
- Q4, Q5, Q6: value 20V/1A -> 60V/265mA
- R1: value 10R -> 10K
- R10, R11, R22: value 1.1K -> 10K
- R12, R16: value 100K -> 10K
- R13: value 1.1K -> 140K, 1%
- R14: value 1.1K -> 10K, 1%
- R15, R19, R20: value 1.1K -> 1K
- R17: value 100K -> 10mR/3W/1%; footprint SAMPI:RES0603 -> SAMPI:SHU2512
- R18, R24: value 100K -> 1K
- R2: value 10R -> 191K, 1%
- R21: value 1.1K -> 4.7R; footprint SAMPI:RES0603 -> SAMPI:RES1206
- R23, R26: value 100K -> 4.7R; footprint SAMPI:RES0603 -> SAMPI:RES1206
- R25: value 100K -> 1.2M
- R27: value 10R -> 100K, 1%
- R28: value 100K -> 100K, 1%
- R29, R44: value 1.1K -> 100K, 1%
- R3: value 5.2K -> 10K, 1%
- R30: value 1M -> 1.1K, 1%; footprint SAMPI:RES1206 -> SAMPI:RES0603
- R31: value 470K -> 10R, 1%
- R32, R41: value 10R -> 10R, 1%
- R33, R47: value 1.1K -> 10R, 1%
- R34, R35: value 100K -> 10R, 1%
- R37: value 100K -> 10K, 1%
- R38: value 10R -> 10K, 1%
- R39: value 1.1K -> 4.99K, 1%
- R4: value 10R -> 1M; footprint SAMPI:RES0603 -> SAMPI:RES1206
- R40: value 10R -> 4.99K, 1%
- R42: value 5.2K -> 10R, 1%
- R43: value 10mR/3W/1% -> 100K, 1%; footprint SAMPI:SHU2512 -> SAMPI:RES0603
- R45, R46: value 4.3K -> 100K, 1%
- R48: value 10K -> 10R, 1%
- R49: value 10mR/3W/1% -> 1K; footprint SAMPI:SHU2512 -> SAMPI:RES0603
- R5, R7: value 1.1K -> 1M; footprint SAMPI:RES0603 -> SAMPI:RES1206
- R50: value 10R -> 1K
- R51, R52: value 10R -> 2.2K
- R53, R56, R57: value 100K -> 2.2K
- R54: value 10K -> 2.2K
- R55: value 4.3K -> 2.2K
- R58: value 1.1K -> 2.2K
- R6, R8, R9: value 100K -> 1M; footprint SAMPI:RES0603 -> SAMPI:RES1206
- RV1: value 10K -> 20K; footprint Liem:HDM-3x2.54-TH -> SAMPI:TC33X-2
- U1: value IPM 600V/15A -> SMPS 16V±2%/0.6A; footprint SAMPI:CIPOS-MINI -> SAMPI:TDFN8_2x3_MCHP
- U10: value SMPS 12V±2%/0.8A -> DIGI ISO; footprint SAMPI:TDFN8_2x3_MCHP -> SAMPI:SOIC8_ALL
- U11: value 2Mbit SRAM -> I=±10A; footprint SAMPI:SOIC8_3.9_MCHP -> SAMPI:SOIC8_ALL
- U12: value OP-1CH -> I=±10A; footprint SAMPI:SOT353 -> SAMPI:SOIC8_ALL
- U13: value LDO 3.3V±0.5%/1A -> CMP-1CH; footprint SAMPI:DFN8_3x3_MCHP -> SAMPI:SOT25_DIODES
- U14: value SMPS 15V±2%/0.6A -> ISO OPAMP 1-CH; footprint SAMPI:TDFN8_2x3_MCHP -> SAMPI:SOP8-2.54
- U15: value I=±10A -> ISO OPAMP 1-CH; footprint SAMPI:SOIC8_ALL -> SAMPI:SOP8-2.54
- U16: value I=±10A -> ISEN 50mV/V; footprint SAMPI:SOIC8_ALL -> SAMPI:SOT363
- U17: value LDO 5V±0.4%/250mA -> OP-1CH; footprint SAMPI:SOT-89 -> SAMPI:SOT353
- U2: value OP-1CH -> LDO 5V±1%; footprint SAMPI:SOT353 -> SAMPI:SOT-89
- U3: value ISEN 50mV/V -> SMPS 12V±2%/0.8A; footprint SAMPI:SOT363 -> SAMPI:TDFN8_2x3_MCHP
- U4: value CMP-1CH -> LDO 5V±1%; footprint SAMPI:SOT25_DIODES -> SAMPI:SOT-89
- U5: value ISEN 50mV/V -> LDO 3V3±2%; footprint SAMPI:SOT363 -> SAMPI:SOT-223-3
- U6: value ISEN 50mV/V -> LDO 3.3V±0.1%/20mA; footprint SAMPI:SOT363 -> SAMPI:SOT-23-6_MCHP
- U7: value OP-1CH -> IPM 600V/15A; footprint SAMPI:SOT353 -> SAMPI:CIPOS-MINI
- U8: value OP-1CH -> DIGI ISO; footprint SAMPI:SOT353 -> SAMPI:SOIC8_ALL
- U9: value ISO6740 -> DIGI ISO; footprint SAMPI:SOIC16-W -> SAMPI:SOIC8_ALL
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Connections:
- B1 pad 1: Net-(RL1-NC) -> Net-(RL2-NC)
- C10 pad 1: AGND -> GND_INV
- C10 pad 2: /MCU/MC_ALT_IU_SEN -> +16V_INV
- C11 pad 2: /Inverter/MC_UW -> CHASSIS
- C13 pad 1: /Inverter/MC_UU -> AC1
- C13 pad 2: Net-(C13-Pad2) -> CHASSIS
- C14 pad 1: VDC -> GND_INV
- C14 pad 2: PGND -> +5V_INV
- C15 pad 1: AGND -> AC2
- C15 pad 2: /Inverter/MC_TEMP_SEN -> AC1
- C17 pad 1: +15V -> PGND
- C17 pad 2: GND -> VDC
- C2 pad 1: Net-(U1-VBU) -> GND_INV
- C2 pad 2: Net-(U1-VSU) -> +24V_INV
- C20 pad 1: /MCU/MC_UU_DIV -> GND_MCU
- C20 pad 2: AGND -> Net-(U3-VCC)
- C21 pad 1: GND -> Net-(MD2-ACN)
- C21 pad 2: /MCU/~{MC_PWM_FLT} -> Net-(MD2-ACL)
- C22 pad 1: AGND -> Net-(U3-SW)
- C22 pad 2: Net-(C22-Pad2) -> Net-(U3-BOOST)
- C23 pad 1: Net-(D2-COM) -> Net-(U3-VFB)
- C23 pad 2: AGND -> +12V_MCU
- C24 pad 1: AGND -> GND_MCU
- C24 pad 2: AVDD -> +24V_MCU
- C26 pad 1: /MCU/MC_UV_DIV -> GND_MCU
- C26 pad 2: AGND -> +12V_MCU
- C28 pad 1: Net-(D3-COM) -> GND_MCU
- C28 pad 2: AGND -> +12V_MCU
- C29 pad 1: GND -> GND_MCU
- C29 pad 2: VREF -> +12V_MCU
- C30 pad 1: AGND -> GND_MCU
- C30 pad 2: /MCU/MC_IV_SEN -> +5V_MCU
- C31 pad 1: AGND -> GND_MCU
- C31 pad 2: /MCU/MC_VR_DIV -> +5V_MCU
- C32 pad 1: Net-(C32-Pad1) -> GND_MCU
- C32 pad 2: Net-(C32-Pad2) -> +3V3_MCU
- C33 pad 1: GND -> GND_MCU
- C33 pad 2: /MCU/~{BT_UBT} -> +5V_MCU
- C36 pad 1: GND -> GND_ADC
- C36 pad 2: /ENCODER/ENC_HOME -> +3V3_ADC
- C37 pad 1: Net-(D9-COM) -> GND_ADC
- C37 pad 2: Net-(D9-A1) -> +3V3_ADC
- C42 pad 1: AGND -> +16V_INV
- C42 pad 2: AVDD -> GND_INV
- C44 pad 1: /MCU/MC_UW_DIV -> Net-(U7-VBV)
- C44 pad 2: AGND -> Net-(U7-VSV)
- C45 pad 1: Net-(D17-COM) -> Net-(U7-VBW)
- C45 pad 2: AGND -> Net-(U7-VSW)
- C46 pad 1: AGND -> GND_INV
- C46 pad 2: AVDD -> +5V_INV
- C48 pad 1: /MCU/MC_UDC_DIV -> GND_INV
- C48 pad 2: AGND -> +5V_INV
- C49 pad 1: Net-(C32-Pad1) -> VDC
- C49 pad 2: CHASSIS -> PGND
- C5 pad 1: Net-(U1-VBV) -> Net-(U1-SW)
- C5 pad 2: Net-(U1-VSV) -> Net-(U1-BOOST)
- C50 pad 1: GND -> VDC
- C50 pad 2: +24V -> PGND
- C51 pad 1: GND -> GND_MCU
- C51 pad 2: /ENCODER/ENC_A -> +5V_MCU
- C52 pad 1: GND -> GND_MCU
- C52 pad 2: /ENCODER/ENC_B -> Net-(U11-FILTER)
- C53 pad 1: Net-(C32-Pad2) -> GND_MCU
- C53 pad 2: CHASSIS -> +3V3_MCU
- C55 pad 1: GND -> GND_MCU
- C55 pad 2: Net-(MD4-VI+) -> +3V3_MCU
- C56 pad 1: AC1 -> GND_MCU
- C56 pad 2: CHASSIS -> +5V_MCU
- C57 pad 1: GND -> GND_MCU
- C57 pad 2: Net-(U10-VCC) -> Net-(U12-FILTER)
- C58 pad 1: GND -> /INVERTER/MC_U
- C58 pad 2: +15V -> Net-(C58-Pad2)
- C59 pad 1: AC2 -> Net-(C59-Pad1)
- C59 pad 2: AC1 -> /INVERTER/MC_V
- C60 pad 1: GND -> /INVERTER/MC_W
- C60 pad 2: /ENCODER/ENC_INDEX -> Net-(C60-Pad2)
- C61 pad 1: AC2 -> GND_INV
- C61 pad 2: CHASSIS -> +5V_INV
- C62 pad 1: GND -> GND_INV
- C62 pad 2: Net-(MD3-VI+) -> Net-(RV1-WIPER)
- C63 pad 1: Net-(U10-SW) -> GND_INV
- C63 pad 2: Net-(U10-BOOST) -> /INVERTER/IPM_TEMP_SEN
- C64 pad 1: GND -> Net-(D15-COM)
- C64 pad 2: GND1 -> Net-(D15-A1)
- C65 pad 1: GND -> Net-(D16-COM)
- C65 pad 2: +5V -> Net-(D16-A1)
- C66 pad 1: Net-(U10-VFB) -> +5V_INV
- C66 pad 2: +12V -> GND_INV
- C67 pad 1: GND1 -> +5V_INV
- C67 pad 2: +24V_ISO -> GND_INV
- C69 pad 1: GND -> +5V_MCU
- C69 pad 2: +12V -> GND_MCU
- C7 pad 1: Net-(U1-VBW) -> Net-(MD1-ACN)
- C7 pad 2: Net-(U1-VSW) -> Net-(MD1-ACL)
- C70 pad 1: GND -> Net-(U16-IN-)
- C70 pad 2: +24V -> Net-(U16-IN+)
- C72 pad 1: GND -> GND_MCU
- C72 pad 2: +5V -> +5V_MCU
- C73 pad 1: GND_ISO -> GND_MCU
- C73 pad 2: +5V_ISO -> +5V_MCU
- C74 pad 1: GND -> GND_ADC
- C74 pad 2: +3V3 -> /MCU/MC_UDC_DIV
- C75 pad 1: GND -> GND_ADC
- C75 pad 2: GND1 -> Net-(U16-OUT)
- C76 pad 1: GND1 -> GND_ADC
- C76 pad 2: +5V_ISO -> /MCU/MC_IDC_SEN
- C77 pad 1: GND -> GND_MCU
- C77 pad 2: Net-(U13-CDELAY) -> Net-(U18-IN+)
- C78 pad 1: GND -> GND_MCU
- C78 pad 2: +3V3 -> Net-(U19-IN+)
- C79 pad 1: PGND -> GND_MCU
- C79 pad 2: VDC -> +5V_MCU
- C8 pad 1: Net-(D1-COM) -> Net-(C8-Pad1)
- C8 pad 2: Net-(D1-A1) -> Net-(C11-Pad1)
- C80 pad 1: GND1 -> GND_MCU
- C80 pad 2: +5V_ISO -> +5V_MCU
- C82 pad 1: GND -> GND_ADC
- C82 pad 2: +24V -> /MCU/MC_IV_SEN
- C83 pad 1: GND -> GND_MCU
- C83 pad 2: Net-(U14-VCC) -> /ENCODER/V_ENC
- C84 pad 1: Net-(U14-SW) -> GND_MCU
- C84 pad 2: Net-(U14-BOOST) -> /ENCODER/ENC_HOME
- C85 pad 1: Net-(U14-VFB) -> GND_MCU
- C85 pad 2: +15V -> /ENCODER/ENC_INDEX
- C86 pad 1: GND -> GND_MCU
- C86 pad 2: +3V3 -> /ENCODER/ENC_B
- C87 pad 1: AGND -> GND_MCU
- C87 pad 2: AVDD -> /ENCODER/ENC_A
- C9 pad 1: GND -> Net-(C8-Pad1)
- C9 pad 2: VREF -> CHASSIS
- D1 pad 1: Net-(D1-A1) -> GND_INV
- D1 pad 2: Net-(D1-A1) -> +24V_INV
- D10 pad 1: GND -> GND_INV
- D10 pad 2: /Inverter/MC_PWM_UH -> /INVERTER/IPM_PWM_WH
- D10 pad 3: /Inverter/MC_PWM_VH -> /INVERTER/IPM_PWM_WL
- D10 pad 4: +3V3 -> +5V_INV
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Other:
- board size 154 x 178.5 mm -> 159.9 x 155.6 mm

Commit message: V1 schematic update 18
Parts:
- removed B1: 220V/50W, SAMPI:LAMP_6.35MM
- removed BR1: 400V/10A, SAMPI:GBJ25xx
- removed C1, C25: 470uF/35V, SAMPI:CAP_ELEC-10.3x10.3-DIA10
- removed C10, C22, C24, C26, C32, C4, C5: 100nF, SAMPI:CAP0603
- removed C11, C13, C16, C9: 100pF/2kV, SAMPI:CAP1206
- removed C12: 470uF/25V, SAMPI:CAP_ELEC-10.3x10.3-DIA10
- removed C14, C20, C3, C30: 10uF, SAMPI:CAP0603
- removed C15, C8: 1uF/400V, SAMPI:ECWFE2W105
- removed C17, C21, C7: 100nF/400V, SAMPI:CAP_FILM_6.0x12.0x12.5-P10
- removed C18: 680uF/450V, SAMPI:ESMQ451VSN681MA50S
- removed C19, C2, C28, C29: 10uF/35V, SAMPI:CAP1206
- removed C23, C6: 3.3nF, SAMPI:CAP0603
- removed C27: 470uF/16V, SAMPI:CAP_ELEC-8.3x8.3-DIA8.0
- removed C34: 220uF/6.3V, SAMPI:CAP1411
- removed D1, D6: 24V, SAMPI:DO-214AA-12
- removed D2, D5: 75V/150mA, SAMPI:SOD-323
- removed D3, D4: 6V2, SAMPI:SOD80C-LL34
- removed D7: PWR, SAMPI:LED0603
- removed FT1, FT4: 15mH/500mA, SAMPI:EE8.3
- removed FT2: 5mH/2.5A, SAMPI:IND-SQ1010
- removed FT3: 120R@100MHz, SAMPI:FT0603
- removed G1: 300V, SAMPI:GDT1812_3532
- removed L1: 68uH/1A, SAMPI:IND-8D43-8045
- removed L2: 56uH/1A, SAMPI:IND-8D43-8045
- removed M1, M2, M3, M4: 470V/1.2kA, SAMPI:MOV5MM
- removed MD1: 24V±2%/3W, SAMPI:HLK-PMxx
- removed MD2: 24V±2%/10W, SAMPI:HLK-10M
- removed R1, R10, R11, R12: 10K, SAMPI:RES0603
- removed R13: 140K, 1%, SAMPI:RES0603
- removed R14, R3: 10K, 1%, SAMPI:RES0603
- removed R15: 1K, SAMPI:RES0603
- removed R2: 191K, 1%, SAMPI:RES0603
- removed R4, R5, R6, R7, R8, R9: 1M, SAMPI:RES1206
- removed RL1, RL2: 5V/30A, SAMPI:SLA-12VDC-SL-C
- removed U1: SMPS 16V±2%/0.6A, SAMPI:TDFN8_2x3_MCHP
- removed U2, U4: LDO 5V±1%, SAMPI:SOT-89
- removed U3: SMPS 12V±2%/0.8A, SAMPI:TDFN8_2x3_MCHP
- removed U5: LDO 3V3±2%, SAMPI:SOT-223-3
- added C88: 100uF/450V, SAMPI:CAP_ELEC-18.0x51.5-LS7.5, F.Cu at (45.5, 88.8)
- added J14: MCU PWR, SAMPI:HDM1x8x2.54_TH_RA, F.Cu at (76.6, 77.2)
- added J15: INV PWR & RELAYS, SAMPI:HDM1x8x2.54_TH_RA, F.Cu at (40.8, 50.8)
- added J16: HIGH VOLTAGE OUTPUTS, SAMPI:HDF1x10x2.54_TH_RA, F.Cu at (49.4, 77.2)
- added J2: U, SAMPI:QC-6.3, F.Cu at (107.5, 21.1)
- added Q8: 60V/265mA, SAMPI:SOT23, F.Cu at (137.9, 128.0)
- added Q9: 60V/265mA, SAMPI:SOT23, F.Cu at (142.5, 128.0)
- J3: value AC POWER INPUT -> V; footprint SAMPI:TMB3_9.5 -> SAMPI:QC-6.3
- J4: value FAN -> W; footprint SAMPI:HDM-2x2.54-TH -> SAMPI:QC-6.3
- J5: value MOTOR -> N; footprint SAMPI:TMB4_9.5 -> SAMPI:QC-6.3
- Q1, Q2: value 20V/1A -> 60V/265mA
- moved J4 106.1 mm to (107.5, 30.3)
- moved Q1 54.7 mm to (128.7, 128.0)
- moved Q2 54.7 mm to (133.3, 128.0)
- moved MD3 50.2 mm to (80.4, 90.8)
- moved J5 45.8 mm to (108.0, 15.8)
- moved J3 35.9 mm to (107.5, 25.7)
- moved U7 35.7 mm to (89.7, 48.1)
Connections:
- J3 pad 1: CHASSIS -> /INVERTER/MC_V
- J4 pad 1: +12V_MCU -> /INVERTER/MC_W
- MD3 pad L10: /INVERTER POWER/~{DEV_RELAY} -> /MCU POWER/~{DEV_RELAY}
- MD3 pad L9: /INVERTER POWER/PWR_RELAY -> /MCU POWER/PWR_RELAY
- Q1 pad 1: /INVERTER POWER/PWR_RELAY -> /ENCODER/V_ENC
- Q1 pad 2: GND_MCU -> /ENCODER/PULSE_A
- Q2 pad 1: /INVERTER POWER/~{DEV_RELAY} -> /ENCODER/V_ENC
- Q2 pad 2: GND_MCU -> /ENCODER/PULSE_B
- Q4 pad 3: /ENCODER/HOME -> Net-(Q4-D)
- Q5 pad 3: /ENCODER/INDEX -> Net-(Q5-D)
- Q6 pad 3: /ENCODER/PULSE_B -> Net-(Q2-D)
- Q7 pad 3: /ENCODER/PULSE_A -> Net-(Q1-D)
Other:
- board size 159.9 x 155.6 mm -> 98 x 98 mm

Commit message: V1 schematic update 20
Parts:
- added C1: 10uF/35V, SAMPI:CAP1206, F.Cu at (184.2, 109.0)
- added C2: 10uF/35V, SAMPI:CAP1206, F.Cu at (186.5, 109.0)
- added SH10: SCREW HOLDER, SAMPI:SCREWHOLE-2.5M, F.Cu at (130.3, 155.1)
- added SH8: SCREW HOLDER, SAMPI:SCREWHOLE-2.5M, F.Cu at (130.2, 142.6)
- added SH9: SCREW HOLDER, SAMPI:SCREWHOLE-2.5M, F.Cu at (130.3, 149.6)
- U7: moved to B.Cu
- moved SH3 196.2 mm to (275.9, 23.8)
- moved U7 160.8 mm to (250.3, 56.7)
- moved C88 154.6 mm to (193.6, 44.4), turned to -90 degrees
- moved SH2 149.3 mm to (275.9, 117.3)
- moved SH4 146.5 mm to (182.4, 23.8)
- moved J15 144.8 mm to (181.8, 83.8), turned to 90 degrees
- moved J16 137.7 mm to (181.8, 39.4), turned to 90 degrees
- moved MD3 133.7 mm to (214.1, 94.2)
- moved J14 108.6 mm to (181.8, 104.2), turned to 90 degrees
- moved J1 101.7 mm to (246.3, 112.2)
- moved C83 100.8 mm to (211.7, 111.8), turned to 90 degrees
- moved J11 89.2 mm to (197.8, 114.6)
- moved FT5 87.7 mm to (192.3, 101.6), turned to 90 degrees
- moved U6 83.8 mm to (189.6, 101.6)
- moved C37 83.5 mm to (190.4, 105.2), turned to -90 degrees
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Connections:
- J11 pad 1: /ENCODER/PULSE_A -> +24V_MCU
- J11 pad 2: /ENCODER/PULSE_B -> +12V_MCU
- J11 pad 3: /ENCODER/INDEX -> /ENCODER/V_ENC
- J11 pad 4: /ENCODER/HOME -> GND_MCU
- J11 pad 5: GND_MCU -> /ENCODER/HOME
- J11 pad 6: /ENCODER/V_ENC -> /ENCODER/INDEX
- J11 pad 7: +12V_MCU -> /ENCODER/PULSE_B
- J11 pad 8: +24V_MCU -> /ENCODER/PULSE_A
- J14 pad 2: +3V3_MCU -> +24V_MCU
- J14 pad 3: +5V_MCU -> +12V_MCU
- J14 pad 6: +12V_MCU -> +5V_MCU
- J14 pad 7: +24V_MCU -> +3V3_MCU
- J15 pad 1: GND_INV -> /MCU POWER/~{DEV_RELAY}
- J15 pad 2: +16V_INV -> /MCU POWER/PWR_RELAY
- J15 pad 7: /MCU POWER/~{DEV_RELAY} -> +16V_INV
- J15 pad 8: /MCU POWER/PWR_RELAY -> GND_INV
- J16 pad 1: CHASSIS -> PGND
- J16 pad 10: VDC -> CHASSIS
- J16 pad 2: CHASSIS -> PGND
- J16 pad 5: PGND -> VDC
- J16 pad 6: PGND -> VDC
- J16 pad 9: VDC -> CHASSIS
Routing:
- net GND_MCU: track 0.00 -> 15.7 mm
- net +12V_MCU: track 0.00 -> 14.2 mm
- net +5V_MCU: track 0.00 -> 11.4 mm
- net +24V_MCU: track 0.00 -> 9.61 mm
- net GND_ADC: track 0.00 -> 8.83 mm
- net +3V3_ADC: track 0.00 -> 5.18 mm
- net /ENCODER/V_ENC: track 0.00 -> 1.28 mm
Other:
- outline, holes or cut-outs redrawn
