File: V1/Design/HW.ACIM-INV/HW.ACIM-INV.kicad_pcb (KiCad board)
At the start: 4 copper layers, 98 x 98 mm, 164 parts, among them J1 MCDBG, J11 ENCODER, J14 MCU PWR, J15 INV PWR & RELAYS, J16 HIGH VOLTAGE OUTPUTS, J2 U, J3 V, J4 W, J5 N, M5 560V/1.75kA, M6 560V/1.75kA, M7 560V/1.75kA, Q1 60V/265mA, Q2 60V/265mA, Q3 20V/1A, Q4 60V/265mA, Q5 60V/265mA, Q6 60V/265mA, Q7 60V/265mA, Q8 60V/265mA, Q9 60V/265mA, U10 DIGI ISO, U11 I=±10A, U12 I=±10A, U13 CMP-1CH, U14 ISO OPAMP 1-CH, U15 ISO OPAMP 1-CH, U16 ISEN 50mV/V, U17 OP-1CH, U18 OP-1CH, U19 OP-1CH, U6 LDO 3.3V±0.1%/20mA, U7 IPM 600V/15A, U8 DIGI ISO, U9 DIGI ISO

Commit message: V1 schematic update 21
Parts:
- moved C75 284.9 mm to (294.0, 46.7)
- moved R36 284.9 mm to (305.2, 36.3)
- moved R42 284.9 mm to (305.2, 51.9)
- moved U14 284.9 mm to (293.9, 59.8)
- moved C64 284.9 mm to (290.3, 36.3)
- moved C66 284.9 mm to (290.3, 41.5)
- moved C68 284.9 mm to (290.3, 46.7)
- moved C70 284.9 mm to (290.3, 51.9)
- moved C72 284.9 mm to (294.0, 38.9)
- moved C76 284.9 mm to (294.0, 49.3)
- moved D15 284.9 mm to (295.4, 68.6)
- moved R31 284.9 mm to (301.5, 41.5)
- moved R35 284.9 mm to (301.5, 51.9)
- moved U16 284.9 mm to (304.2, 68.4)
- moved R32 284.9 mm to (301.5, 44.1)
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Connections:
- D17 pad A: /MCU/IND_ERR -> Net-(D17-PadA)
- D17 pad K: Net-(D17-PadK) -> GND_MCU
- D18 pad A: /MCU/IND_RUN -> Net-(D18-PadA)
- D18 pad K: Net-(D18-PadK) -> GND_MCU
- R49 pad 1: Net-(D17-PadK) -> /MCU/IND_ERR
- R49 pad 2: GND_MCU -> Net-(D17-PadA)
- R50 pad 1: Net-(D18-PadK) -> /MCU/IND_RUN
- R50 pad 2: GND_MCU -> Net-(D18-PadA)
Routing:
- net VDC: track 0.00 -> 85.6 mm
- net /INVERTER/MC_U: track 0.00 -> 59.2 mm, vias 0 -> 4
- net CHASSIS: track 0.00 -> 56.1 mm
- net /ENCODER/V_ENC: track 1.28 -> 53.1 mm
- net /ENCODER/HOME: track 0.00 -> 40.7 mm
- net Net-(G2-Pad1): track 0.00 -> 39.0 mm
- net PGND: track 0.00 -> 37.9 mm
- net /INVERTER/MC_W: track 0.00 -> 35.7 mm
- net +3V3_MCU: track 0.00 -> 33.4 mm, vias 0 -> 4
- net /ENCODER/INDEX: track 0.00 -> 31.2 mm
- net /INVERTER/MC_V: track 0.00 -> 22.4 mm
- net /ENCODER/PULSE_B: track 0.00 -> 21.8 mm
- net GND_MCU: track 15.7 -> 32.3 mm, vias 0 -> 2
- net Net-(U11-IPP1): track 0.00 -> 14.2 mm
- net /ENCODER/PULSE_A: track 0.00 -> 12.3 mm
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Other:
- outline, holes or cut-outs redrawn
