File: V1/Design/HW.ACIM-INV/HW.ACIM-INV.kicad_pcb (KiCad board)
At the start: 4 copper layers, 98 x 98 mm, 163 parts, among them J1 MCDBG, J11 ENCODER, J14 MCU PWR, J15 INV PWR & RELAYS, J16 HIGH VOLTAGE OUTPUTS, J2 U, J3 V, J4 W, J5 N, M5 560V/1.75kA, M6 560V/1.75kA, M7 560V/1.75kA, Q1 60V/265mA, Q2 60V/265mA, Q3 20V/1A, Q4 60V/265mA, Q5 60V/265mA, Q6 60V/265mA, Q7 60V/265mA, Q8 60V/265mA, Q9 60V/265mA, U1 I=±10A, U10 DIGI ISO, U11 I=±10A, U12 I=±10A, U13 CMP-1CH, U15 ISO OPAMP 1-CH, U17 OP-1CH, U18 OP-1CH, U19 OP-1CH, U2 OP-1CH, U6 LDO 3.3V±0.1%/20mA, U7 IPM 600V/15A, U8 DIGI ISO, U9 DIGI ISO

Commit message: V1 schematic update 25
Parts:
- added FT2: 120R@100MHz, SAMPI:FB10MM-TH, F.Cu at (191.8, 82.6)
- added FT3: 120R@100MHz, SAMPI:FB10MM-TH, F.Cu at (191.8, 77.5)
- added FT4: 120R@100MHz, SAMPI:FB10MM-TH, F.Cu at (226.8, 82.6)
- added FT6: 120R@100MHz, SAMPI:FB10MM-TH, F.Cu at (226.8, 77.5)
- moved D11 128.0 mm to (274.6, 104.8), turned to 180 degrees
- moved R18 127.6 mm to (270.9, 112.6), turned to 180 degrees
- moved D13 126.5 mm to (276.1, 101.0), turned to 180 degrees
- moved R19 125.2 mm to (270.9, 110.0), turned to 180 degrees
- moved D12 123.3 mm to (271.4, 102.4), turned to 180 degrees
- moved R20 123.0 mm to (270.9, 107.4), turned to 180 degrees
- moved C55 111.7 mm to (257.8, 95.3)
- moved R22 111.2 mm to (263.8, 95.3)
- moved C54 106.1 mm to (251.0, 95.3)
- moved C53 100.6 mm to (244.2, 95.3)
- moved C77 88.1 mm to (236.4, 94.1), turned to 180 degrees
- moved C78 85.6 mm to (236.4, 88.5), turned to 180 degrees
- moved C79 83.4 mm to (233.5, 94.1), turned to 180 degrees
- moved C80 82.1 mm to (233.5, 89.7), turned to 180 degrees
- moved C81 79.4 mm to (230.7, 92.9), turned to 180 degrees
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Connections:
- J15 pad 5: +5V_INV -> Net-(FT2-Pad1)
- J15 pad 7: +16V_INV -> Net-(FT3-Pad1)
- R1 pad 1: /POWER MEASUREMENT/MC_IDC_HAL -> /INVERTER/MC_IDC_HAL
Routing:
- net +3V3_MCU: track 110.1 -> 171.0 mm
- net /MCU/IND_ERR: track 0.00 -> 52.4 mm, vias 0 -> 2
- net +16V_INV: track 103.4 -> 53.4 mm
- net /MCU/IND_RUN: track 2.00 -> 49.1 mm, vias 1 -> 0
- net GND_MCU: track 216.1 -> 243.1 mm
- net /ENCODER/ENC_HOME: track 44.7 -> 70.3 mm
- net /ENCODER/ENC_INDEX: track 37.7 -> 63.0 mm
- net Net-(FT3-Pad2): track 0.00 -> 25.0 mm
- net Net-(FT2-Pad2): track 0.00 -> 25.0 mm
- net /ENCODER/ENC_A: track 23.4 -> 35.6 mm
- net /ENCODER/ENC_B: track 30.3 -> 41.4 mm
- net GND_ADC: track 33.2 -> 42.1 mm
- net /INVERTER/MC_PWM_VL: track 41.5 -> 35.7 mm
- net /MCU/MC_IV_SEN: track 0.00 -> 5.37 mm
- net +5V_MCU: track 23.7 -> 29.0 mm
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
Commit message: V1 schematic update 26
Routing:
- added copper zone on F.Cu, net Net-(U1-IPP1)
- added copper zone on In1.Cu, net Net-(U1-IPP1)
- added copper zone on F.Cu, net PGND
- added copper zone on In1.Cu, net PGND
- added copper zone on F.Cu, net VDC
- added copper zone on In1.Cu, net VDC
Other:
- outline, holes or cut-outs redrawn

Commit message: V1 schematic update 27
Parts:
- added D7: PV, SAMPI:LED0603, F.Cu at (275.4, 101.9)
- added D8: PU, SAMPI:LED0603, F.Cu at (275.4, 104.2)
- added D9: PW, SAMPI:LED0603, F.Cu at (275.4, 99.7)
- added R4: 1K, SAMPI:RES0603, F.Cu at (272.4, 104.2)
- added R5: 1K, SAMPI:RES0603, F.Cu at (272.4, 101.9)
- added R6: 1K, SAMPI:RES0603, F.Cu at (272.4, 99.7)
- moved D13 9.99 mm to (275.4, 110.9)
- moved D12 5.71 mm to (275.4, 106.4)
- moved R18 4.51 mm to (275.4, 112.8), turned to 0 degrees
- moved D11 3.97 mm to (275.4, 108.7)
- moved FT2 2.54 mm to (191.8, 80.0)
- moved FT3 2.54 mm to (191.8, 75.0)
- moved FT4 2.54 mm to (226.8, 80.0)
- moved FT6 2.54 mm to (226.8, 75.0)
- moved R19 2.01 mm to (272.4, 108.7)
- moved R20 1.80 mm to (272.4, 106.4)
Routing:
- net /INVERTER/MC_PWM_UH: track 27.3 -> 66.4 mm, vias 0 -> 2
- net /INVERTER/MC_PWM_VH: track 29.4 -> 62.5 mm, vias 0 -> 2
- net /INVERTER/MC_PWM_WH: track 35.9 -> 62.6 mm, vias 0 -> 2
- net GND_MCU: track 243.1 -> 269.5 mm
- net /INVERTER/MC_PWM_UL: track 30.4 -> 54.9 mm, vias 0 -> 2
- net /INVERTER/MC_PWM_VL: track 35.7 -> 53.7 mm, vias 0 -> 2
- net /INVERTER/MC_PWM_WL: track 41.4 -> 57.2 mm, vias 0 -> 2
- net +3V3_MCU: track 171.0 -> 177.5 mm, vias 4 -> 5
- net Net-(D13-PadA): track 0.00 -> 1.91 mm
- net Net-(D9-PadA): track 0.00 -> 1.53 mm
- net Net-(D8-PadA): track 0.00 -> 1.53 mm
- net Net-(D7-PadA): track 0.00 -> 1.53 mm
- net Net-(D12-PadA): track 0.00 -> 1.53 mm
- net Net-(D11-PadA): track 0.00 -> 1.53 mm
- net Net-(FT3-Pad1): track 5.00 -> 6.05 mm
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- added copper zone on B.Cu, net CHASSIS
- added copper zone on F.Cu, net CHASSIS
- added copper zone on In1.Cu, net CHASSIS
- added copper zone on In2.Cu, net CHASSIS
Other:
- outline, holes or cut-outs redrawn
