File: V1/Design/HW.ACIM-INV/HW.ACIM-INV.kicad_pcb (KiCad board)
At the start: 4 copper layers, 98 x 98 mm, 169 parts, among them J1 MCDBG, J11 ENCODER, J14 MCU PWR, J15 INV PWR & RELAYS, J16 HIGH VOLTAGE OUTPUTS, J2 U, J3 V, J4 W, J5 N, M5 560V/1.75kA, M6 560V/1.75kA, M7 560V/1.75kA, Q1 60V/265mA, Q2 60V/265mA, Q3 20V/1A, Q4 60V/265mA, Q5 60V/265mA, Q6 60V/265mA, Q7 60V/265mA, Q8 60V/265mA, Q9 60V/265mA, U1 I=±10A, U10 DIGI ISO, U11 I=±10A, U12 I=±10A, U13 CMP-1CH, U15 ISO OPAMP 1-CH, U17 OP-1CH, U18 OP-1CH, U19 OP-1CH, U2 OP-1CH, U6 LDO 3.3V±0.1%/20mA, U7 IPM 600V/15A, U8 DIGI ISO, U9 DIGI ISO

Commit message: V1 layout
Routing:
- net GND_MCU: track 308.9 -> 3.33 mm, vias 14 -> 191
- net GND_INV: track 209.4 -> 2.35 mm, vias 2 -> 65
- net GND_ADC: track 89.4 -> 58.3 mm
- added copper zone on B.Cu, net /INVERTER/MC_W
- added copper zone on In2.Cu, net /INVERTER/MC_W
- added copper zone on F.Cu, net Net-(C58-Pad2)
- added copper zone on F.Cu, net Net-(C59-Pad1)
- added copper zone on F.Cu, net Net-(C60-Pad2)
- added copper zone on B.Cu, net Net-(U11-IPP1)
- added copper zone on In2.Cu, net Net-(U11-IPP1)
- added copper zone on B.Cu, net Net-(U12-IPP1)
- added copper zone on In2.Cu, net Net-(U12-IPP1)
Other:
- outline, holes or cut-outs redrawn
- board text added: "+3V3"
- board text added: "DBRX"
- board text added: "DBTX"
- board text added: "DVRX"
- board text added: "DVTX"
- board text added: "GND"
- board text added: "HW.ACIM-INV_REV1.0"
- board text added: "PGC"
- board text added: "PGD"
- board text added: "USB+"
- board text added: "USB-"
- board text added: "VBUS"
- board text added: "~{MCLR}"

Commit message: HW.ACIM-INV-V1.0
Parts:
- added G***: LOGO, LOGO, F.Cu at (231.8, 108.4)
- added G***: LOGO, LOGO, F.Cu at (272.0, 58.6)
- added G***: LOGO, LOGO, F.Cu at (246.2, 58.6)
- added G***: LOGO, LOGO, F.Cu at (186.1, 70.5)
- added G***: LOGO, LOGO, F.Cu at (221.2, 23.7)
- added G***: LOGO, LOGO, F.Cu at (272.2, 23.7)
- added G***: LOGO, LOGO, F.Cu at (186.3, 23.8)
- added G***: LOGO, LOGO, F.Cu at (186.1, 117.2)
- added G***: LOGO, LOGO, F.Cu at (274.3, 114.6)
Other:
- board text added: "CHASSIS"
- board text added: "HW.ACIM-INV V1.0"
- board text added: "PGND"
- board text added: "U"
- board text added: "V"
- board text added: "VDC"
- board text added: "W"
- board text removed: "HW.ACIM-INV_REV1.0"
