File: V1/Design/HW.ACIM-INV/MCUPOWER.kicad_sch (KiCad schematic)
At the start: 42 parts, among them J2 FAN, U10 SMPS 5V±2%/1.2A, U12 SMPS 12V±2%/0.8A, U13 LDO 5V±0.4%/250mA, U2 LDO 3.3V±0.5%/1A

Commit message: V1 schematic update 14
Parts:
- removed C65, C66: 22pF, SAMPI:CAP0603, symbol SAMPI:CERCAP
- removed C68: 470uF/35V, SAMPI:CAP_ELEC-10.3x10.3-DIA10, symbol SAMPI:ELECCAP
- removed C70: 10uF, SAMPI:CAP0603, symbol SAMPI:CERCAP
- removed FT4: 120R@100MHz, SAMPI:FT0603, symbol SAMPI:FerriteBead
- removed L2: 22uH/1.5A, SAMPI:IND-8D43-8045, symbol SAMPI:IND
- removed R11: 53.6K, 1%, SAMPI:RES0603, symbol SAMPI:RES
- removed R13: 10K, 1%, SAMPI:RES0603, symbol SAMPI:RES
- removed R7: 100K, SAMPI:RES0603, symbol SAMPI:RES
- removed U10: SMPS 5V±2%/1.2A, SAMPI:TDFN8_2x3_MCHP, symbol SAMPI:MCP16311-TDFN
- removed U13: LDO 5V±0.4%/250mA, SAMPI:SOT-89, symbol SAMPI:MCP1702
- removed U2: LDO 3.3V±0.5%/1A, SAMPI:DFN8_3x3_MCHP, symbol SAMPI:MCP1727
- added U10: LDO 5V±1%, SAMPI:SOT-89, symbol SAMPI:LDO_BDxxFA1FP3
- added U13: LDO 3.3V±0.1%/20mA, SAMPI:SOT-23-6_MCHP, symbol SAMPI:MCP1501
- added U2: LDO 3V3±2%, SAMPI:SOT-223-3, symbol SAMPI:LDO_MCP1755
- C26: Checked (none) -> OK; Unit Price (none) -> 0.079
- C29: value 10uF -> 22pF; Checked (none) -> OK; MFT Samsung -> Walsin; MNP CL10A106MQ8NNNC -> 0603N220J500CT; Unit Price (none) -> 0.012
- C41, C43: Checked (none) -> OK; Unit Price (none) -> 0.0146
- C50: value 3.3nF -> 10uF; Checked (none) -> OK; MNP CL10B332KB8NNNC -> CL10A106MQ8NNNC; Unit Price (none) -> 0.079
- C63: value 100nF -> 10uF/35V; MNP CL10B104KB8NNNC -> CL10A106MQ8NNNC
Connections:
- net VREF is gone; now on net +5V_ADC: C71.2
- net GND: no longer C21.1, C22.1, C26.1, C27.-, C29.1, C30.1, C40.1, C41.1, C55.1, C58.-, C63.1, C64.1, C69.-, C71.1, D5.1 (A1), FT5.2, MD1.4 (DC-), R15.1, U12.5 (PGND), U12.8 (AGND), U12.9 (EP)
- net GND_ADC: now reaches C50.1
- net GND_ADC: now also C26.1, C29.1, C41.1, C43.1, C71.1, FT5.2, U13.2 (GND3), U13.3 (GND1), U13.5 (GND2)
- net +5V_ADC: now reaches C29.2
- net +5V_ADC: now also C26.2, C41.2, U10.1 (VO), U13.4 (~{SHDN}), U13.6 (VDD)
- net +3V3_ADC: now reaches C43.2
- net +3V3_ADC: now also C50.2, U13.1 (OUT)
- net +12V renamed +12V_MCU
- net +12V_MCU: now also C21.2, C63.2, U10.3 (VCC), U2.1 (VIN)
- net +24V renamed +24V_MCU
- net +24V_MCU: no longer C21.2
- net +3V3 renamed +3V3_MCU
- net +3V3_MCU: now also U2.3 (VO)
- removed net +5V: C26.2, C50.2, C63.2
- net AGND renamed GND_MCU
- net GND_MCU: now also C21.1, C22.1, C27.-, C30.1, C40.1, C55.1, C58.-, C63.1, C64.1, C69.-, D5.1 (A1), MD1.4 (DC-), R15.1, U12.5 (PGND), U12.8 (AGND), U12.9 (EP), U10.2 (GND), U2.2 (GND), U2.4 (EP)
- no-connect marks 1 -> 0
Other:
- moved on the sheet: C22, C30, C44, C54, C55, C58, C64, C69, C71, FAN1, FT5, J2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

Commit message: V1 schematic update 15
Connections:
- net GND_ADC: no longer C26.1, C29.1, C41.1, C71.1, U13.3 (GND1)
- net GND_MCU: now also C26.1, C29.1, C41.1, C71.1, U13.3 (GND1)
- net +5V_ADC renamed +5V_MCU
Other:
- company: TON DUC THANG UNIVERSITY -> (none)
- moved on the sheet: C26, C29, C41, C43, C50, C55, C58, C71, FT5, U13

Commit message: V1 schematic update 16
Parts:
- added D4: PWR, SAMPI:LED0603, symbol SAMPI:WLED
- added R1: 1K, SAMPI:RES0603, symbol SAMPI:RES
- C21, C22, C63: footprint SAMPI:CAP0603 -> SAMPI:CAP1206; MFT Samsung -> (none); MNP CL10A106MQ8NNNC -> (none)
- C26, C50: Checked OK -> (none); Unit Price 0.079 -> (none)
- C29: Checked OK -> (none); Unit Price 0.012 -> (none)
- C41, C43: Checked OK -> (none); Unit Price 0.0146 -> (none)
- R8: value 100K -> 10K; MFT YAGEO -> (none); MNP RC0603FR-07100KL -> (none)
- U13: Checked OK -> (none); Unit Price 1 -> (none)
Connections:
- net +3V3_MCU: now also R1.1
- net GND_MCU: now also D4.K
- new net: D4.A, R1.2
Other:
- moved on the sheet: C55, C58, C63, U2

Commit message: V1 schematic update 17
Parts:
- C19: renamed from C22; MFT (none) -> Murata; MNP (none) -> GRT31CR6YA106ME01L
- C23: renamed from C54; now not fitted; now left out of the parts list
- C25: renamed from C27; MFT KEMET -> KYAVX; MNP A768MS477M1ELAE017 -> APD1012471M035R
- C27: renamed from C69; value 470uF/35V -> 470uF/16V; footprint SAMPI:CAP_ELEC-10.3x10.3-DIA10 -> SAMPI:CAP_ELEC-8.3x8.3-DIA8.0; MNP A768MS477M1ELAE017 -> A768KS477M1CLAE017
- C28: renamed from C63; MFT (none) -> Murata; MNP (none) -> GRT31CR6YA106ME01L
- C29: renamed from C21; MFT (none) -> Murata; MNP (none) -> GRT31CR6YA106ME01L
- L2: renamed from L3; MFT Bourns Inc. -> Bourns
- MD2: renamed from MD1; footprint SAMPI:LD10-23BxxR2-RC -> SAMPI:HLK-10M
- R12: renamed from R8; MFT (none) -> YAGEO; MNP (none) -> RC0603JR-0710KL
- R13: renamed from R14; MNP RC0603FR-07100KL -> RC0603FR-07140KL
- R15: renamed from R1; MFT (none) -> YAGEO; MNP (none) -> RC0603JR-071KL
- U3: renamed from U12; MFT Microchip Technology -> Microchip
- renumbered C30 to C20, C57 to C21, C44 to C22, C40 to C24, C64 to C26, C71 to C30, C26 to C31, C55 to C32, C29 to C33, C58 to C34, C41 to C35, C43 to C36, C50 to C37, D5 to D6, D4 to D7, FT2 to FT4, J2 to J4, R15 to R14, U10 to U4, U2 to U5, U13 to U6
Connections:
- net +24V_MCU: now also MD2.4 (DC+); no longer MD2.5 (DC+)
- net GND_MCU: now also MD2.3 (DC-); no longer MD2.4 (DC-)

Commit message: V1 schematic update 18
Parts:
- removed C19, C28, C29: 10uF/35V, SAMPI:CAP1206, symbol SAMPI:CERCAP
- removed C20, C30: 10uF, SAMPI:CAP0603, symbol SAMPI:CERCAP
- removed C21: 100nF/400V, SAMPI:CAP_FILM_6.0x12.0x12.5-P10, symbol SAMPI:CERCAP
- removed C22, C24, C26, C32: 100nF, SAMPI:CAP0603, symbol SAMPI:CERCAP
- removed C23: 3.3nF, SAMPI:CAP0603, symbol SAMPI:CERCAP
- removed C25: 470uF/35V, SAMPI:CAP_ELEC-10.3x10.3-DIA10, symbol SAMPI:ELECCAP
- removed C27: 470uF/16V, SAMPI:CAP_ELEC-8.3x8.3-DIA8.0, symbol SAMPI:ELECCAP
- removed C34: 220uF/6.3V, SAMPI:CAP1411, symbol SAMPI:ELECCAP
- removed D6: 24V, SAMPI:DO-214AA-12, symbol SAMPI:DIODE-TVS
- removed D7: PWR, SAMPI:LED0603, symbol SAMPI:WLED
- removed FAN1: AC/DC FAN, symbol SAMPI:FAN
- removed FT4: 15mH/500mA, SAMPI:EE8.3, symbol SAMPI:CK_Choke_2
- removed J4: FAN, SAMPI:HDM-2x2.54-TH, symbol SAMPI:SIL02-2
- removed L2: 56uH/1A, SAMPI:IND-8D43-8045, symbol SAMPI:IND
- removed MD2: 24V±2%/10W, SAMPI:HLK-10M, symbol SAMPI:AC-DC
- removed R12: 10K, SAMPI:RES0603, symbol SAMPI:RES
- removed R13: 140K, 1%, SAMPI:RES0603, symbol SAMPI:RES
- removed R14: 10K, 1%, SAMPI:RES0603, symbol SAMPI:RES
- removed R15: 1K, SAMPI:RES0603, symbol SAMPI:RES
- removed U3: SMPS 12V±2%/0.8A, SAMPI:TDFN8_2x3_MCHP, symbol SAMPI:MCP16311-TDFN
- removed U4: LDO 5V±1%, SAMPI:SOT-89, symbol SAMPI:LDO_BDxxFA1FP3
- removed U5: LDO 3V3±2%, SAMPI:SOT-223-3, symbol SAMPI:LDO_MCP1755
- added J14: MCU PWR, SAMPI:HDM1x8x2.54_TH_RA, symbol SAMPI:SIL08
- added J15: INV PWR & RELAYS, SAMPI:HDM1x8x2.54_TH_RA, symbol SAMPI:SIL08
Connections:
- net +12V_MCU: now also J14.6
- net +24V_MCU: now also J14.7
- net +3V3_MCU: now also J14.2
- net +5V_MCU: now also J14.3
- net GND_MCU: now also J14.1, J14.4, J14.5, J14.8
- new net +16V_INV: J15.2
- new net +5V_INV: J15.4
- new net GND_INV: J15.1, J15.3
- new net PWR_RELAY: J15.8
- new net ~{DEV_RELAY}: J15.7
Other:
- note removed: "HIGH VOLTAGE ZONE"
- note removed: "LOW VOLTAGE ZONE"

Commit message: V1 schematic update 20
Connections:
- net +12V_MCU: now also J14.3; no longer J14.6
- net +16V_INV: now also J15.7; no longer J15.2
- net +24V_MCU: now also J14.2; no longer J14.7
- net +3V3_MCU: now also J14.7; no longer J14.2
- net +5V_INV: now also J15.5; no longer J15.4
- net +5V_MCU: now also J14.6; no longer J14.3
- net GND_INV: now also J15.6, J15.8; no longer J15.1, J15.3
- net PWR_RELAY: now also J15.2; no longer J15.8
- net ~{DEV_RELAY}: now also J15.1; no longer J15.7
Other:
- moved on the sheet: C31, C33, C35, C36, C37, FT5, J14, U6

Commit message: V1 schematic update 22
Changed lines of the file:
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@@
 			(effects
 				(font
-					(size 1.5 1.5)
+					(face "Consolas")
+					(size 1.27 1.27)
 					(bold yes)
 				)
@@
 			(effects
 				(font
-					(size 1.27 1.27)
+					(face "Consolas")
+					(size 1.016 1.016)
+					(thickness 0.254)
 				)
 				(justify left)
@@
 			(effects
 				(font
-					(size 1.27 1.27)
+					(face "Consolas")
+					(size 1.016 1.016)
+					(thickness 0.254)
 				)
 				(hide yes)
@@
 			(effects
 				(font
-					(size 1.27 1.27)
+					(face "Consolas")
+					(size 1.016 1.016)
+					(thickness 0.254)
 				)
 				(hide yes)
@@
 			(effects
 				(font
-					(size 1.27 1.27)
+					(face "Consolas")
+					(size 1.016 1.016)
+					(thickness 0.254)
 				)
 				(hide yes)
@@
 			(effects
 				(font
-					(size 1.27 1.27)
+					(face "Consolas")
+					(size 1.016 1.016)
+					(thickness 0.254)
 				)
 				(hide yes)
@@
 			(effects
 				(font
-					(size 1.27 1.27)
+					(face "Consolas")
+					(size 1.016 1.016)
+					(thickness 0.254)
 				)
 				(hide yes)
@@
 			(effects
 				(font
-					(size 1.27 1.27)
+					(face "Consolas")
+					(size 1.016 1.016)
+					(thickness 0.254)
 				)
 				(hide yes)
@@
 			(effects
 				(font
-					(size 1.27 1.27)
+					(face "Consolas")
+					(size 1.016 1.016)
+					(thickness 0.254)
 				)
 				(hide yes)
@@
 			(effects
 				(font
-					(size 1.5 1.5)
+					(face "Consolas")
+					(size 1.27 1.27)
 					(bold yes)
 				)
@@
 			(effects
 				(font
-					(size 1.27 1.27)
+					(face "Consolas")
+					(size 1.016 1.016)
+					(thickness 0.254)
 				)
 				(justify left)
@@
 			(effects
 				(font
-					(size 1.27 1.27)
+					(face "Consolas")
+					(size 1.016 1.016)
+					(thickness 0.254)
 				)
 				(hide yes)
@@
 			(effects
 				(font
-					(size 1.27 1.27)
+					(face "Consolas")
+					(size 1.016 1.016)
+					(thickness 0.254)
 				)
 				(hide yes)
@@
 			(effects
 				(font
-					(size 1.27 1.27)
+					(face "Consolas")
+					(size 1.016 1.016)
+					(thickness 0.254)
 				)
 				(hide yes)
@@
 			(effects
 				(font
-					(size 1.27 1.27)
+					(face "Consolas")
+					(size 1.016 1.016)
+					(thickness 0.254)
 				)
 				(hide yes)
@@
 			(effects
 				(font
-					(size 1.27 1.27)
+					(face "Consolas")
+					(size 1.016 1.016)
+					(thickness 0.254)
 				)
 				(hide yes)
@@
 			(effects
 				(font
-					(size 1.27 1.27)
+					(face "Consolas")
+					(size 1.016 1.016)
+					(thickness 0.254)
 				)
 				(hide yes)
@@
 			(effects
 				(font
-					(size 1.27 1.27)
-				)
-				(hide yes)
+					(face "Consolas")
+					(size 1.016 1.016)
+					(thickness 0.254)
+				)
+				(hide yes)

Commit message: V1 schematic update 25
Parts:
- added FT2, FT3, FT4, FT6: 120R@100MHz, SAMPI:FB10MM-TH, symbol SAMPI:FerriteBead
Connections:
- net +16V_INV: now also FT6.2; no longer J15.7
- net +5V_INV: now also FT4.2; no longer J15.5
- new net: FT2.2, FT4.1
- new net: FT2.1, J15.5
- new net: FT3.1, J15.7
- new net: FT3.2, FT6.1
