File: V1/Design/HW.ACIM-INV/MCUPOWER.kicad_sch (KiCad schematic)
At the start: 13 parts, among them J14 MCU PWR, J15 INV PWR & RELAYS, U6 LDO 3.3V±0.1%/20mA

Commit message: V1 schematic update 28
Parts:
- removed FT2, FT3, FT4, FT6: 120R@100MHz, SAMPI:FB10MM-TH, symbol SAMPI:FerriteBead
Connections:
- net +16V_INV: now also J15.7
- net +5V_INV: now also J15.5

Commit message: V1 schematic update 29
Connections:
- net GND_ADC: now also U6.3 (GND1); no longer U6.5 (GND2)
- net GND_MCU: now also U6.5 (GND2); no longer U6.3 (GND1)

Commit message: Label & Case
Parts:
- C31, C33, C35, C36, C37, FT5, U6: now not fitted

Commit message: Update schematic
Parts:
- C31, C33, C35, C36, C37, FT5, U6: now fitted
Changed lines of the file:
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@@
 		(in_bom yes)
 		(on_board yes)
-		(dnp yes)
+		(dnp no)
 		(property "Reference" "#PWR0200"
 			(at 210.82 29.21 0)
@@
 		(in_bom yes)
 		(on_board yes)
-		(dnp yes)
+		(dnp no)
 		(property "Reference" "#PWR063"
 			(at 149.86 34.29 0)
@@
 		(in_bom yes)
 		(on_board yes)
-		(dnp yes)
+		(dnp no)
 		(property "Reference" "#PWR03"
 			(at 129.54 21.59 0)
@@
 		(in_bom yes)
 		(on_board yes)
-		(dnp yes)
+		(dnp no)
 		(property "Reference" "U6"
 			(at 168.91 13.335 0)
@@
 		(in_bom yes)
 		(on_board yes)
-		(dnp yes)
+		(dnp no)
 		(property "Reference" "#PWR0205"
 			(at 231.14 34.29 0)
@@
 		(in_bom yes)
 		(on_board yes)
-		(dnp yes)
+		(dnp no)
 		(property "Reference" "C33"
 			(at 146.05 22.86 90)
@@
 		(in_bom yes)
 		(on_board yes)
-		(dnp yes)
+		(dnp no)
 		(property "Reference" "#PWR0206"
 			(at 241.3 36.83 0)
@@
 		(in_bom yes)
 		(on_board yes)
-		(dnp yes)
+		(dnp no)
 		(property "Reference" "C35"
 			(at 152.4 22.8599 90)
@@
 		(in_bom yes)
 		(on_board yes)
-		(dnp yes)
+		(dnp no)
 		(fields_autoplaced yes)
 		(property "Reference" "C37"
@@
 		(in_bom yes)
 		(on_board yes)
-		(dnp yes)
+		(dnp no)
 		(property "Reference" "#PWR0198"
 			(at 220.98 34.29 0)
@@
 		(in_bom yes)
 		(on_board yes)
-		(dnp yes)
+		(dnp no)
 		(property "Reference" "#PWR0201"
 			(at 210.82 26.67 0)
@@
 		(in_bom yes)
 		(on_board yes)
-		(dnp yes)
+		(dnp no)
 		(fields_autoplaced yes)
 		(property "Reference" "C31"
@@
 		(in_bom yes)
 		(on_board yes)
-		(dnp yes)
+		(dnp no)
 		(property "Reference" "#PWR060"
 			(at 139.7 34.29 0)
@@
 		(in_bom yes)
 		(on_board yes)
-		(dnp yes)
+		(dnp no)
 		(property "Reference" "C36"
 			(at 189.23 22.8599 90)
@@
 		(in_bom yes)
 		(on_board yes)
-		(dnp yes)
+		(dnp no)
 		(property "Reference" "#PWR065"
 			(at 160.02 36.83 0)
@@
 		(in_bom yes)
 		(on_board yes)
-		(dnp yes)
+		(dnp no)
 		(property "Reference" "#PWR0195"
 			(at 220.98 21.59 0)
@@
 		(in_bom yes)
 		(on_board yes)
-		(dnp yes)
+		(dnp no)
 		(property "Reference" "#PWR0196"
 			(at 220.98 24.13 0)
@@
 		(in_bom yes)
 		(on_board yes)
-		(dnp yes)
+		(dnp no)
 		(property "Reference" "#PWR066"
 			(at 177.8 36.83 0)
@@
 		(in_bom yes)
 		(on_board yes)
-		(dnp yes)
+		(dnp no)
 		(property "Reference" "#PWR068"
 			(at 196.85 21.59 0)
@@
 		(in_bom yes)
 		(on_board yes)
-		(dnp yes)
+		(dnp no)
 		(property "Reference" "#PWR0204"
 			(at 241.3 31.75 0)
@@
 		(in_bom yes)
 		(on_board yes)
-		(dnp yes)
+		(dnp no)
 		(property "Reference" "FT5"
 			(at 169.545 26.67 0)
@@
 		(in_bom yes)
 		(on_board yes)
-		(dnp yes)
+		(dnp no)
 		(property "Reference" "#PWR069"
 			(at 196.85 34.29 0)
@@
 		(in_bom yes)
 		(on_board yes)
-		(dnp yes)
+		(dnp no)
 		(property "Reference" "#PWR0202"
 			(at 210.82 19.05 0)
@@
 		(in_bom yes)
 		(on_board yes)
-		(dnp yes)
+		(dnp no)
 		(property "Reference" "#PWR067"
 			(at 186.69 34.29 0)
@@
 		(in_bom yes)
 		(on_board yes)
-		(dnp yes)
+		(dnp no)
 		(property "Reference" "#PWR0203"
 			(at 231.14 29.21 0)
@@
 		(in_bom yes)
 		(on_board yes)
-		(dnp yes)
+		(dnp no)
 		(property "Reference" "#PWR058"
 			(at 129.54 34.29 0)
@@
 		(in_bom yes)
 		(on_board yes)
-		(dnp yes)
+		(dnp no)
 		(property "Reference" "#PWR0199"
 			(at 210.82 36.83 0)
@@
 		(in_bom yes)
 		(on_board yes)
-		(dnp yes)
+		(dnp no)
 		(property "Reference" "#PWR0197"
 			(at 220.98 31.75 0)
