File: V1/Design/HW.ACIM-INV/POWERMEASUREMENT.kicad_sch (KiCad schematic)
At the start: 34 parts, among them U18 OP-1CH, U19 OP-1CH, U6 ISEN 50mV/V, U7 ISO OPAMP 1-CH, U8 OP-1CH

Commit message: V1 schematic update 14
Parts:
- added C65, C75: 1nF, SAMPI:CAP0603, symbol SAMPI:CERCAP
- added C66, C68, C73, C74: 100nF, SAMPI:CAP0603, symbol SAMPI:CERCAP
- added D18: GP DIODE, SAMPI:SOT23, symbol SAMPI:DIODE_ARR1
- added R11, R13, R19, R21: 10R, SAMPI:RES0603, symbol SAMPI:RES
- added R7: 100R, SAMPI:RES0603, symbol SAMPI:RES
- added U17: ISO OPAMP 1-CH, symbol SAMPI:ISO-OPAMP
- R77: value 1.1K -> 1K
Connections:
- net GND is gone; now on net GND_ADC: U7.5 (GND2)
- net at C37.1, D9.3 (COM), R51.1: now also U7.3 (VIN-); no longer U6.5 (IN-)
- net at D17.3 (COM), R73.2, R77.1: now also R11.2; no longer C45.1, U8.1 (IN+)
- net at C37.2, D9.1 (A1), D9.2 (K2)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: now also U7.2 (VIN+); no longer U6.4 (IN+)
- net +5V_INV: now reaches U7.1 (VDD1)
- net +5V_INV: now also D17.2 (K2), C66.1, C73.1, U17.1 (VDD1)
- net at U7.6 (VOUT-): now also R21.2
- net at U7.7 (VOUT+): now also R19.2
- net +3V3_ADC: now reaches U7.8 (VDD2)
- net +3V3_ADC: now also C38.2, U6.3 (V+), C68.1, C74.1, U17.8 (VDD2)
- removed net +3V3_ISO: C38.2, C46.2, D17.2 (K2), U6.3 (V+), U8.5 (VDD)
- net AGND renamed GND_ADC
- net GND_ADC: now also C100.1, C38.1, C39.1, C45.2, C46.1, C48.2, U6.1 (REF), U6.2 (GND), C68.2, C74.2, U17.5 (GND2); no longer U18.2 (VSS), U19.2 (VSS)
- net AVDD: no longer names the net of C104.2, U19.5 (VDD)
- net AVDD: no longer C95.2, U18.5 (VDD)
- removed net GND_ISO: C100.1, C38.1, C39.1, C45.2, C46.1, C48.2, D17.1 (A1), R77.2, U6.1 (REF), U6.2 (GND), U7.4 (GND1), U8.2 (VSS)
- net MC_IDC_SEN_N renamed MC_IDC_N
- net MC_IDC_SEN_P renamed MC_IDC_P
- new net: R13.2, R7.1, R77.2
- new net: C45.1, U8.1 (IN+)
- new net: C46.2, U8.5 (VDD)
- new net: C65.2, D18.1 (A1), D18.2 (K2), R11.1, U17.2 (VIN+)
- new net: C65.1, D18.3 (COM), R13.1, U17.3 (VIN-)
- new net: C75.2, R19.1, U6.4 (IN+)
- new net: C75.1, R21.1, U6.5 (IN-)
- new net: C95.2, U18.5 (VDD)
- new net GND_INV: C66.2, C73.2, D17.1 (A1), R7.2, U17.4 (GND1), U7.4 (GND1)
Other:
- moved on the sheet: C100, C37, C38, C39, C45, C46, C48, D17, D9, R50, R51, R52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

Commit message: V1 schematic update 15
Parts:
- removed C103, C106: 1nF, SAMPI:CAP0603, symbol SAMPI:CERCAP
- removed C104: 100nF, SAMPI:CAP0603, symbol SAMPI:CERCAP
- removed R100, R78: 10R, SAMPI:RES0603, symbol SAMPI:RES
- removed R98, R99: 100K, SAMPI:RES0603, symbol SAMPI:RES
- added C70: 100nF, SAMPI:CAP0603, symbol SAMPI:CERCAP
- added C76, C77: 1nF, SAMPI:CAP0603, symbol SAMPI:CERCAP
- added R22, R23: 100K, SAMPI:RES0603, symbol SAMPI:RES
- added R24, R25: 10R, SAMPI:RES0603, symbol SAMPI:RES
- added R26, R27: 10K, SAMPI:RES0603, symbol SAMPI:RES
- added R28, R29: 4.99K, SAMPI:RES0603, symbol SAMPI:RES
- C46, C48: value 100nF -> 1nF; MNP CL10B104KB8NNNC -> CL10B102KB8NNNC
- U6: MFT Diodes -> Onsemi; MNP ZXCT199QA1DW-7 -> NCS199A1RSQT2G
Connections:
- net +3V3_ADC is gone; now on net +5V_MCU: C38.2, C68.1, C74.1, U17.8 (VDD2), U6.3 (V+), U7.8 (VDD2)
- net GND_ADC: now also C48.1, C76.1; no longer C102.1, C38.1, C45.2, C46.1, C48.2, C68.2, C74.2, C95.1, R96.2, U17.5 (GND2), U6.2 (GND), U7.5 (GND2)
- net MC_IU_HAL: now also R22.1; no longer R97.1
- net MC_IU_SEN: now also C48.2, R24.1; no longer C10.2, R80.1
- net MC_IV_HAL: now also R97.1
- net MC_IV_SEN: now also C10.2, R80.1
- net MC_VDC_DIV: now also C76.2, R25.1; no longer C48.1
- net +5V_MCU: now reaches U19.5 (VDD)
- net +5V_MCU: now also C45.2, C95.2, U18.5 (VDD), U8.5 (VDD), C70.2
- net at U19.3 (IN-): now also C77.1, R27.1, R29.1; no longer U19.4 (OUT)
- net at U8.1 (IN+): now also C46.2, R22.2, R23.1; no longer C45.1
- net GND_MCU: now reaches U8.2 (VSS)
- net GND_MCU: now also C102.1, C38.1, C45.1, C46.1, C68.2, C74.2, C95.1, R96.2, U17.5 (GND2), U18.2 (VSS), U19.2 (VSS), U6.2 (GND), U7.5 (GND2), C70.1, R23.2, R28.2
- net at U8.3 (IN-), U8.4 (OUT): now also R24.2
- net at U17.6 (VOUT-): now also R27.2
- net at U17.7 (VOUT+): now also R26.2
- net at U19.1 (IN+): now also C77.2, R26.1, R28.1
- new net: R25.2, R29.2, U19.4 (OUT)
Other:
- note added: "VOUT=(VOUTP-VOUTN)×(4.99k/10k)+VCM"
- company: TON DUC THANG UNIVERSITY -> (none)
- moved on the sheet: C10, C102, C95, R80, R96, R97, U18

Commit message: V1 schematic update 16
Parts:
- R22, R23, R62, R67, R73, R96, R97: value 100K -> 100K, 1%
- R26, R27: value 10K -> 10K, 1%; MNP RC0603FR-0710RL -> RC0603FR-0710KL
- R28, R29: value 4.99K -> 4.99K, 1%; MFT YAGEO -> (none); MNP RC0603FR-0710RL -> (none)
- R7, R77: MFT YAGEO -> (none); MNP AC0603FR-071K1L -> (none)
Connections:
- net MC_VDC_DIV renamed MC_UDC_DIV
Other:
- note added: "HIGH VOLTAGE ZONE"
- note added: "LOW VOLTAGE ZONE"
- moved on the sheet: C10, C102, C45, C46, C48, C95, R22, R23, R24, R80, R96, R97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

Commit message: V1 schematic update 17
Parts:
- removed R7: 100R, SAMPI:RES0603, symbol SAMPI:RES
- R30: renamed from R77; value 1K -> 1.1K, 1%; MFT (none) -> YAGEO; MNP (none) -> RC0603FR-071K1L
- R31: renamed from R50; value 10R -> 10R, 1%
- R32: renamed from R51; value 10R -> 10R, 1%
- R33: renamed from R11; value 10R -> 10R, 1%
- R34: renamed from R13; value 10R -> 10R, 1%
- R35: renamed from R19; value 10R -> 10R, 1%
- R36: renamed from R21; value 10R -> 10R, 1%
- R39: renamed from R28; MFT (none) -> YAGEO; MNP (none) -> RC0603FR-074K99L
- R40: renamed from R29; MFT (none) -> YAGEO; MNP (none) -> RC0603FR-074K99L
- R41: renamed from R25; value 10R -> 10R, 1%
- R42: renamed from R52; value 10R -> 10R, 1%
- R47: renamed from R24; value 10R -> 10R, 1%
- R48: renamed from R80; value 10R -> 10R, 1%
- U14: renamed from U7; footprint (none) -> SAMPI:SOP8-2.54
- U15: renamed from U17; footprint (none) -> SAMPI:SOP8-2.54
- renumbered C37 to C64, C73 to C66, C66 to C67, C74 to C68, C68 to C69, C75 to C70, C77 to C71, C38 to C72, C70 to C73, C76 to C74, C100 to C75, C39 to C76, C46 to C77, C102 to C78, C45 to C79, C95 to C80, C48 to C81, C10 to C82, D17 to D14, D9 to D15, D18 to D16, R62 to R27, R67 to R28, R73 to R29, R26 to R37, R27 to R38, R22 to R43, R23 to R44, R97 to R45, R96 to R46, U6 to U16, U19 to U17, U8 to U18, U18 to U19
Connections:
- net GND_INV: now also R30.2, R34.2

Commit message: V1 schematic update 22
Parts:
- removed C64, C70, C75, C76: 1nF, SAMPI:CAP0603, symbol SAMPI:CERCAP
- removed C66, C68, C72: 100nF, SAMPI:CAP0603, symbol SAMPI:CERCAP
- removed D15, D16: GP DIODE, SAMPI:SOT23, symbol SAMPI:DIODE_ARR1
- removed R31, R32, R35, R36, R42: 10R, 1%, SAMPI:RES0603, symbol SAMPI:RES
- removed U14: ISO OPAMP 1-CH, SAMPI:SOP8-2.54, symbol SAMPI:ISO-OPAMP
- removed U16: ISEN 50mV/V, SAMPI:SOT363, symbol SAMPI:ZXCT199Q
- added C10: 100pF/2kV, SAMPI:CAP1206, symbol SAMPI:CERCAP
- added C5, C7: 1nF, SAMPI:CAP0603, symbol SAMPI:CERCAP
- added C6: 100nF, SAMPI:CAP0603, symbol SAMPI:CERCAP
- added R1, R2: 100K, 1%, SAMPI:RES0603, symbol SAMPI:RES
- added R3: 10R, 1%, SAMPI:RES0603, symbol SAMPI:RES
- added U2: OP-1CH, SAMPI:SOT353, symbol SAMPI:NCV21871SQ3T2G
Connections:
- net +5V_MCU: now also C6.2, U2.5 (VDD)
- net GND_ADC: now also C7.1
- net GND_MCU: now also C5.1, C6.1, R2.2, U2.2 (VSS)
- net MC_IDC_SEN: now also C7.2, R3.1
- net VDC: now also C10.1
- new net: C5.2, R1.2, R2.1, U2.1 (IN+)
- new net: R3.2, U2.3 (IN-), U2.4 (OUT)
- new net MC_IDC_HAL: R1.1
- new net PGND: C10.2
Other:
- note removed: "VOUT=(ILoad*RSen)*Gain+Vref Gain=50, Vref=0, RSen=5mR, Imax=13A, Vout=3.25V"
- moved on the sheet: D14, R27, R28, R29, R30, R33, R34

Commit message: Label & Case
Parts:
- C10, C5, C6, C65, C67, C69, C7, C71, C73, C74, C77, C78, C79, C80, C81, C82, D14, R1, R2, R27, R28, R29, R3, R30, R33, R34, R37, R38, R39, R40, R41, R43, R44, R45, R46, R47, R48, U15, U17, U18, U19, U2: now not fitted

Commit message: Update schematic
Parts:
- C10, C5, C6, C65, C67, C69, C7, C71, C73, C74, C77, C78, C79, C80, C81, C82, D14, R1, R2, R27, R28, R29, R3, R30, R33, R34, R37, R38, R39, R40, R41, R43, R44, R45, R46, R47, R48, U15, U17, U18, U19, U2: now fitted
