File: V2/Design/HW.ACIM-INV/Inverter.kicad_sch (KiCad schematic)
At the start: 72 parts, among them J16 HIGH VOLTAGE OUTPUTS, J2 U, J3 V, J4 W, J5 N, J6 U, J7 V, J8 W, J9 N, M5 560V/1.75kA, M6 560V/1.75kA, M7 560V/1.75kA, U13 CMP-1CH, U7 IPM 600V/15A

Commit message: V2 diagram & schematic update 2
Parts:
- removed C3, C51, C56, C61, C62, C63: 100nF, SAMPI:CAP0603, symbol SAMPI:CERCAP
- removed C4, C52, C57: 1nF, SAMPI:CAP0603, symbol SAMPI:CERCAP
- removed C46, C47, C48, C53, C54, C55: 10uF, SAMPI:CAP0603, symbol SAMPI:CERCAP
- removed C9: 680uF/450V, SAMPI:ESMQ451VSN681MA50S, symbol SAMPI:ELECCAP
- removed D1, D2, D3, D4, D5, D6: 5VZ, Liem:SOD-123FL_12, symbol SAMPI:TVS
- removed R22: 10K, SAMPI:RES0603, symbol SAMPI:RES
- removed R25: 1.2M, SAMPI:RES0603, symbol SAMPI:RES
- removed RV1: 20K, SAMPI:TC33X-2, symbol SAMPI:POT
- removed U13: CMP-1CH, SAMPI:SOT25_DIODES, symbol SAMPI:CMP-1CH
- added C11, C12, C13, C9: 1nF, SAMPI:CAP0603, symbol SAMPI:CERCAP
- added D1, D2, D?: 24VZ, SAMPI:SOD-123FL, symbol SAMPI:KDZ3.6B
- added D3, D4, D5, D6: 3.3VZ, SAMPI:SOD-123FL, symbol SAMPI:KDZ3.6B
- added R10, R7, R8, R9: 100R, SAMPI:RES0603, symbol SAMPI:RES
- added R?: SHUNT, symbol SAMPI:SHUNT
- added U?: NON-INVERT BUFFER, SAMPI:TSSOP20-4.4X6.5-0.65P, symbol SAMPI:74VHC541
- R16: value 10K -> 10K, 1%
Connections:
- net GND_INV: now also C11.1, C12.1, C13.1, C9.1, D3.A, D4.A, D5.A, D6.A
- net IPM_PWM_UH: now also C9.2, R7.1
- net IPM_PWM_UL: now also C11.2, R8.1
- net MC_PWM_UH: now also D3.K, R7.2
- net MC_PWM_UL: now also D4.K, R8.2
- net MC_U: now also U7.22 (U)
- net MC_W: now also U7.20 (W)
- net PGND: now also C8.2
- net at C39.+, C44.1, U7.4 (VBV): now also D1.K
- net at C39.-, C44.2, U7.3 (VSV): now also D1.A
- net at C38.+, C43.1, U7.2 (VBU): now also D?.K
- net at C38.-, C43.2, U7.1 (VSU): now also D?.A
- net at C40.-, C45.2, U7.5 (VSW): now also D2.A
- net at C40.+, C45.1, U7.6 (VBW): now also D2.K
- now unconnected: U7.17 (NW), U7.18 (NV), U7.19 (NU)
Other:
- note removed: "HIGH VOLTAGE ZONE"
- note removed: "LOW VOLTAGE ZONE"
- moved on the sheet: C38, C39, C40, C43, C44, C45, C49, C50, C8, C88, D13, D8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

Commit message: V2 diagram & schematic update 3
Parts:
- removed R?: SHUNT, symbol SAMPI:SHUNT
- added C14, C15: 1nF, SAMPI:CAP0603, symbol SAMPI:CERCAP
- added C46: 100nF, SAMPI:CAP0603, symbol SAMPI:CERCAP
- added D10, D15: 3.3VZ, SAMPI:SOD-123FL, symbol SAMPI:KDZ3.6B
- added J12: DIL20, symbol Liem:DIL20
- added R11, R12: 100R, SAMPI:RES0603, symbol SAMPI:RES
- added R17, R22, R24, R25, R31, R32: 10K, SAMPI:RES0603, symbol SAMPI:RES
Connections:
- net GND_INV: now also U?.1 (~{OE0}), U?.10 (GND), U?.19 (~{OE1}), U?.8 (A6), U?.9 (A7), C14.1, C15.1, C46.2, D10.A, D15.A, R17.2, R22.2, R24.2, R25.2, R31.2, R32.2
- net IPM_PWM_VH: now also C12.2, R9.1
- net IPM_PWM_VL: now also C13.2, R10.1
- net IPM_PWM_WH: now also C14.2, R11.1
- net IPM_PWM_WL: now also C15.2, R12.1
- net MC_PWM_UH: now also U?.2 (A0); no longer D3.K, R7.2
- net MC_PWM_UL: now also U?.3 (A1); no longer D4.K, R8.2
- net MC_PWM_VH: now also U?.4 (A2)
- net MC_PWM_VL: now also U?.5 (A3)
- net MC_PWM_WH: now also U?.6 (A4)
- net MC_PWM_WL: now also U?.7 (A5)
- net MC_U: no longer U7.22 (U)
- net MC_V: no longer U7.21 (V)
- net MC_W: no longer U7.20 (W)
- net BUF_PWM_VH: now reaches R9.2
- net BUF_PWM_VH: now also D5.K, U?.16 (Y2), R24.1
- net BUF_PWM_WL: now reaches U?.13 (Y5)
- net BUF_PWM_WL: now also D15.K, R12.2, R32.1
- net BUF_PWM_WH: now reaches U?.14 (Y4)
- net BUF_PWM_WH: now also D10.K, R11.2, R31.1
- net BUF_PWM_VL: now reaches U?.15 (Y3)
- net BUF_PWM_VL: now also D6.K, R10.2, R25.1
- net BUF_PWM_UL: now reaches U?.17 (Y1)
- net BUF_PWM_UL: now also D4.K, R8.2, R22.1
- net BUF_PWM_UH: now reaches U?.18 (Y0)
- net BUF_PWM_UH: now also D3.K, R7.2, R17.1
- net +3V3_INV: now reaches U?.20 (VCC)
- net +3V3_INV: now also C46.1
- no-connect marks 0 -> 2
Other:
- moved on the sheet: C11, C41, C9, D13, D3, D4, D8, R16, R18, R4, R7, R8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

Commit message: V2 diagram & schematic update 4
Connections:
- net VDC: now also J12.1, J12.2
- net IPM_NW: now reaches U7.17 (NW)
- net IPM_NV: now reaches U7.18 (NV)
- net IPM_NU: now reaches U7.19 (NU)
- net IPM_W: now reaches U7.20 (W)
- net IPM_V: now reaches U7.21 (V)
- net IPM_U: now reaches U7.22 (U)
Other:
- moved on the sheet: J12
Changed lines of the file:
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@@
 		)
 	)
+	(hierarchical_label "IPM_NV"
+		(shape output)
+		(at 92.71 81.28 0)
+		(effects
+			(font
+				(size 1.27 1.27)
+			)
+			(justify left)
+		)
+	)
 	(hierarchical_label "BUF_PWM_VH"
 		(shape input)
@@
 		)
 	)
+	(hierarchical_label "IPM_U"
+		(shape output)
+		(at 92.71 36.83 0)
+		(effects
+			(font
+				(size 1.27 1.27)
+			)
+			(justify left)
+		)
+	)
 	(hierarchical_label "IPM_PWM_UL"
 		(shape output)
@@
 		)
 	)
+	(hierarchical_label "IPM_NW"
+		(shape output)
+		(at 92.71 95.25 0)
+		(effects
+			(font
+				(size 1.27 1.27)
+			)
+			(justify left)
+		)
+	)
 	(hierarchical_label "MC_PWM_VL"
 		(shape input)
@@
 		)
 	)
+	(hierarchical_label "IPM_NU"
+		(shape output)
+		(at 92.71 67.31 0)
+		(effects
+			(font
+				(size 1.27 1.27)
+			)
+			(justify left)
+		)
+	)
 	(hierarchical_label "IPM_TEMP_SEN"
 		(shape output)
@@
 		)
 	)
+	(hierarchical_label "IPM_W"
+		(shape output)
+		(at 92.71 57.15 0)
+		(effects
+			(font
+				(size 1.27 1.27)
+			)
+			(justify left)
+		)
+	)
 	(hierarchical_label "BUF_PWM_WL"
 		(shape input)
@@
 		)
 	)
+	(hierarchical_label "IPM_V"
+		(shape output)
+		(at 92.71 46.99 0)
+		(effects
+			(font
+				(size 1.27 1.27)
+			)
+			(justify left)
+		)
+	)
 	(hierarchical_label "MC_PWM_VH"
 		(shape input)
@@
 	)
 	(symbol
+		(lib_id "power:VDC")
+		(at 139.7 44.45 90)
+		(unit 1)
+		(exclude_from_sim no)
+		(in_bom yes)
+		(on_board yes)
+		(dnp no)
+		(property "Reference" "#PWR0101"
+			(at 142.24 44.45 0)
+			(effects
+				(font
+					(face "Consolas")
+					(size 1.27 1.27)
+					(thickness 0.254)
+					(bold yes)
+				)
+				(hide yes)
+			)
+		)
+		(property "Value" "VDC"
+			(at 135.255 44.45 90)
+			(effects
+				(font
+					(face "Consolas")
+					(size 1.016 1.016)
+					(thickness 0.127)
+				)
+			)
+		)
+		(property "Footprint" ""
+			(at 139.7 44.45 0)
+			(effects
+				(font
+					(face "Consolas")
+					(size 1.016 1.016)
+					(thickness 0.127)
+				)
+				(hide yes)
+			)
+		)
+		(property "Datasheet" ""
+			(at 139.7 44.45 0)
+			(effects
+				(font
+					(face "Consolas")
+					(size 1.016 1.016)
+					(thickness 0.127)
+				)
+				(hide yes)
+			)
+		)
+		(property "Description" ""
+			(at 139.7 44.45 0)
+			(effects
+				(font
+					(face "Consolas")
+					(size 1.016 1.016)
+					(thickness 0.127)
+				)
+				(hide yes)
+			)
+		)
+		(pin "1"
+		)
+		(instances
+			(project "HW.ACIM-INV"
+				(path "/20f80521-75f2-4ccc-bb34-c9566e70ef5c/220ce183-b27e-490b-828f-5201e8e92b41"
+					(reference "#PWR0101")
+					(unit 1)
+				)
+			)
+		)
+	)
+	(symbol
 		(lib_id "SAMPI:KDZ3.6B")
 		(at 33.02 170.18 270)
@@
 	)
 	(symbol
+		(lib_id "power:VDC")
+		(at 148.59 44.45 270)
+		(mirror x)
+		(unit 1)
+		(exclude_from_sim no)
+		(in_bom yes)
+		(on_board yes)
+		(dnp no)
+		(property "Reference" "#PWR0102"
+			(at 146.05 44.45 0)
+			(effects
+				(font
+					(face "Consolas")
+					(size 1.27 1.27)
+					(thickness 0.254)
+					(bold yes)
+				)
+				(hide yes)
+			)
+		)
+		(property "Value" "VDC"
+			(at 153.035 44.45 90)
+			(effects
+				(font
+					(face "Consolas")
+					(size 1.016 1.016)
+					(thickness 0.127)
+				)
+			)
+		)
+		(property "Footprint" ""
+			(at 148.59 44.45 0)
+			(effects
+				(font
+					(face "Consolas")
+					(size 1.016 1.016)
+					(thickness 0.127)
+				)
+				(hide yes)
+			)
+		)
+		(property "Datasheet" ""
+			(at 148.59 44.45 0)
+			(effects
+				(font
+					(face "Consolas")
+					(size 1.016 1.016)
+					(thickness 0.127)
+				)
+				(hide yes)
+			)
+		)
+		(property "Description" ""
+			(at 148.59 44.45 0)
+			(effects
+				(font
+					(face "Consolas")
+					(size 1.016 1.016)
+					(thickness 0.127)
+				)
+				(hide yes)
+			)
+		)
+		(pin "1"
+		)
+		(instances
+			(project "HW.ACIM-INV"
+				(path "/20f80521-75f2-4ccc-bb34-c9566e70ef5c/220ce183-b27e-490b-828f-5201e8e92b41"
+					(reference "#PWR0102")
+					(unit 1)
+				)
+			)
+		)
+	)
+	(symbol
 		(lib_id "SAMPI:GND_MCU")
 		(at 181.61 157.48 0)
@@
 	(symbol
 		(lib_id "Liem:DIL20")
-		(at 130.175 45.085 0)
+		(at 144.145 41.275 0)
 		(unit 1)
 		(exclude_from_sim no)
@@
 		(on_board yes)
 		(dnp no)
-		(fields_autoplaced yes)
 		(property "Reference" "J12"
-			(at 130.175 42.545 0)
+			(at 144.145 39.37 0)
 			(effects
 				(font
@@
 		)
 		(property "Value" "DIL20"
-			(at 130.175 45.085 0)
+			(at 144.145 41.91 0)
 			(effects
 				(font
@@
 		)
 		(property "Footprint" ""
-			(at 130.175 45.085 0)
+			(at 144.145 41.275 0)
 			(effects
 				(font
@@
 		)
 		(property "Datasheet" ""
-			(at 130.175 45.085 0)
+			(at 144.145 41.275 0)
 			(effects
 				(font
@@
 		)
 		(property "Description" ""
-			(at 130.175 45.085 0)
+			(at 144.145 41.275 0)
 			(effects
 				(font
