File: V1/Design/HW.ACIM-MCU-ADAP/HW.ACIM-MCU-ADAP.kicad_pcb (KiCad board)
At the start: 4 copper layers, 81.1 x 67.8 mm, 138 parts, among them J1 U, J101 HEADER 2x15POS, J102 HEADER 2x15POS, J2 V, J3 W, J4 PGND, J5 QWIIC, U1 ISO OPAMP 1-CH, U101 MIPS 32-bit DSC, U102 24MHz, U15 ISO OPAMP 1-CH, U17 OP-1CH, U2 ISO OPAMP 1-CH, U3 OP-1CH, U4 OP-1CH, U5 LDO 3.3V

Commit message: HW.ACIM-MCU-ADAP_V0.0 update ibom
Parts:
- D1, D14, D2: value GP DIODE -> BAV99

Commit message: Update Adaptor
Parts:
- turned U5 to 90 degrees
Connections:
- U5 pad 2: Net-(MD1-DC+) -> +3V3_ISO
- U5 pad 3: +3V3_ISO -> Net-(MD1-DC+)
Routing:
- net Net-(MD1-DC+): track 8.55 -> 10.4 mm
